File: testBench.brd (EAGLE design)
At the start: 35.5 x 54.3 mm, 29 parts, among them IC1 NCS21911SN2T1G, IC2 NCS21911SN2T1G, IC3 NCS21911SN2T1G, IC4 NCS21911SN2T1G, IC5 NCS21911SN2T1G

Commit message: This is my second PCB for opamp test bench
Parts:
- moved C10 2.29 mm to (15.0, 15.2)
- moved C2 2.29 mm to (21.3, 49.5)
- moved C5 2.29 mm to (15.0, 36.8)
- moved C6 2.29 mm to (15.0, 30.5)
- moved C8 2.29 mm to (15.0, 27.9)
- moved R10 2.29 mm to (15.0, 2.54)
- moved R11 2.29 mm to (15.0, 10.2)
- moved R12 2.29 mm to (15.0, 7.62)
- moved R3 2.29 mm to (15.0, 34.3)
- moved R4 2.29 mm to (15.0, 25.4)
- moved R5 2.29 mm to (15.0, 22.9)
- moved R6 2.29 mm to (15.0, 17.8)
- moved R8 2.29 mm to (15.0, 20.3)
- moved R9 2.29 mm to (15.0, 5.08)
- moved C1 2.29 mm to (18.8, 49.5)
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Routing:
- net OUTPUT3: track 47.5 -> 30.7 mm, vias 3 -> 2
- net VCC3: track 18.0 -> 30.3 mm
- net VCC2: track 19.5 -> 24.2 mm
- net N$9: track 0.37 -> 4.86 mm
- net OUTPUT4: track 50.1 -> 45.8 mm, vias 0 -> 4
- net VCC4: track 28.8 -> 32.6 mm
- net OUTPUT2: track 22.9 -> 25.2 mm, vias 2 -> 0
- net OUTPUT1: track 21.5 -> 23.8 mm, vias 2 -> 0
- net INPUT3: track 11.3 -> 13.6 mm, vias 2 -> 1
- net INPUT5: track 10.3 -> 12.5 mm
- net VCC1: track 23.3 -> 24.9 mm, vias 0 -> 1
- net INPUT2: track 22.4 -> 21.0 mm, vias 2 -> 1
- net INPUT4: track 18.9 -> 19.7 mm, vias 2 -> 1
- net INPUT1: track 31.2 -> 30.7 mm, vias 2 -> 1
Other:
- board size 35.5 x 54.3 mm -> 34.3 x 54.3 mm
- board text added: "GND"
- board text added: "IN1"
- board text added: "IN2"
- board text added: "IN3"
- board text added: "IN4"
- board text added: "IN5"
- board text added: "OUT1"
- board text added: "OUT2"
- board text added: "OUT3"
- board text added: "OUT4"
- board text added: "VCC1"
- board text added: "VCC2"
- board text added: "VCC3"
- board text added: "VCC4"

Commit message: This is my third PCB for opamp test bench
Parts:
- moved JP3 1.27 mm to (2.54, 26.7)
Connections:
- removed net N$44: JP3.15
- new net EMPTY: JP3.5
- net GND: now also JP3.10; no longer JP3.9
- net INPUT1: now also JP3.11; no longer JP3.10
- net INPUT2: now also JP3.12; no longer JP3.11
- net INPUT3: now also JP3.13; no longer JP3.12
- net INPUT4: now also JP3.14; no longer JP3.13
- net INPUT5: now also JP3.15; no longer JP3.14
- net VCC1: now also JP3.6; no longer JP3.5
- net VCC2: now also JP3.7; no longer JP3.6
- net VCC3: now also JP3.8; no longer JP3.7
- net VCC4: now also JP3.9; no longer JP3.8
Routing:
- net VCC4: track 32.6 -> 25.8 mm
- net INPUT1: track 30.7 -> 35.3 mm
- net VCC1: track 24.9 -> 28.0 mm
- net INPUT4: track 19.7 -> 16.8 mm
- net INPUT2: track 21.0 -> 23.5 mm
- net VCC3: track 30.3 -> 31.8 mm
- net VCC2: track 24.2 -> 25.8 mm
- net INPUT5: track 12.5 -> 14.1 mm
- net INPUT3: track 13.6 -> 15.2 mm
- net OUTPUT4: track 45.8 -> 44.7 mm
- net OUTPUT2: track 25.2 -> 24.7 mm
- net OUTPUT1: track 23.8 -> 23.3 mm

Commit message: PCB test bench fourth version
Parts:
- removed C1, C10, C12, C3, C6: CGA3E2X7R1H104K080AE, SamacSys_Parts:CAPC1608X90N
- added TP1, TP2, TP3, TP4, TP5, TP6, TP7, TP8: (no value), SamacSys_Parts:1.85X3.45_MM
- moved R6 8.92 mm to (23.4, 20.8), turned to 90 degrees
Connections:
- removed net N$16: C11.1, IC5.5
- removed net N$17: C10.2, IC5.2
- removed net N$2: C1.2, IC1.2
- removed net N$3: C2.1, IC1.5
- removed net N$4: C3.2, IC2.2
- removed net N$5: C4.1, IC2.5
- removed net N$6: C6.2, IC3.2
- removed net N$7: C7.1, IC3.5
- removed net N$8: C13.1, IC4.5
- removed net N$9: C12.2, IC4.2
- net GND: now also C11.2, C13.2, C2.2, C4.2, C7.2, IC1.2, IC2.2, IC3.2, IC4.2, IC5.2, TP1.TP, TP3.TP, TP5.TP, TP7.TP; no longer C1.1, C10.1, C12.1, C3.1, C6.1
- net OUTPUT1: now also TP2.TP
- net OUTPUT2: now also TP4.TP
- net OUTPUT3: now also TP6.TP
- net OUTPUT4: now also TP8.TP
- net VCC1: now also C2.1, IC1.5; no longer C2.2
- net VCC2: now also C4.1, IC2.5; no longer C4.2
- net VCC3: now also C11.1, C7.1, IC3.5, IC5.5; no longer C11.2, C7.2
- net VCC4: now also C13.1, IC4.5; no longer C13.2
Routing:
- net OUTPUT3: track 31.1 -> 42.2 mm
- net OUTPUT4: track 44.7 -> 52.8 mm
- net N$6: track 6.83 -> 0.00 mm
- net VCC3: track 31.8 -> 38.0 mm, vias 0 -> 3
- net GND: track 0.00 -> 5.01 mm, vias 20 -> 22
- net OUTPUT1: track 23.3 -> 28.2 mm
- net N$9: track 4.86 -> 0.00 mm
- net N$2: track 4.29 -> 0.00 mm
- net N$4: track 4.29 -> 0.00 mm
- net N$20: track 10.2 -> 14.3 mm
- net N$17: track 3.56 -> 0.00 mm
- net OUTPUT2: track 24.7 -> 27.8 mm
- net N$18: track 5.40 -> 7.47 mm
- net N$5: track 2.07 -> 0.00 mm
- net N$8: track 2.07 -> 0.00 mm
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Other:
- board size 34.3 x 54.3 mm -> 36.8 x 54.3 mm

Commit message: PCB test bench fifth version
Parts:
- flipped JP3 to the bottom
Other:
- board text added: "John Tran BAJA SAE 2021-2022"
Changed lines of the file:
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@@
 <setting verticaltext="up"/>
 </settings>
-<grid distance="10" unitdist="mil" unit="mil" style="lines" multiple="1" display="no" altdistance="5" altunitdist="mil" altunit="mil"/>
+<grid distance="50" unitdist="mil" unit="mil" style="lines" multiple="1" display="no" altdistance="5" altunitdist="mil" altunit="mil"/>
 <layers>
 <layer number="1" name="Top" color="4" fill="1" visible="yes" active="yes"/>
@@
 <text x="29.718" y="3.048" size="1.27" layer="25" rot="R90">OUT4</text>
 <text x="29.718" y="23.368" size="1.27" layer="25" rot="R90">OUT3</text>
+<text x="31.75" y="8.89" size="1.778" layer="22" rot="MR0">John Tran
+BAJA SAE 2021-2022</text>
 </plain>
 <attributes>
@@
 <attribute name="NAME" x="12.446" y="36.83" size="0.8128" layer="25" align="center"/>
 </element>
-<element name="JP3" library="pinhead" library_urn="urn:adsk.eagle:library:325" package="1X15" package3d_urn="urn:adsk.eagle:package:22424/2" value="" x="2.54" y="26.67" smashed="yes" rot="R270">
-<attribute name="NAME" x="1.1938" y="47.5488" size="0.8128" layer="25" ratio="10"/>
-<attribute name="POPULARITY" value="4" x="2.54" y="26.67" size="1.778" layer="27" rot="R270" display="off"/>
-<attribute name="VALUE" x="-0.635" y="45.72" size="1.27" layer="27" rot="R270"/>
+<element name="JP3" library="pinhead" library_urn="urn:adsk.eagle:library:325" package="1X15" package3d_urn="urn:adsk.eagle:package:22424/2" value="" x="2.54" y="26.67" smashed="yes" rot="MR270">
+<attribute name="NAME" x="3.8862" y="47.5488" size="0.8128" layer="26" ratio="10" rot="MR0"/>
+<attribute name="POPULARITY" value="4" x="2.54" y="26.67" size="1.778" layer="28" rot="MR270" display="off"/>
+<attribute name="VALUE" x="5.715" y="45.72" size="1.27" layer="28" rot="MR270"/>
 </element>
 <element name="TP1" library="SamacSys_Parts" package="1.85X3.45_MM" value="" x="24.384" y="47.752" smashed="yes">
@@
 <contactref element="JP3" pad="1"/>
 <wire x1="19.726" y1="43.18" x2="21.316" y2="44.77" width="0.254" layer="1"/>
-<wire x1="2.54" y1="44.45" x2="3.81" y2="43.18" width="0.254" layer="1"/>
 <wire x1="3.81" y1="43.18" x2="19.726" y2="43.18" width="0.254" layer="1"/>
 <contactref element="TP2" pad="TP"/>
 <wire x1="26.2128" y1="44.8818" x2="21.4278" y2="44.8818" width="0.254" layer="1"/>
 <wire x1="21.4278" y1="44.8818" x2="21.316" y2="44.77" width="0.254" layer="1"/>
+<wire x1="2.54" y1="44.45" x2="3.81" y2="43.18" width="0.254" layer="1"/>
 </signal>
 <signal name="GND">
@@
 <wire x1="15.306" y1="44.77" x2="18.816" y2="44.77" width="0.254" layer="1"/>
 <contactref element="JP3" pad="11"/>
+<wire x1="6.35" y1="22.86" x2="6.35" y2="37.084" width="0.254" layer="16"/>
 <wire x1="2.54" y1="19.05" x2="6.35" y2="22.86" width="0.254" layer="16"/>
-<wire x1="6.35" y1="22.86" x2="6.35" y2="37.084" width="0.254" layer="16"/>
 </signal>
 <signal name="OUTPUT2">
@@
 <contactref element="TP4" pad="TP"/>
 <wire x1="18.816" y1="36.51" x2="18.816" y2="38.334" width="0.254" layer="1"/>
-<wire x1="18.816" y1="38.334" x2="15.24" y2="41.91" width="0.254" layer="1"/>
-<wire x1="15.24" y1="41.91" x2="2.54" y2="41.91" width="0.254" layer="1"/>
+<wire x1="15.24" y1="41.91" x2="18.816" y2="38.334" width="0.254" layer="1"/>
 <wire x1="26.2128" y1="34.7218" x2="21.4278" y2="34.7218" width="0.254" layer="1"/>
 <wire x1="21.4278" y1="34.7218" x2="21.316" y2="34.61" width="0.254" layer="1"/>
+<wire x1="2.54" y1="41.91" x2="15.24" y2="41.91" width="0.254" layer="1"/>
 </signal>
 <signal name="N$13">
@@
 <wire x1="9.906" y1="33.274" x2="7.62" y2="35.56" width="0.254" layer="16"/>
 <via x="7.62" y="35.56" extent="1-16" drill="0.35"/>
-<wire x1="7.62" y1="35.56" x2="3.81" y2="35.56" width="0.254" layer="1"/>
-<wire x1="3.81" y1="35.56" x2="2.54" y2="36.83" width="0.254" layer="1"/>
+<wire x1="3.81" y1="35.56" x2="7.62" y2="35.56" width="0.254" layer="1"/>
 <contactref element="TP8" pad="TP"/>
 <wire x1="26.4668" y1="4.2418" x2="23.1902" y2="4.2418" width="0.254" layer="1"/>
@@
 <wire x1="20.13613125" y1="5.08" x2="19.18613125" y2="6.03" width="0.254" layer="1"/>
 <wire x1="22.352" y1="5.08" x2="20.13613125" y2="5.08" width="0.254" layer="1"/>
+<wire x1="2.54" y1="36.83" x2="3.81" y2="35.56" width="0.254" layer="1"/>
 </signal>
 <signal name="N$15">
@@
 <signal name="INPUT2">
 <contactref element="R3" pad="1"/>
-<wire x1="12.446" y1="27.94" x2="12.446" y2="34.29" width="0.254" layer="16"/>
 <via x="12.446" y="34.29" extent="1-16" drill="0.35"/>
+<wire x1="12.446" y1="26.67" x2="12.446" y2="34.29" width="0.254" layer="16"/>
 <wire x1="12.446" y1="34.29" x2="14.0462" y2="34.29" width="0.254" layer="1"/>
 <contactref element="JP3" pad="12"/>
 <wire x1="2.54" y1="16.51" x2="12.446" y2="26.416" width="0.254" layer="16"/>
-<wire x1="12.446" y1="26.416" x2="12.446" y2="27.94" width="0.254" layer="16"/>
+<wire x1="12.446" y1="26.416" x2="12.446" y2="26.67" width="0.254" layer="16"/>
 </signal>
 <signal name="INPUT5">
 <contactref element="JP3" pad="15"/>
-<wire x1="2.54" y1="8.89" x2="6.35" y2="12.7" width="0.254" layer="1"/>
-<wire x1="6.35" y1="12.7" x2="11.43" y2="12.7" width="0.254" layer="1"/>
+<wire x1="6.35" y1="12.7" x2="11.496" y2="12.7" width="0.254" layer="1"/>
 <contactref element="R11" pad="2"/>
 <wire x1="14.036" y1="10.16" x2="11.496" y2="12.7" width="0.254" layer="1"/>
-<wire x1="11.496" y1="12.7" x2="11.43" y2="12.7" width="0.254" layer="1"/>
+<wire x1="2.54" y1="8.89" x2="6.35" y2="12.7" width="0.254" layer="1"/>
 </signal>
 <signal name="INPUT4">
@@
 <wire x1="8.636" y1="2.54" x2="14.036" y2="2.54" width="0.254" layer="1"/>
 <contactref element="JP3" pad="14"/>
+<wire x1="8.636" y1="5.08" x2="8.636" y2="2.54" width="0.254" layer="16"/>
 <wire x1="2.54" y1="11.43" x2="8.636" y2="5.334" width="0.254" layer="16"/>
-<wire x1="8.636" y1="5.334" x2="8.636" y2="2.54" width="0.254" layer="16"/>
+<wire x1="8.636" y1="5.334" x2="8.636" y2="5.08" width="0.254" layer="16"/>
 </signal>
 <signal name="N$1">
@@
 <wire x1="12.446" y1="22.86" x2="14.0462" y2="22.86" width="0.254" layer="1"/>
 <contactref element="JP3" pad="13"/>
+<wire x1="11.43" y1="22.86" x2="12.446" y2="22.86" width="0.254" layer="16"/>
 <wire x1="2.54" y1="13.97" x2="11.43" y2="22.86" width="0.254" layer="16"/>
-<wire x1="11.43" y1="22.86" x2="12.446" y2="22.86" width="0.254" layer="16"/>
 </signal>
 <signal name="N$18">
@@
 <wire x1="11.176" y1="38.354" x2="10.16" y2="39.37" width="0.254" layer="16"/>
 <via x="10.16" y="39.37" extent="1-16" drill="0.35"/>
-<wire x1="10.16" y1="39.37" x2="2.54" y2="39.37" width="0.254" layer="1"/>
 <contactref element="TP6" pad="TP"/>
 <wire x1="23.368" y1="21.828" x2="26.1018" y2="24.5618" width="0.254" layer="1"/>
@@
 <wire x1="12.192" y1="21.59" x2="11.176" y2="22.606" width="0.254" layer="1"/>
 <wire x1="20.066" y1="22.352" x2="17.272" y2="22.352" width="0.254" layer="1"/>
+<wire x1="2.54" y1="39.37" x2="10.16" y2="39.37" width="0.254" layer="1"/>
 </signal>
 <signal name="N$20">
@@
 <wire x1="7.62" y1="31.75" x2="19.304" y2="31.75" width="0.254" layer="1"/>
 <contactref element="JP3" pad="8"/>
-<wire x1="2.54" y1="26.67" x2="7.62" y2="31.75" width="0.254" layer="1"/>
 <contactref element="IC5" pad="5"/>
 <contactref element="C11" pad="1"/>
@@
 <via x="20.066" y="16.764" extent="1-16" drill="0.35"/>
 <wire x1="20.066" y1="16.764" x2="20.066" y2="19.558" width="0.254" layer="16"/>
+<wire x1="2.54" y1="26.67" x2="7.62" y2="31.75" width="0.254" layer="1"/>
 </signal>
 <signal name="VCC2">
@@
 <via x="13.97" y="40.64" extent="1-16" drill="0.35"/>
 <wire x1="15.24" y1="41.91" x2="13.97" y2="40.64" width="0.254" layer="16"/>
-<wire x1="2.54" y1="29.21" x2="13.97" y2="40.64" width="0.254" layer="1"/>
 <contactref element="IC2" pad="5"/>
 <contactref element="C4" pad="1"/>
@@
 <via x="17.78" y="41.91" extent="1-16" drill="0.35"/>
 <wire x1="17.78" y1="41.91" x2="15.24" y2="41.91" width="0.254" layer="16"/>
+<wire x1="2.54" y1="29.21" x2="13.97" y2="40.64" width="0.254" layer="1"/>
 </signal>
 <signal name="VCC1">
 <contactref element="JP3" pad="6"/>
-<wire x1="2.54" y1="31.75" x2="5.08" y2="34.29" width="0.254" layer="16"/>
 <wire x1="5.08" y1="34.29" x2="5.08" y2="36.83" width="0.254" layer="16"/>
 <contactref element="IC1" pad="5"/>
@@
 <wire x1="18.542" y1="48.768" x2="21.062" y2="48.768" width="0.254" layer="1"/>
 <wire x1="21.062" y1="48.768" x2="21.316" y2="48.514" width="0.254" layer="1"/>
+<wire x1="2.54" y1="31.75" x2="5.08" y2="34.29" width="0.254" layer="16"/>
 </signal>
 <signal name="EMPTY">

Commit message: pcb test bench 6th version
Parts:
- removed R6: CRCW080510M0FKEB, SamacSys_Parts:RESC2012X50N
Connections:
- removed net N$18: IC5.1, R6.1, R7.1
- net OUTPUT3: now also IC5.1, R7.1; no longer R6.2
Routing:
- net N$18: track 7.47 -> 0.00 mm
- net OUTPUT3: track 42.2 -> 49.1 mm, vias 2 -> 4
- net GND: vias 22 -> 44
Changed lines of the file:
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@@
 <drawing>
 <settings>
-<setting alwaysvectorfont="yes"/>
+<setting alwaysvectorfont="no"/>
 <setting verticaltext="up"/>
 </settings>
-<grid distance="50" unitdist="mil" unit="mil" style="lines" multiple="1" display="no" altdistance="5" altunitdist="mil" altunit="mil"/>
+<grid distance="10" unitdist="mil" unit="mil" style="lines" multiple="1" display="no" altdistance="5" altunitdist="mil" altunit="mil"/>
 <layers>
 <layer number="1" name="Top" color="4" fill="1" visible="yes" active="yes"/>
@@
 <attribute name="NAME" x="21.336" y="22.098" size="0.8128" layer="25" rot="R180" align="center"/>
 </element>
-<element name="R6" library="SamacSys_Parts" package="RESC2012X50N" value="CRCW080510M0FKEB" x="23.368" y="20.828" smashed="yes" rot="R90">
-<attribute name="DESCRIPTION" value="Thick Film Resistors - SMD 1/8watt 10Mohms 1% 100ppm" x="23.368" y="20.828" size="1.778" layer="27" rot="R90" display="off"/>
-<attribute name="HEIGHT" value="0.5mm" x="23.368" y="20.828" size="1.778" layer="27" rot="R90" display="off"/>
-<attribute name="MANUFACTURER_NAME" value="Vishay" x="23.368" y="20.828" size="1.778" layer="27" rot="R90" display="off"/>
-<attribute name="MANUFACTURER_PART_NUMBER" value="CRCW080510M0FKEB" x="23.368" y="20.828" size="1.778" layer="27" rot="R90" display="off"/>
-<attribute name="MOUSER_PART_NUMBER" value="71-CRCW080510M0FKEB" x="23.368" y="20.828" size="1.778" layer="27" rot="R90" display="off"/>
-<attribute name="MOUSER_PRICE-STOCK" value="https://www.mouser.co.uk/ProductDetail/Vishay-Dale/CRCW080510M0FKEB?qs=LOX6nxTstiZgWRbGVrXCVQ%3D%3D" x="23.368" y="20.828" size="1.778" layer="27" rot="R90" display="off"/>
-<attribute name="NAME" x="23.368" y="23.114" size="0.8128" layer="25" align="center"/>
-</element>
 <element name="R8" library="SamacSys_Parts" package="RESC2013X65N" value="TNPW080510K0BEEN" x="14.986" y="20.32" smashed="yes" rot="R180">
 <attribute name="DESCRIPTION" value="RESISTOR, 0805 10K Ohms +/-0.1% 0.125 W" x="14.986" y="20.32" size="1.778" layer="27" rot="R180" display="off"/>
@@
 <via x="34.29" y="41.91" extent="1-16" drill="0.35"/>
 <via x="24.13" y="41.91" extent="1-16" drill="0.35"/>
-<via x="17.78" y="33.02" extent="1-16" drill="0.35"/>
+<via x="18.542" y="32.766" extent="1-16" drill="0.35"/>
 <contactref element="IC4" pad="2"/>
 <wire x1="18.44586875" y1="5.08" x2="18.816" y2="5.08" width="0.254" layer="1"/>
@@
 <wire x1="18.288" y1="25.4" x2="17.272" y2="26.416" width="0.254" layer="1"/>
 <via x="17.272" y="26.416" extent="1-16" drill="0.35"/>
+<via x="19.05" y="41.91" extent="1-16" drill="0.35"/>
+<via x="27.432" y="27.94" extent="1-16" drill="0.35"/>
+<via x="23.114" y="27.94" extent="1-16" drill="0.35"/>
+<via x="24.13" y="32.004" extent="1-16" drill="0.35"/>
+<via x="14.986" y="29.972" extent="1-16" drill="0.35"/>
+<via x="14.732" y="32.766" extent="1-16" drill="0.35"/>
+<via x="11.176" y="15.748" extent="1-16" drill="0.35"/>
+<via x="11.43" y="6.096" extent="1-16" drill="0.35"/>
+<via x="11.176" y="11.43" extent="1-16" drill="0.35"/>
+<via x="15.24" y="15.748" extent="1-16" drill="0.35"/>
+<via x="29.21" y="32.004" extent="1-16" drill="0.35"/>
+<via x="29.21" y="19.05" extent="1-16" drill="0.35"/>
+<via x="24.13" y="19.05" extent="1-16" drill="0.35"/>
+<via x="7.112" y="15.748" extent="1-16" drill="0.35"/>
+<via x="7.112" y="10.922" extent="1-16" drill="0.35"/>
+<via x="7.112" y="28.702" extent="1-16" drill="0.35"/>
+<via x="7.112" y="23.368" extent="1-16" drill="0.35"/>
+<via x="14.986" y="39.116" extent="1-16" drill="0.35"/>
+<via x="19.812" y="12.446" extent="1-16" drill="0.35"/>
+<via x="15.24" y="12.7" extent="1-16" drill="0.35"/>
+<via x="19.812" y="7.874" extent="1-16" drill="0.35"/>
+<via x="24.13" y="6.35" extent="1-16" drill="0.35"/>
+<wire x1="18.816" y1="16.51" x2="15.24" y2="15.748" width="0" layer="19" extent="1-1"/>
 </signal>
 <signal name="INPUT1">
@@
 <wire x1="2.54" y1="13.97" x2="11.43" y2="22.86" width="0.254" layer="16"/>
 </signal>
-<signal name="N$18">
-<contactref element="IC5" pad="1"/>
-<contactref element="R6" pad="1"/>
-<contactref element="R7" pad="1"/>
-<wire x1="18.796" y1="19.3802" x2="18.816" y2="19.3602" width="0.254" layer="1"/>
-<wire x1="18.816" y1="19.3602" x2="18.816" y2="17.46" width="0.254" layer="1"/>
-<wire x1="23.368" y1="19.828" x2="21.836" y2="18.296" width="0.254" layer="1"/>
-<wire x1="21.836" y1="18.296" x2="21.828" y2="18.288" width="0.254" layer="1"/>
-<wire x1="18.816" y1="17.46" x2="19.652" y2="18.296" width="0.254" layer="1"/>
-<wire x1="19.652" y1="18.296" x2="21.836" y2="18.296" width="0.254" layer="1"/>
-</signal>
 <signal name="OUTPUT3">
-<contactref element="R6" pad="2"/>
 <contactref element="JP3" pad="3"/>
 <via x="11.176" y="30.48" extent="1-16" drill="0.35"/>
-<wire x1="11.176" y1="22.606" x2="11.176" y2="30.48" width="0.254" layer="1"/>
 <wire x1="11.176" y1="30.48" x2="11.176" y2="38.354" width="0.254" layer="16"/>
 <wire x1="11.176" y1="38.354" x2="10.16" y2="39.37" width="0.254" layer="16"/>
 <via x="10.16" y="39.37" extent="1-16" drill="0.35"/>
 <contactref element="TP6" pad="TP"/>
-<wire x1="23.368" y1="21.828" x2="26.1018" y2="24.5618" width="0.254" layer="1"/>
-<wire x1="26.1018" y1="24.5618" x2="26.4668" y2="24.5618" width="0.254" layer="1"/>
-<wire x1="23.368" y1="21.828" x2="20.59" y2="21.828" width="0.254" layer="1"/>
-<wire x1="20.59" y1="21.828" x2="20.066" y2="22.352" width="0.254" layer="1"/>
-<wire x1="17.272" y1="22.352" x2="16.51" y2="21.59" width="0.254" layer="1"/>
-<wire x1="16.51" y1="21.59" x2="12.192" y2="21.59" width="0.254" layer="1"/>
-<wire x1="12.192" y1="21.59" x2="11.176" y2="22.606" width="0.254" layer="1"/>
-<wire x1="20.066" y1="22.352" x2="17.272" y2="22.352" width="0.254" layer="1"/>
+<wire x1="26.1018" y1="24.5618" x2="26.416" y2="24.5618" width="0.254" layer="1"/>
+<wire x1="26.416" y1="24.5618" x2="26.4668" y2="24.5618" width="0.254" layer="1"/>
 <wire x1="2.54" y1="39.37" x2="10.16" y2="39.37" width="0.254" layer="1"/>
+<contactref element="IC5" pad="1"/>
+<contactref element="R7" pad="1"/>
+<wire x1="18.796" y1="19.3802" x2="18.816" y2="19.3602" width="0.254" layer="1"/>
+<wire x1="18.816" y1="19.3602" x2="18.816" y2="17.46" width="0.254" layer="1"/>
+<wire x1="18.816" y1="17.46" x2="19.898" y2="18.542" width="0.254" layer="1"/>
+<wire x1="19.898" y1="18.542" x2="22.352" y2="18.542" width="0.254" layer="1"/>
+<wire x1="22.352" y1="18.542" x2="26.416" y2="22.606" width="0.254" layer="1"/>
+<wire x1="26.416" y1="22.606" x2="26.416" y2="24.5618" width="0.254" layer="1"/>
+<wire x1="18.796" y1="19.3802" x2="18.4658" y2="19.05" width="0.254" layer="1"/>
+<wire x1="18.4658" y1="19.05" x2="17.018" y2="19.05" width="0.254" layer="1"/>
+<via x="17.018" y="19.05" extent="1-16" drill="0.35"/>
+<wire x1="17.018" y1="19.05" x2="12.954" y2="19.05" width="0.254" layer="16"/>
+<wire x1="12.954" y1="19.05" x2="11.176" y2="20.828" width="0.254" layer="16"/>
+<via x="11.176" y="20.828" extent="1-16" drill="0.35"/>
+<wire x1="11.176" y1="20.828" x2="11.176" y2="30.48" width="0.254" layer="1"/>
 </signal>
 <signal name="N$20">
@@
 <wire x1="16.8656" y1="21.2598" x2="18.796" y2="21.2598" width="0.254" layer="1"/>
 <wire x1="21.316" y1="15.56" x2="20.234" y2="14.478" width="0.254" layer="1"/>
-<wire x1="20.234" y1="14.478" x2="17.526" y2="14.478" width="0.254" layer="1"/>
-<wire x1="17.526" y1="14.478" x2="15.9258" y2="16.0782" width="0.254" layer="1"/>
-<wire x1="15.9258" y1="16.0782" x2="15.9258" y2="20.32" width="0.254" layer="1"/>
+<wire x1="20.234" y1="14.478" x2="18.034" y2="14.478" width="0.254" layer="1"/>
+<wire x1="18.034" y1="14.478" x2="15.9258" y2="16.5862" width="0.254" layer="1"/>
+<wire x1="15.9258" y1="16.5862" x2="15.9258" y2="20.32" width="0.254" layer="1"/>
 </signal>
 <signal name="VCC4">
@@
 <wire x1="21.336" y1="38.57" x2="21.336" y2="36.53" width="0.254" layer="1"/>
 <wire x1="21.336" y1="36.53" x2="21.316" y2="36.51" width="0.254" layer="1"/>
-<wire x1="21.336" y1="38.57" x2="21.12" y2="38.57" width="0.254" layer="1"/>
-<wire x1="21.12" y1="38.57" x2="17.78" y2="41.91" width="0.254" layer="1"/>
-<via x="17.78" y="41.91" extent="1-16" drill="0.35"/>
-<wire x1="17.78" y1="41.91" x2="15.24" y2="41.91" width="0.254" layer="16"/>
+<wire x1="21.336" y1="38.57" x2="20.358" y2="38.57" width="0.254" layer="1"/>
+<wire x1="20.358" y1="38.57" x2="17.018" y2="41.91" width="0.254" layer="1"/>
+<via x="17.018" y="41.91" extent="1-16" drill="0.35"/>
+<wire x1="17.018" y1="41.91" x2="15.24" y2="41.91" width="0.254" layer="16"/>
 <wire x1="2.54" y1="29.21" x2="13.97" y2="40.64" width="0.254" layer="1"/>
 </signal>

Commit message: pcb test bench 7th version
Routing:
- net GND: vias 44 -> 45
Changed lines of the file:
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@@
 <via x="19.812" y="7.874" extent="1-16" drill="0.35"/>
 <via x="24.13" y="6.35" extent="1-16" drill="0.35"/>
-<wire x1="18.816" y1="16.51" x2="15.24" y2="15.748" width="0" layer="19" extent="1-1"/>
+<via x="17.018" y="17.526" extent="1-16" drill="0.35"/>
 </signal>
 <signal name="INPUT1">
