File: testBench.brd (EAGLE design)
At the start: 36.8 x 54.3 mm, 31 parts, among them IC1 NCS21911SN2T1G, IC2 NCS21911SN2T1G, IC3 NCS21911SN2T1G, IC4 NCS21911SN2T1G, IC5 NCS21911SN2T1G

Commit message: PCB test bench version 8th
Parts:
- added LED1, LED2, LED3, LED4: 150080GS75000, SamacSys_Parts:LEDM2012X80N
- added R13, R14, R15, R16: ERJ-P06J431V, SamacSys_Parts:ERJP06_(0805)
- moved C11 10.2 mm to (31.5, 20.3)
- moved C13 10.2 mm to (31.5, 8.89)
- moved C2 10.2 mm to (31.5, 49.5)
- moved C4 10.2 mm to (31.5, 39.4)
- moved C5 10.2 mm to (25.1, 36.8)
- moved C7 10.2 mm to (31.5, 29.2)
- moved C8 10.2 mm to (25.1, 27.9)
- moved C9 10.2 mm to (29.0, 29.2)
- moved IC1 10.2 mm to (30.2, 45.7)
- moved IC2 10.2 mm to (30.2, 35.6)
- moved IC3 10.2 mm to (30.2, 25.4)
- moved IC4 10.2 mm to (30.2, 5.08)
- moved IC5 10.2 mm to (30.2, 16.5)
- moved JP3 10.2 mm to (12.7, 26.7)
- moved R10 10.2 mm to (25.1, 2.54)
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Connections:
- new net N$23: LED1.2, R13.2
- new net N$30: LED2.2, R14.2
- new net N$31: LED3.2, R15.2
- new net N$32: LED4.2, R16.2
- net GND: now also LED1.1, LED2.1, LED3.1, LED4.1
- net VCC1: now also R13.1
- net VCC2: now also R14.1
- net VCC3: now also R15.1
- net VCC4: now also R16.1
Routing:
- net VCC1: track 29.5 -> 34.6 mm
- net VCC4: track 27.5 -> 32.6 mm
- net VCC2: track 27.5 -> 32.4 mm
- net VCC3: track 38.0 -> 42.3 mm
- net N$32: track 0.00 -> 3.98 mm
- net N$23: track 0.00 -> 3.72 mm
- net N$30: track 0.00 -> 3.14 mm
- net N$31: track 0.00 -> 3.09 mm
- net GND: vias 45 -> 53
Other:
- board size 36.8 x 54.3 mm -> 47 x 54.3 mm
