File: FAST_DEPLOY_E_FUSE.sch (EAGLE design)
At the start: 23 parts, among them IC1 LTC4222CUH#PBF, U1 SSM6N67NU,LF

Commit message: 2 Efuses are on board now with seperate net names
Parts:
- added C10, C6, C7: CGA5L2C0G1H104J160AA, SamacSys_Parts:CGA5L2C0G1H104J160AA
- added C8: CGA4J3X7R1H105K125AB, SamacSys_Parts:CGA4J3X7R1H105K125AB
- added C9: CGA3E2X7R1H683K080AA, SamacSys_Parts:CGA3E2X7R1H683K080AA
- added IC2: LTC4222CUH#PBF, SamacSys_Parts:LTC4222CUH#PBF
- added R17, R18, R23, R24, R28, R31: CRCW06032K00FKEAC, SamacSys_Parts:CRCW06032K00FKEAC
- added R19, R26, R27: CRCW060310K0JNEAC, SamacSys_Parts:CRCW060310K0JNEAC
- added R20, R21: CRCW080510R0JNEAHP, SamacSys_Parts:CRCW080510R0JNEAHP
- added R22: CRCW08055K90FKTA, SamacSys_Parts:CRCW08055K90FKTA
- added R25, R29: WSK2512R0250FEA, SamacSys_Parts:WSK2512R0250FEA
- added R30: CRCW12067K00JNTA, SamacSys_Parts:CRCW12067K00JNTA
- added R32: CRCW0603820RFKEA, SamacSys_Parts:CRCW0603820RFKEA
- added U2: SSM6N67NU,LF, SamacSys_Parts:SSM6N67NU,LF
Connections:
- net !ALERT renamed !ALERT_0
- net !EN_1 renamed !EN_1_0
- net !EN_2 renamed !EN_2_0
- net ADCIN_1 renamed ADCIN_1_0
- net ADCIN_2 renamed ADCIN_2_0
- net GPIO1 renamed GPIO1_0
- net GPIO2 renamed GPIO2_0
- net ON_SIGNAL renamed ON_SIGNAL_0
- net SCL renamed SCL_0
- net SDA renamed SDA_0
- new net !ALERT_1: IC2.!ALERT
- new net !EN_1_1: IC2.!EN1
- new net !EN_2_1: IC2.!EN2
- new net ADCIN_1_1: IC2.ADIN1
- new net ADCIN_2_1: IC2.ADIN2
- new net ARD0_1: IC2.ADR0
- new net ARD1_1: IC2.ADR1
- new net ARD2_1: IC2.ADR2
- new net FB1_JUNCTION_1: IC2.FB1, R27.2, R28.2
- new net FB2_JUNCTION_1: IC2.FB2, R17.2, R18.1
- new net GATE1_1: IC2.GATE1, R20.2
- new net GATE2_1: IC2.GATE2, R21.2
- new net GATE_1_INPUT_1: R20.1, U2.5
- new net GATE_2_INPUT_1: R21.1, U2.2
- new net GPIO1_1: IC2.GPIO1, R26.1
- new net GPIO2_1: IC2.GPIO2, R19.1
- new net I_SENSE1_OUT_1: IC2.SENSE1-, R29.E1
- new net I_SENSE2_OUT_1: IC2.SENSE2-, R25.E1
- new net ON_SIGNAL_1: IC2.ON
- new net OV1_1: IC2.OV1, R31.2, R32.1
- new net OV2_1: IC2.OV2, R22.2, R24.1
- new net PIN_FET1_1: R29.I1, U2.4
- new net PIN_FET2_1: R25.I1, U2.1
- new net SCL_1: IC2.SCL
- new net SDA_1: IC2.SDA
- new net SETUP_1: C7.1, IC2.CONFIG, IC2.INTVCC
- new net SS_1: C9.1, IC2.SS
- new net TIMER_1: C8.1, IC2.TIMER
- new net UV1_1: C10.1, IC2.UV1, R30.2, R31.1
- new net UV2_1: C6.1, IC2.UV2, R22.1, R23.2
- new net VOUT_1_1: IC2.SOURCE1, R26.2, R27.1, U2.3
- new net VOUT_2_1: IC2.SOURCE2, R17.1, R19.2, U2.6
- new net VSENSE_1_1: IC2.VDD1, R29.E2
- new net VSENSE_2_1: IC2.VDD2, R25.E2
- net GND: now also C10.2, C6.2, C7.2, C8.2, C9.2, IC2.GND, IC2.GND1, R18.2, R24.2, R28.1, R32.2
- net VIN_12V: now also R29.I2, R30.1
- net VIN_3.3V_5V: now also R23.1, R25.I2

Commit message: Added ADM1177 and power reg with some pin headers
Parts:
- added C11, C12: CGA5L2C0G1H104J160AA, SamacSys_Parts:CGA5L2C0G1H104J160AA
- added C13, C14: CGA4J3X7R1H105K125AB, SamacSys_Parts:CGA4J3X7R1H105K125AB
- added C15, C16: CGA5L3X7R1H225K160AB, SamacSys_Parts:CGA5L3X7R1H225K160AB
- added IC3, IC4: ADM1177-2ARMZ-R7, SamacSys_Parts:ADM1177-2ARMZ-R7
- added IC5: MCP1792T-3302H_CB, SamacSys_Parts:MCP1792T-3302H_CB
- added J1, J10, J11, J12, J13, J14, J15, J16, J17, J18, J19, J2, J20, J3, J4, J5, J6, J7, J8, J9: JUMPERSNT-100-BK-T, SamacSys_Parts:JUMPERSNT-100-BK-T
- added R33, R34: WSK2512R0250FEA, SamacSys_Parts:WSK2512R0250FEA
- added R35, R36: CRCW06032K00FKEAC, SamacSys_Parts:CRCW06032K00FKEAC
- added U3: SSM6N67NU,LF, SamacSys_Parts:SSM6N67NU,LF
Connections:
- removed net ARD0_0: IC1.ADR0
- removed net ARD0_1: IC2.ADR0
- removed net ARD1_0: IC1.ADR1
- removed net ARD1_1: IC2.ADR1
- removed net ARD2_0: IC1.ADR2
- removed net ARD2_1: IC2.ADR2
- new net 3.3V_LOGIC: C16.1, IC5.VOUT, J10.IN1, J14.IN1, J15.IN1, J16.IN1, J18.IN1, J2.IN1, J20.IN1, J4.IN1, J8.IN1, J9.IN1
- new net ADR0_0: IC1.ADR0, J10.IN2, J5.IN2
- new net ADR0_1: IC2.ADR0, J11.IN2, J16.IN2
- new net ADR1_0: IC1.ADR1, J6.IN2, J9.IN2
- new net ADR1_1: IC2.ADR1, J12.IN2, J15.IN2
- new net ADR2_0: IC1.ADR2, J7.IN2, J8.IN2
- new net ADR2_1: IC2.ADR2, J13.IN2, J14.IN2
- new net ADR_0: IC3.ADR, J17.IN2, J18.IN2
- new net ADR_1: IC4.ADR, J19.IN2, J20.IN2
- new net GATE_2: IC3.GATE, R35.2
- new net GATE_3: IC4.GATE, R36.2
- new net GATE_CONNECT_0: R35.1, U3.2
- new net GATE_CONNECT_1: R36.1, U3.5
- new net GND1: J19.IN1
- new net I_SENSE0: IC3.SENSE, R33.E1
- new net I_SENSE1: IC4.SENSE, R34.E1
- new net N$10: C13.1, IC3.TIMER
- new net N$11: C14.1, IC4.TIMER
- new net N$12: C12.1, IC4.SS
- new net N$9: C11.1, IC3.SS
- new net ON_0: IC3.ON, J1.IN2, J2.IN2
- new net ON_1: IC4.ON, J3.IN2, J4.IN2
- new net SCL_2: IC3.SCL
- new net SCL_3: IC4.SCL
- new net SDA_2: IC3.SDA
- new net SDA_3: IC4.SDA
- new net VIN>5V: C15.1, IC5.VIN
- new net VIN_0: R33.I2, U3.1
- new net VIN_1: R34.I2, U3.4
- new net VOUT_3: U3.6
- new net VOUT_4: U3.3
- new net VOUT_FET_0: R33.I1
- new net VOUT_FET_1: R34.I1
- new net V_SENSE0: IC3.VCC, R33.E2
- new net V_SENSE1: IC4.VCC, R34.E2
- net GND: now also C11.2, C12.2, C13.2, C14.2, C15.2, C16.2, IC3.GND, IC4.GND, IC5.GND, J1.IN1, J11.IN1, J12.IN1, J13.IN1, J17.IN1, J3.IN1, J5.IN1, J6.IN1, J7.IN1
Other:
- note added: "Enable or disable IC Set addressing"
- note added: "Pins to swap between selecting high or low for addressing"

Commit message: Schematic is laid out, missing test points and connector, nearly ready for board layout
Parts:
- added IC6: 74HC4852BQ,115, SamacSys_Parts:74HC4852BQ,115
- added J21, J22, J23, J24, J25, J26, J27, J28, J29, J30, J31, J32: JUMPERSNT-100-BK-T, SamacSys_Parts:JUMPERSNT-100-BK-T
- added LED1, LED10, LED11, LED12, LED13, LED2, LED3, LED4, LED5, LED6, LED7, LED8, LED9: AA3021LSYSK_J3-TR, SamacSys_Parts:AA3021LSYSK_J3-TR
- added R37, R38, R39, R40, R41, R42, R56, R57, R58, R59, R60, R61, R62: CRCW0603820RFKEA, SamacSys_Parts:CRCW0603820RFKEA
- added R43, R44, R45, R46, R47, R48, R49, R50, R51, R52, R53, R54, R55: CRCW06032K00FKEAC, SamacSys_Parts:CRCW06032K00FKEAC
Connections:
- new net !ENABLE_MUX: IC6.!E, R51.1, R62.2
- new net LED_1: LED1.K, R37.1
- new net LED_10: LED10.K, R59.1
- new net LED_11: LED11.K, R60.1
- new net LED_12: LED12.K, R61.1
- new net LED_13: LED13.K, R62.1
- new net LED_2: LED2.K, R38.1
- new net LED_3: LED3.K, R39.1
- new net LED_4: LED4.K, R40.1
- new net LED_5: LED5.K, R41.1
- new net LED_6: LED6.K, R42.1
- new net LED_7: LED7.K, R56.1
- new net LED_8: LED8.K, R57.1
- new net LED_9: LED9.K, R58.1
- new net S0: IC6.S0, R48.1
- new net S1: IC6.S1, R49.1
- new net SCL_IN: IC6.2Z, R54.1, R56.2
- new net SDA_IN: IC6.1Z, R45.1, R59.2
- net !ALERT_0: now also R37.2
- net !ALERT_1: now also R40.2
- net !EN_1_0: now also J22.IN2, J26.IN2
- net !EN_1_1: now also J28.IN2, J32.IN2
- net !EN_2_0: now also J21.IN2, J25.IN2
- net !EN_2_1: now also J27.IN2, J31.IN2
- net 3.3V_LOGIC: now also IC6.VCC, J23.IN1, J25.IN1, J26.IN1, J29.IN1, J31.IN1, J32.IN1, LED1.A, LED10.A, LED11.A, LED12.A, LED13.A, LED2.A, LED3.A, LED4.A, LED5.A, LED6.A, LED7.A, LED8.A, LED9.A, R43.2, R44.2, R45.2, R46.2, R47.2, R48.2, R49.2, R50.2, R51.2, R52.2, R53.2, R54.2, R55.2
- net GND: now also IC6.GND, IC6.N.C., IC6.NC, J21.IN1, J22.IN1, J24.IN1, J27.IN1, J28.IN1, J30.IN1
- net ON_SIGNAL_0: now also J23.IN2, J24.IN2
- net ON_SIGNAL_1: now also J29.IN2, J30.IN2
- net SCL_0: now also IC6.2Y0, R38.2, R50.1
- net SCL_1: now also IC6.2Y1, R41.2, R52.1
- net SCL_2: now also IC6.2Y2, R55.1, R57.2
- net SCL_3: now also IC6.2Y3, R53.1, R60.2
- net SDA_0: now also IC6.1Y0, R39.2, R44.1
- net SDA_1: now also IC6.1Y1, R42.2, R46.1
- net SDA_2: now also IC6.1Y2, R47.1, R58.2
- net SDA_3: now also IC6.1Y3, R43.1, R61.2
Other:
- note added: "LED turns on when !Alert triggers can only sink 2-3mA With no error, pin stays high"
- note added: "LED turns on when I2C pins go low"
- note added: "LED turns on when I2C pins go low and checks if MUX is on"

Commit message: added some test points
Parts:
- added TP1, TP10, TP11, TP12, TP13, TP14, TP15, TP16, TP17, TP18, TP19, TP2, TP20, TP21, TP22, TP23, TP24, TP25, TP26, TP27, TP28, TP29, TP3, TP30, TP31, TP32, TP33, TP34, TP35, TP36, TP37, TP38, TP39, TP4, TP40, TP41, TP42, TP43, TP44, TP5, TP6, TP7, TP8, TP9: S1751-46R, SamacSys_Parts:S1751-46R
Connections:
- net !ALERT_0: now also TP3.1
- net !ALERT_1: now also TP17.1
- net ADCIN_1_0: now also TP1.1
- net ADCIN_1_1: now also TP15.1
- net ADCIN_2_0: now also TP6.1
- net ADCIN_2_1: now also TP20.1
- net GATE1: now also TP29.1
- net GATE1_1: now also TP31.1
- net GATE2: now also TP30.1
- net GATE2_1: now also TP32.1
- net GATE_2: now also TP35.1
- net GATE_3: now also TP39.1
- net GND: now also TP10.1, TP21.1, TP22.1, TP23.1, TP24.1, TP7.1, TP8.1, TP9.1
- net I_SENSE0: now also TP34.1
- net I_SENSE1: now also TP38.1
- net I_SENSE1_OUT: now also TP12.1
- net I_SENSE1_OUT_1: now also TP26.1
- net I_SENSE2_OUT: now also TP14.1
- net I_SENSE2_OUT_1: now also TP28.1
- net ON_0: now also TP36.1
- net ON_1: now also TP40.1
- net ON_SIGNAL_0: now also TP2.1
- net ON_SIGNAL_1: now also TP16.1
- net SCL_0: now also TP4.1
- net SCL_1: now also TP18.1
- net SCL_2: now also TP42.1
- net SCL_3: now also TP44.1
- net SDA_0: now also TP5.1
- net SDA_1: now also TP19.1
- net SDA_2: now also TP41.1
- net SDA_3: now also TP43.1
- net VSENSE_1: now also TP11.1
- net VSENSE_2: now also TP13.1, TP25.1
- net VSENSE_2_1: now also TP27.1
- net V_SENSE0: now also TP33.1
- net V_SENSE1: now also TP37.1

Commit message: Schematics have been finsihed, now moving into layout
Parts:
- added JP1: (no value), pinhead:PINHD-1X6
- added JP2: (no value), pinhead:PINHD-1X7
- added JP3: (no value), pinhead:PINHD-1X4
- added JP4: (no value), pinhead:PINHD-1X5
- added TP45, TP46, TP47, TP48, TP49, TP50, TP51, TP52, TP53, TP54: S1751-46R, SamacSys_Parts:S1751-46R
Connections:
- net !ALERT_0: now also JP2.2
- net !ALERT_1: now also JP2.1
- net !ENABLE_MUX: now also JP2.3
- net ADCIN_1_0: now also JP3.4
- net ADCIN_1_1: now also JP3.2
- net ADCIN_2_0: now also JP3.3
- net ADCIN_2_1: now also JP3.1
- net GATE_1_INPUT: now also TP50.1
- net GATE_1_INPUT_1: now also TP52.1
- net GATE_2_INPUT: now also TP49.1
- net GATE_2_INPUT_1: now also TP51.1
- net GATE_CONNECT_0: now also TP54.1
- net GATE_CONNECT_1: now also TP53.1
- net S0: now also JP2.7
- net S1: now also JP2.6
- net SCL_IN: now also JP2.4
- net SDA_IN: now also JP2.5
- net VIN>5V: now also JP4.5
- net VIN_0: now also JP4.4; no longer U3.1
- net VIN_1: now also JP4.3; no longer U3.4
- net VIN_12V: now also JP4.1
- net VIN_3.3V_5V: now also JP4.2
- net VOUT_1: now also JP1.4, TP45.1
- net VOUT_1_1: now also JP1.2, TP47.1
- net VOUT_2: now also JP1.3, TP46.1
- net VOUT_2_1: now also JP1.1, TP48.1
- net VOUT_3: now also JP1.6
- net VOUT_4: now also JP1.5
- net VOUT_FET_0: now also U3.1
- net VOUT_FET_1: now also U3.4
Other:
- note added: "I2C mux"

Commit message: ~60% through layout
Parts:
- added C17: CGA5L2C0G1H104J160AA, SamacSys_Parts:CGA5L2C0G1H104J160AA
Connections:
- net 3.3V_LOGIC: now also C17.2, R50.1; no longer R50.2
- net GND: now also C17.1
- net SCL_0: now also R50.2; no longer R50.1
- net SDA_0: now also R46.1; no longer R44.1
- net SDA_1: now also R44.1; no longer R46.1
- net SDA_2: now also R43.1; no longer R47.1
- net SDA_3: now also R47.1; no longer R43.1
- net VSENSE_1_1: now also TP25.1
- net VSENSE_2: no longer TP25.1
Other:
- moved on the sheet: R43, R44, R46, R47, R50

Commit message: No real changes made yet, moving between projects
Parts:
- removed U1, U2: SSM6N67NU,LF, SamacSys_Parts:SSM6N67NU,LF
- added M1, M2, M3, M4: NTLUS4C12NTAG, SamacSys_Parts:NTLUS4C12NTAG
Connections:
- net GATE_1_INPUT: now also M1.G; no longer U1.5
- net GATE_1_INPUT_1: now also M3.G; no longer U2.5
- net GATE_2_INPUT: now also M2.G; no longer U1.2
- net GATE_2_INPUT_1: now also M4.G; no longer U2.2
- net PIN_FET1: now also M1.D; no longer U1.4
- net PIN_FET1_1: now also M3.D; no longer U2.4
- net PIN_FET2: now also M2.D; no longer U1.1
- net PIN_FET2_1: now also M4.D; no longer U2.1
- net VOUT_1: now also M1.S; no longer U1.3
- net VOUT_1_1: now also M3.S; no longer U2.3
- net VOUT_2: now also M2.S; no longer U1.6
- net VOUT_2_1: now also M4.S; no longer U2.6
Other:
- moved on the sheet: R20, R21, R4, R5

Commit message: Close to finsihing
Parts:
- removed J1, J10, J11, J12, J13, J14, J15, J16, J17, J18, J19, J2, J20, J21, J22, J23, J24, J25, J26, J27, J28, J29, J3, J30, J31, J32, J4, J5, J6, J7, J8, J9: JUMPERSNT-100-BK-T, SamacSys_Parts:JUMPERSNT-100-BK-T
- removed JP2: (no value), pinhead:PINHD-1X7
- removed U3: SSM6N67NU,LF, SamacSys_Parts:SSM6N67NU,LF
- added JP10, JP11, JP12, JP13, JP14, JP15, JP16, JP17, JP18, JP19, JP20, JP5, JP6, JP7, JP8, JP9: (no value), pinhead:PINHD-1X3
- added JP21: (no value), pinhead:PINHD-1X2
- added JP22: (no value), pinhead:PINHD-1X5
- added LED14, LED15: AA3021LSYSK_J3-TR, SamacSys_Parts:AA3021LSYSK_J3-TR
- added M5, M6: NTLUS4C12NTAG, SamacSys_Parts:NTLUS4C12NTAG
- added R63, R64: CRCW0603820RFKEA, SamacSys_Parts:CRCW0603820RFKEA
Connections:
- removed net GND1: J19.IN1
- new net LED_14: LED14.K, R63.1
- new net LED_15: LED15.K, R64.1
- net !ALERT_0: now also JP21.1; no longer JP2.2
- net !ALERT_1: now also JP21.2; no longer JP2.1
- net !ENABLE_MUX: now also JP22.5; no longer JP2.3
- net !EN_1_0: now also JP11.2; no longer J22.IN2, J26.IN2
- net !EN_1_1: now also JP14.2; no longer J28.IN2, J32.IN2
- net !EN_2_0: now also JP12.2; no longer J21.IN2, J25.IN2
- net !EN_2_1: now also JP15.2; no longer J27.IN2, J31.IN2
- net 3.3V_LOGIC: now also JP10.1, JP11.1, JP12.1, JP13.1, JP14.1, JP15.1, JP16.1, JP17.1, JP18.1, JP19.1, JP20.1, JP5.1, JP6.1, JP7.1, JP8.1, JP9.1, LED14.A, LED15.A; no longer J10.IN1, J14.IN1, J15.IN1, J16.IN1, J18.IN1, J2.IN1, J20.IN1, J23.IN1, J25.IN1, J26.IN1, J29.IN1, J31.IN1, J32.IN1, J4.IN1, J8.IN1, J9.IN1
- net ADR0_0: now also JP5.2; no longer J10.IN2, J5.IN2
- net ADR0_1: now also JP8.2; no longer J11.IN2, J16.IN2
- net ADR1_0: now also JP6.2; no longer J6.IN2, J9.IN2
- net ADR1_1: now also JP9.2; no longer J12.IN2, J15.IN2
- net ADR2_0: now also JP7.2; no longer J7.IN2, J8.IN2
- net ADR2_1: now also JP10.2; no longer J13.IN2, J14.IN2
- net ADR_0: now also JP18.2; no longer J17.IN2, J18.IN2
- net ADR_1: now also JP20.2; no longer J19.IN2, J20.IN2
- net GATE_CONNECT_0: now also M5.G; no longer U3.2
- net GATE_CONNECT_1: now also M6.G; no longer U3.5
- net GND: now also JP10.3, JP11.3, JP12.3, JP13.3, JP14.3, JP15.3, JP16.3, JP17.3, JP18.3, JP19.3, JP20.3, JP5.3, JP6.3, JP7.3, JP8.3, JP9.3; no longer J1.IN1, J11.IN1, J12.IN1, J13.IN1, J17.IN1, J21.IN1, J22.IN1, J24.IN1, J27.IN1, J28.IN1, J3.IN1, J30.IN1, J5.IN1, J6.IN1, J7.IN1
- net ON_0: now also JP17.2; no longer J1.IN2, J2.IN2
- net ON_1: now also JP19.2; no longer J3.IN2, J4.IN2
- net ON_SIGNAL_0: now also JP13.2; no longer J23.IN2, J24.IN2
- net ON_SIGNAL_1: now also JP16.2; no longer J29.IN2, J30.IN2
- net S0: now also JP22.1, R63.2; no longer JP2.7
- net S1: now also JP22.2, R64.2; no longer JP2.6
- net SCL_IN: now also JP22.4; no longer JP2.4
- net SDA_IN: now also JP22.3; no longer JP2.5
- net VOUT_3: now also M5.S; no longer U3.6
- net VOUT_4: now also M6.S; no longer U3.3
- net VOUT_FET_0: now also M5.D; no longer U3.1
- net VOUT_FET_1: now also M6.D; no longer U3.4
Other:
- note added: "LED turns on when S0 or S1 lines go low"
- moved on the sheet: LED1, LED2, LED3, LED4, LED5, LED6, M3, R20, R35, R36, R37, R38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
