File: FAST_DEPLOY_E_FUSE.brd (EAGLE design)
At the start: 160 x 100 mm, 182 parts, among them IC1 LTC4222CUH#PBF, IC2 LTC4222CUH#PBF, IC3 ADM1177-2ARMZ-R7, IC4 ADM1177-2ARMZ-R7, IC5 MCP1792T-3302H_CB, IC6 74HC4852BQ,115, M1 NTLUS4C12NTAG, M2 NTLUS4C12NTAG, M3 NTLUS4C12NTAG, M4 NTLUS4C12NTAG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

Commit message: Close to finsihing
Parts:
- removed JP2: (no value), pinhead:1X07
- added JP21: (no value), pinhead:1X02
- added JP22: (no value), pinhead:1X05
- moved TP10 179.4 mm to (97.0, 45.9), turned to 90 degrees
- moved TP7 178.5 mm to (97.0, 76.4), turned to 90 degrees
- moved TP9 177.9 mm to (97.0, 56.1), turned to 90 degrees
- moved TP8 177.6 mm to (97.0, 66.2), turned to 90 degrees
- moved TP24 173.0 mm to (92.4, 46.1), turned to 90 degrees
- moved TP21 172.0 mm to (92.4, 76.5), turned to 90 degrees
- moved TP23 171.5 mm to (92.4, 56.2), turned to 90 degrees
- moved TP22 171.2 mm to (92.4, 66.4), turned to 90 degrees
- moved R40 92.6 mm to (39.3, 59.4), turned to 180 degrees
- moved LED4 91.2 mm to (39.2, 54.9), turned to 270 degrees
- moved TP41 87.7 mm to (74.3, 40.0)
- moved TP43 87.6 mm to (74.3, 36.3)
- moved TP42 86.0 mm to (59.1, 38.2)
- moved TP44 85.4 mm to (59.0, 33.9)
- moved TP4 80.0 mm to (80.9, 40.0)
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Connections:
- net !ALERT_0: now also JP21.1; no longer JP2.2
- net !ALERT_1: now also JP21.2; no longer JP2.1
- net !ENABLE_MUX: now also JP22.5; no longer JP2.3
- net S0: now also JP22.1; no longer JP2.7
- net S1: now also JP22.2; no longer JP2.6
- net SCL_IN: now also JP22.4; no longer JP2.4
- net SDA_IN: now also JP22.3; no longer JP2.5
Routing:
- net !ALERT_1: track 0.00 -> 84.7 mm, vias 0 -> 4
- net !ALERT_0: track 0.00 -> 47.0 mm, vias 0 -> 4
- net SCL_1: track 9.71 -> 40.5 mm, vias 1 -> 3
- net SDA_IN: track 8.67 -> 37.5 mm, vias 1 -> 2
- net S0: track 8.91 -> 36.4 mm, vias 1 -> 2
- net SCL_0: track 12.8 -> 39.9 mm, vias 1 -> 3
- net !ENABLE_MUX: track 10.9 -> 36.6 mm, vias 1 -> 3
- net SCL_IN: track 9.01 -> 33.0 mm
- net S1: track 11.6 -> 35.5 mm, vias 1 -> 2
- net SDA_0: track 7.90 -> 28.9 mm, vias 1 -> 3
- net SCL_2: track 10.1 -> 30.9 mm, vias 1 -> 3
- net SDA_2: track 13.0 -> 30.7 mm, vias 1 -> 2
- net SCL_3: track 9.07 -> 26.2 mm, vias 1 -> 3
- net SDA_3: track 7.58 -> 22.7 mm, vias 1 -> 3
- net SDA_1: track 9.72 -> 23.6 mm, vias 1 -> 3
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
Commit message: Needs final labeling touch ups
Parts:
- added TP55, TP56, TP57, TP58, TP59, TP60, TP61, TP62: S1751-46R, SamacSys_Parts:S175146R
- moved TP10 86.7 mm to (10.4, 50.3)
- moved TP23 86.3 mm to (7.37, 41.9)
- moved TP21 83.4 mm to (9.04, 78.8)
- moved TP22 61.0 mm to (33.4, 50.8)
- moved TP9 48.4 mm to (51.4, 39.9)
- moved TP24 41.3 mm to (51.3, 48.6)
- moved TP7 34.6 mm to (63.0, 83.1)
- moved TP8 34.5 mm to (63.0, 60.2)
- moved R1 0.40 mm to (20.8, 28.9)
- moved R2 0.40 mm to (20.8, 28.9)
Connections:
- net GND: now also TP55.1, TP56.1, TP57.1, TP58.1, TP59.1, TP60.1, TP61.1, TP62.1
Routing:
- net 3.3V_LOGIC: track 134.2 -> 466.5 mm, vias 3 -> 8
- net SDA_1: track 23.6 -> 108.0 mm, vias 3 -> 5
- net SCL_1: track 40.5 -> 119.3 mm, vias 3 -> 5
- net SCL_0: track 39.9 -> 100.5 mm, vias 3 -> 7
- net SDA_0: track 28.9 -> 80.5 mm, vias 3 -> 4
- net SCL_3: track 26.2 -> 74.7 mm, vias 3 -> 4
- net SDA_3: track 22.7 -> 62.8 mm, vias 3 -> 4
- net SCL_2: track 30.9 -> 55.6 mm, vias 3 -> 4
- net GND: track 0.00 -> 24.3 mm, vias 0 -> 145
- net SDA_2: track 30.7 -> 48.9 mm, vias 2 -> 3
- net VOUT_2: track 59.3 -> 66.5 mm, vias 2 -> 3
- net V_SENSE1: track 8.08 -> 12.5 mm
- net GATE_3: track 20.9 -> 24.7 mm
- net VOUT_FET_1: track 4.28 -> 7.82 mm
- net GATE_CONNECT_1: track 1.54 -> 4.57 mm
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- added copper zone on layer 1, net GND
- added copper zone on layer 16, net GND
Other:
- board size 160 x 100 mm -> 102.1 x 92.8 mm
