File: LTC4222.sch (EAGLE design)
At the start: 51 parts, among them IC1 67997-100HLF, IC2 LTC4222, J1 PMV15ENEAR, J2 PMV15ENEAR, P1 S1751-46R, P10 S1751-46R, P11 S1751-46R, P12 S1751-46R, P13 S1751-46R, P14 S1751-46R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

Commit message: Test message V2
Parts:
- removed JP4: (no value), pinhead:PINHD-1X9
- removed P10, P9: S1751-46R, Baja_Parts_Lib:S1751-46R
- removed U$3, U$4: 74HC1G86GW-Q100H, Baja_Parts_Lib:74HC1G86GW-Q100H
- removed U$5: SN74HC74QPWRQ1, Baja_Parts_Lib:SN74HC74QPWRQ1
Connections:
- removed net A_OR_GATE#2: JP4.7, U$4.A
- removed net B_OR_GATE#1: JP4.5, U$3.B
- removed net N$1 (its old number): U$3.Y, U$5.1D
- removed net N$3: IC2.EN2, P10.1, U$4.B, U$5.2Q
- removed net N$4: IC2.EN1, P9.1, U$3.A, U$5.1Q
- removed net N$5: U$4.Y, U$5.2D
- removed net VCC_DFF: JP4.9, U$5.VCC
- removed net VCC_OR_GATE#1: JP4.6, U$3.VCC
- removed net VCC_OR_GATE#2: JP4.8, U$4.VCC
- net ADIN1: no longer JP4.1
- net ADIN2: no longer JP4.4
- net ALERT: no longer JP4.3
- net GND: no longer U$3.GND, U$4.GND, U$5.GND
- net ON: no longer JP4.2
Other:
- moved on the sheet: R5

Commit message: Small alterations
Connections:
- net N$1: now also J1.G
Other:
- moved on the sheet: R5
Changed lines of the file:
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@@
 <part name="SUPPLY2" library="supply2" library_urn="urn:adsk.eagle:library:372" deviceset="GND" device=""/>
 <part name="J1" library="Baja_Parts_Lib" deviceset="PMV15ENEAR" device="" package3d_urn="urn:adsk.eagle:package:31668685/1"/>
-<part name="R5" library="Baja_Parts_Lib" deviceset="TNPW060310R0BEEN" device="" package3d_urn="urn:adsk.eagle:package:31668595/1"/>
 <part name="R6" library="Baja_Parts_Lib" deviceset="TNPW040210K2BEED" device="" package3d_urn="urn:adsk.eagle:package:31668646/1"/>
 <part name="R7" library="Baja_Parts_Lib" deviceset="TNPW06033K57BEEA" device="" package3d_urn="urn:adsk.eagle:package:31668595/1"/>
@@
 <part name="JP2" library="pinhead" library_urn="urn:adsk.eagle:library:325" deviceset="PINHD-1X1" device="" package3d_urn="urn:adsk.eagle:package:22485/2"/>
 <part name="JP3" library="pinhead" library_urn="urn:adsk.eagle:library:325" deviceset="PINHD-1X1" device="" package3d_urn="urn:adsk.eagle:package:22485/2"/>
+<part name="R5" library="Baja_Parts_Lib" deviceset="TNPW060310R0BEEN" device="" package3d_urn="urn:adsk.eagle:package:31668595/1"/>
 </parts>
 <sheets>
@@
 <attribute name="VALUE" x="-119.38" y="187.96" size="1.778" layer="96" rot="MR180"/>
 </instance>
-<instance part="R5" gate="G$1" x="-119.38" y="144.78" smashed="yes" rot="R90">
-<attribute name="NAME" x="-116.84" y="144.78" size="1.778" layer="95" rot="R90"/>
-<attribute name="VALUE" x="-114.3" y="142.24" size="1.778" layer="96" rot="R90"/>
-</instance>
 <instance part="R6" gate="G$1" x="-91.44" y="132.08" smashed="yes" rot="R90">
 <attribute name="NAME" x="-91.44" y="132.08" size="1.778" layer="95" rot="R90"/>
@@
 <attribute name="NAME" x="-191.77" y="-48.895" size="1.778" layer="95" rot="R180"/>
 <attribute name="VALUE" x="-191.77" y="-40.64" size="1.778" layer="96" rot="R180"/>
+</instance>
+<instance part="R5" gate="G$1" x="-119.38" y="142.24" smashed="yes" rot="R90">
+<attribute name="NAME" x="-121.92" y="147.32" size="1.778" layer="95" rot="R90"/>
+<attribute name="VALUE" x="-114.3" y="142.24" size="1.778" layer="96" rot="R90"/>
 </instance>
 </instances>
@@
 <net name="N$11" class="0">
 <segment>
-<pinref part="R5" gate="G$1" pin="P$1"/>
-<wire x1="-119.38" y1="144.78" x2="-119.38" y2="139.7" width="0.1524" layer="91"/>
 <pinref part="IC2" gate="G$1" pin="GATE1"/>
 <pinref part="P5" gate="G$1" pin="1"/>
 <wire x1="-119.38" y1="139.7" x2="-119.38" y2="93.98" width="0.1524" layer="91"/>
-<junction x="-119.38" y="139.7"/>
+<pinref part="R5" gate="G$1" pin="P$1"/>
+<wire x1="-119.38" y1="139.7" x2="-119.38" y2="142.24" width="0.1524" layer="91"/>
 </segment>
 </net>
@@
 <segment>
 <pinref part="R5" gate="G$1" pin="P$2"/>
-<wire x1="-119.38" y1="167.64" x2="-109.22" y2="170.18" width="0.1524" layer="91"/>
-</segment>
-</net>
+<wire x1="-119.38" y1="165.1" x2="-109.22" y2="165.1" width="0.1524" layer="91"/>
+<wire x1="-109.22" y1="165.1" x2="-109.22" y2="170.177" width="0.1524" layer="91"/>
+<pinref part="J1" gate="G$1" pin="G"/>
+<wire x1="-109.22" y1="170.177" x2="-109.22" y2="170.18" width="0.1524" layer="91"/>
+<junction x="-109.22" y="170.177"/>
+</segment>
+</net>

Commit message: PCB Design V1
Connections:
- removed net N$17: C3.1, C4.1
- removed net N$28: R15.P$2
- net GND: now also C3.1, C4.1, R15.P$2
Changed lines of the file:
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@@
 <part name="JP3" library="pinhead" library_urn="urn:adsk.eagle:library:325" deviceset="PINHD-1X1" device="" package3d_urn="urn:adsk.eagle:package:22485/2"/>
 <part name="R5" library="Baja_Parts_Lib" deviceset="TNPW060310R0BEEN" device="" package3d_urn="urn:adsk.eagle:package:31668595/1"/>
+<part name="SUPPLY6" library="supply2" library_urn="urn:adsk.eagle:library:372" deviceset="GND" device=""/>
 </parts>
 <sheets>
@@
 <attribute name="VALUE" x="-76.2" y="-40.64" size="1.778" layer="96" rot="R90"/>
 </instance>
-<instance part="SUPPLY10" gate="GND" x="-88.9" y="20.32" smashed="yes">
-<attribute name="VALUE" x="-90.805" y="17.145" size="1.778" layer="96"/>
+<instance part="SUPPLY10" gate="GND" x="-91.44" y="22.86" smashed="yes">
+<attribute name="VALUE" x="-93.345" y="19.685" size="1.778" layer="96"/>
 </instance>
 <instance part="IC2" gate="G$1" x="-147.32" y="38.1" smashed="yes">
@@
 <attribute name="NAME" x="-121.92" y="147.32" size="1.778" layer="95" rot="R90"/>
 <attribute name="VALUE" x="-114.3" y="142.24" size="1.778" layer="96" rot="R90"/>
+</instance>
+<instance part="SUPPLY6" gate="GND" x="-220.98" y="71.12" smashed="yes">
+<attribute name="VALUE" x="-222.885" y="65.405" size="1.778" layer="96"/>
 </instance>
 </instances>
@@
 <pinref part="SUPPLY11" gate="GND" pin="GND"/>
 <wire x1="-124.46" y1="60.96" x2="-124.46" y2="63.5" width="0.1524" layer="91"/>
+</segment>
+<segment>
+<pinref part="R15" gate="G$1" pin="P$2"/>
+<wire x1="-81.28" y1="27.94" x2="-81.28" y2="30.48" width="0.1524" layer="91"/>
+<pinref part="SUPPLY10" gate="GND" pin="GND"/>
+<wire x1="-81.28" y1="30.48" x2="-91.44" y2="30.48" width="0.1524" layer="91"/>
+<wire x1="-91.44" y1="30.48" x2="-91.44" y2="25.4" width="0.1524" layer="91"/>
+</segment>
+<segment>
+<pinref part="C3" gate="G$1" pin="1"/>
+<wire x1="-208.28" y1="81.28" x2="-213.36" y2="81.28" width="0.1524" layer="91"/>
+<wire x1="-213.36" y1="81.28" x2="-213.36" y2="76.2" width="0.1524" layer="91"/>
+<pinref part="C4" gate="G$1" pin="1"/>
+<wire x1="-213.36" y1="76.2" x2="-213.36" y2="45.72" width="0.1524" layer="91"/>
+<wire x1="-213.36" y1="45.72" x2="-210.82" y2="45.72" width="0.1524" layer="91"/>
+<wire x1="-213.36" y1="76.2" x2="-218.44" y2="76.2" width="0.1524" layer="91"/>
+<pinref part="SUPPLY6" gate="GND" pin="GND"/>
+<wire x1="-218.44" y1="76.2" x2="-218.44" y2="73.66" width="0.1524" layer="91"/>
+<wire x1="-218.44" y1="73.66" x2="-220.98" y2="73.66" width="0.1524" layer="91"/>
 </segment>
 </net>
@@
 <wire x1="-152.4" y1="81.28" x2="-195.58" y2="81.28" width="0.1524" layer="91"/>
 <pinref part="IC2" gate="G$1" pin="SS"/>
-</segment>
-</net>
-<net name="N$17" class="0">
-<segment>
-<pinref part="C3" gate="G$1" pin="1"/>
-<wire x1="-208.28" y1="81.28" x2="-213.36" y2="81.28" width="0.1524" layer="91"/>
-<wire x1="-213.36" y1="81.28" x2="-213.36" y2="76.2" width="0.1524" layer="91"/>
-<pinref part="C4" gate="G$1" pin="1"/>
-<wire x1="-213.36" y1="76.2" x2="-213.36" y2="45.72" width="0.1524" layer="91"/>
-<wire x1="-213.36" y1="45.72" x2="-210.82" y2="45.72" width="0.1524" layer="91"/>
-<wire x1="-213.36" y1="76.2" x2="-218.44" y2="76.2" width="0.1524" layer="91"/>
 </segment>
 </net>
@@
 </segment>
 </net>
-<net name="N$28" class="0">
-<segment>
-<pinref part="R15" gate="G$1" pin="P$2"/>
-<wire x1="-81.28" y1="27.94" x2="-88.9" y2="27.94" width="0.1524" layer="91"/>
-<pinref part="SUPPLY10" gate="GND" pin="GND"/>
-<wire x1="-88.9" y1="22.86" x2="-88.9" y2="27.94" width="0.1524" layer="91"/>
-</segment>
-</net>

Commit message: PCB schematic V1.2
Parts:
- added JP4: (no value), pinhead:PINHD-1X8
Connections:
- new net N$3: IC2.EN1, JP4.1
- new net N$4: IC2.SCL, JP4.5
- new net N$5: IC2.SDA, JP4.6
- new net N$9: IC2.EN2, JP4.8
- net ADIN1: now also JP4.2
- net ADIN2: now also JP4.7
- net ALERT: now also JP4.4
- net ON: now also JP4.3
Changed lines of the file:
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@@
 <part name="R5" library="Baja_Parts_Lib" deviceset="TNPW060310R0BEEN" device="" package3d_urn="urn:adsk.eagle:package:31668595/1"/>
 <part name="SUPPLY6" library="supply2" library_urn="urn:adsk.eagle:library:372" deviceset="GND" device=""/>
+<part name="JP4" library="pinhead" library_urn="urn:adsk.eagle:library:325" deviceset="PINHD-1X8" device="" package3d_urn="urn:adsk.eagle:package:22409/2"/>
 </parts>
 <sheets>
@@
 <attribute name="VALUE" x="-222.885" y="65.405" size="1.778" layer="96"/>
 </instance>
+<instance part="JP4" gate="A" x="-53.34" y="63.5" smashed="yes">
+<attribute name="NAME" x="-59.69" y="76.835" size="1.778" layer="95"/>
+<attribute name="VALUE" x="-59.69" y="50.8" size="1.778" layer="96"/>
+</instance>
 </instances>
 <busses>
@@
 <segment>
 <pinref part="R15" gate="G$1" pin="P$2"/>
-<wire x1="-81.28" y1="27.94" x2="-81.28" y2="30.48" width="0.1524" layer="91"/>
 <pinref part="SUPPLY10" gate="GND" pin="GND"/>
-<wire x1="-81.28" y1="30.48" x2="-91.44" y2="30.48" width="0.1524" layer="91"/>
-<wire x1="-91.44" y1="30.48" x2="-91.44" y2="25.4" width="0.1524" layer="91"/>
+<wire x1="-81.28" y1="27.94" x2="-91.44" y2="27.94" width="0.1524" layer="91"/>
+<wire x1="-91.44" y1="27.94" x2="-91.44" y2="25.4" width="0.1524" layer="91"/>
 </segment>
 <segment>
@@
 <segment>
 <pinref part="IC2" gate="G$1" pin="ADIN2"/>
-<wire x1="-91.44" y1="50.8" x2="-83.82" y2="50.8" width="0.1524" layer="91"/>
-<label x="-81.28" y="50.8" size="1.778" layer="95"/>
+<wire x1="-91.44" y1="50.8" x2="-66.04" y2="50.8" width="0.1524" layer="91"/>
+<wire x1="-66.04" y1="50.8" x2="-66.04" y2="58.42" width="0.1524" layer="91"/>
+<pinref part="JP4" gate="A" pin="7"/>
+<wire x1="-66.04" y1="58.42" x2="-55.88" y2="58.42" width="0.1524" layer="91"/>
 </segment>
 </net>
@@
 <segment>
 <pinref part="IC2" gate="G$1" pin="ALERT"/>
-<wire x1="-91.44" y1="66.04" x2="-83.82" y2="66.04" width="0.1524" layer="91"/>
-<label x="-81.28" y="66.04" size="1.778" layer="95"/>
+<pinref part="JP4" gate="A" pin="4"/>
+<wire x1="-91.44" y1="66.04" x2="-55.88" y2="66.04" width="0.1524" layer="91"/>
 </segment>
 </net>
@@
 <segment>
 <pinref part="IC2" gate="G$1" pin="ON"/>
-<wire x1="-91.44" y1="71.12" x2="-83.82" y2="71.12" width="0.1524" layer="91"/>
-<label x="-81.28" y="71.12" size="1.778" layer="95"/>
+<wire x1="-91.44" y1="71.12" x2="-71.12" y2="71.12" width="0.1524" layer="91"/>
+<wire x1="-71.12" y1="71.12" x2="-71.12" y2="68.58" width="0.1524" layer="91"/>
+<pinref part="JP4" gate="A" pin="3"/>
+<wire x1="-71.12" y1="68.58" x2="-55.88" y2="68.58" width="0.1524" layer="91"/>
 </segment>
 </net>
@@
 <segment>
 <pinref part="IC2" gate="G$1" pin="ADIN1"/>
-<wire x1="-91.44" y1="76.2" x2="-83.82" y2="76.2" width="0.1524" layer="91"/>
-<label x="-81.28" y="76.2" size="1.778" layer="95"/>
+<wire x1="-91.44" y1="76.2" x2="-68.58" y2="76.2" width="0.1524" layer="91"/>
+<pinref part="JP4" gate="A" pin="2"/>
+<wire x1="-68.58" y1="76.2" x2="-68.58" y2="71.12" width="0.1524" layer="91"/>
+<wire x1="-68.58" y1="71.12" x2="-55.88" y2="71.12" width="0.1524" layer="91"/>
 </segment>
 </net>
@@
 </segment>
 </net>
+<net name="N$3" class="0">
+<segment>
+<pinref part="IC2" gate="G$1" pin="EN1"/>
+<wire x1="-91.44" y1="81.28" x2="-66.04" y2="81.28" width="0.1524" layer="91"/>
+<wire x1="-66.04" y1="81.28" x2="-66.04" y2="73.66" width="0.1524" layer="91"/>
+<pinref part="JP4" gate="A" pin="1"/>
+<wire x1="-66.04" y1="73.66" x2="-55.88" y2="73.66" width="0.1524" layer="91"/>
+</segment>
+</net>
+<net name="N$4" class="0">
+<segment>
+<pinref part="IC2" gate="G$1" pin="SCL"/>
+<wire x1="-91.44" y1="60.96" x2="-71.12" y2="60.96" width="0.1524" layer="91"/>
+<wire x1="-71.12" y1="60.96" x2="-71.12" y2="63.5" width="0.1524" layer="91"/>
+<pinref part="JP4" gate="A" pin="5"/>
+<wire x1="-71.12" y1="63.5" x2="-55.88" y2="63.5" width="0.1524" layer="91"/>
+</segment>
+</net>
+<net name="N$5" class="0">
+<segment>
+<pinref part="IC2" gate="G$1" pin="SDA"/>
+<wire x1="-91.44" y1="55.88" x2="-68.58" y2="55.88" width="0.1524" layer="91"/>
+<wire x1="-68.58" y1="55.88" x2="-68.58" y2="60.96" width="0.1524" layer="91"/>
+<pinref part="JP4" gate="A" pin="6"/>
+<wire x1="-68.58" y1="60.96" x2="-55.88" y2="60.96" width="0.1524" layer="91"/>
+</segment>
+</net>
+<net name="N$9" class="0">
+<segment>
+<pinref part="IC2" gate="G$1" pin="EN2"/>
+<wire x1="-91.44" y1="45.72" x2="-63.5" y2="45.72" width="0.1524" layer="91"/>
+<wire x1="-63.5" y1="45.72" x2="-63.5" y2="55.88" width="0.1524" layer="91"/>
+<pinref part="JP4" gate="A" pin="8"/>
+<wire x1="-63.5" y1="55.88" x2="-55.88" y2="55.88" width="0.1524" layer="91"/>
+</segment>
+</net>
