File: MasterPCB_transfer.brd (EAGLE design)
At the start: 443.2 x 345.1 mm, 909 parts, among them IC1 NCS21911SN2T1G, IC10 LDL1117S33R, IC11 LTC4222CUH#PBF, IC12 LTC4222CUH#PBF, IC13 LTC4222CUH#PBF, IC14 LTC4222CUH#PBF, IC15 LTC4222CUH#PBF, IC16 LTC4222CUH#PBF, IC17 LTC4222CUH#PBF, IC18 LTC4222CUH#PBF, IC19 LTC4222CUH#PBF, IC2 NCS21911SN2T1G, IC20 LTC4222CUH#PBF, IC21 LTC4222CUH#PBF, IC22 LTC4222CUH#PBF, IC23 LTC4222CUH#PBF, IC3 NCS21911SN2T1G, IC38 ADS8588HIPM, IC4 LTC4222CUH#PBF, IC5 LP38692SDX-5.0_NOPB, IC6 LP38692SDX-5.0_NOPB, IC7 LDL1117S33R, IC8 LDL1117S33R, IC9 LP38692SDX-5.0_NOPB, J1 SAMTEC-SMM-104-02-X-DJ, M1 NTLUS4C12NTAG, M10 NTLUS4C12NTAG, M11 NTLUS4C12NTAG, M12 NTLUS4C12NTAG, M13 NTLUS4C12NTAG, M14 NTLUS4C12NTAG, M15 NTLUS4C12NTAG, M16 NTLUS4C12NTAG, M17 NTLUS4C12NTAG, M18 NTLUS4C12NTAG, M19 NTLUS4C12NTAG, M2 NTLUS4C12NTAG, M20 NTLUS4C12NTAG, M21 NTLUS4C12NTAG, M22 NTLUS4C12NTAG, M23 NTLUS4C12NTAG, M24 NTLUS4C12NTAG, M25 NTLUS4C12NTAG, M26 NTLUS4C12NTAG, M27 NTLUS4C12NTAG, M28 NTLUS4C12NTAG, M3 NTLUS4C12NTAG, M4 NTLUS4C12NTAG, M5 NTLUS4C12NTAG, M6 NTLUS4C12NTAG, M7 NTLUS4C12NTAG, M8 NTLUS4C12NTAG, M9 NTLUS4C12NTAG

Commit message: Most features complete
Parts:
- added C169: GRM31C5C1E474JE01L, SamacSys_Parts:CAPC3216X180N
- added IC24, IC25, IC26, IC27, IC28, IC29, IC30: NCS21911SN2T1G, SamacSys_Parts:SOT95P275X110-5N
- added IC31: ADIS16500AMLZ, SamacSys_Parts:BGA100C127P10X10_1500X1500X608
- added IC32: LTC6820IUD#PBF, SamacSys_Parts:QFN50P300X300X80-17N
- added J2: SAMTEC-CLP-106-02-X-DJ, SamacSys_Parts:SAMTEC-CLP-106-02-X-D
- added J3: SSM-109-L-SV, SamacSys_Parts:SAMTEC_SSM-109-L-SV
- added R472, R481, R490: GMR100HTCFAR100, SamacSys_Parts:RESC6432X55N
- added R473, R474, R475, R476, R482, R483, R484, R485, R491, R492, R493, R494: RC0402JR-133K3L, SamacSys_Parts:RESC1005X40N
- added R477, R478, R486, R487, R495, R496: MCS04020C1001FE000, SamacSys_Parts:RESC1005X37N
- added R479: CRCW040212K0FKTD, SamacSys_Parts:RESC1005X40N
- added R480: CR0402-FX-1022GLF, SamacSys_Parts:RESC1005X40N
- added R488, R489, R497, R498: RC0402JR-1015KL, SamacSys_Parts:RESC1005X40N
- added R499, R500, R501, R502, R503, R506, R508: ERJ-2RKF2002X, SamacSys_Parts:ERJ2R_(0402)
- added R504, R505, R507, R509: MCS0402MD1002DE000, SamacSys_Parts:RESC1005X37N
- added U$2, U$3, U$4: PTS120601B1K00P100, SamacSys_Parts:RESC3016X70N
Connections:
- new net !IMU_CS: IC31.G3
- new net !IMU_RST: IC31.F3
- new net 14V_BUS_FROM_CONNECTOR: J2.1, R472.1, R473.1
- new net 14V_RAIL_VO: IC24.1, R480.2
- new net 3.3V_NC: J3.01
- new net 5V_BUS_FROM_CONNECTOR: J2.5, R490.1, R491.1
- new net 5V_RAIL_VO: IC26.1, R498.2
- new net 6.5V_BUS_FROM_CONNECTOR: J2.3, R481.1, R482.1
- new net 6.5V_RAIL_VO: IC25.1, R489.2
- new net FAULT1: J2.7
- new net FAULT2: J2.9
- new net FAULT3: J2.11
- new net FB+_1: IC24.3, R477.1, R479.1
- new net FB+_2: IC25.3, R486.1, R488.1
- new net FB+_3: IC26.3, R495.1, R497.1
- new net FB-_1: IC24.4, R478.1, R480.1
- new net FB-_2: IC25.4, R487.1, R489.1
- new net FB-_3: IC26.4, R496.1, R498.1
- new net FIX_NC: J3.04
- new net GPS_EN: J3.02
- new net GPS_RX: J3.06
- new net GPS_TX: J3.05
- new net IMU_DIN: IC31.G6
- new net IMU_DOUT: IC31.H3
- new net IMU_DR: IC31.J6
- new net IMU_SCLK: IC31.H6
- new net IMU_SYNC: IC31.J3
- new net N$347: IC32.2
- new net N$349: IC32.3
- new net N$351: IC32.4
- new net N$352: IC32.5, IC32.6, IC32.7, IC32.8
- new net POWER_TEMP1: J2.8
- new net POWER_TEMP2: J2.10
- new net POWER_TEMP3: J2.12
- new net PPS_NC: J3.09
- new net TEMP1: IC27.3, R471.2, U$1.1
- new net TEMP1_OUT: IC27.1, R503.2
- new net TEMP2: IC28.3, R499.2, U$2.1
- new net TEMP2_OUT: IC28.1, R502.2
- new net TEMP3: IC29.3, R500.2, U$3.1
- new net TEMP3_OUT: IC29.1, R506.2
- new net TEMP4: IC30.3, R501.2, U$4.1
- new net TEMP4_OUT: IC30.1, R508.2
- new net TEMP_FB_1: IC27.4, R503.1, R504.1
- new net TEMP_FB_2: IC28.4, R502.1, R505.1
- new net TEMP_FB_3: IC29.4, R506.1, R507.1
- new net TEMP_FB_4: IC30.4, R508.1, R509.1
- new net V+_1: R473.2, R474.1, R477.2
- new net V+_2: R482.2, R483.1, R486.2
- new net V+_3: R491.2, R492.1, R495.2
- new net V-_1: R475.2, R476.1, R478.2
- new net V-_2: R484.2, R485.1, R487.2
- new net V-_3: R493.2, R494.1, R496.2
- new net VBAT_NC: J3.03
- net 13.5V_BUS: now also IC24.5, IC25.5, IC26.5, IC27.5, IC28.5, IC29.5, IC30.5, R472.2, R475.1
- net 3.3V_SENSORS: now also C169.1, IC31.C7, IC31.D6, IC31.E3, IC31.G1, IC31.H1, IC31.J4, IC31.J5, IC31.K6, J3.08
- net 5V_BUS: now also R490.2, R493.1
- net 5V_ON_BOARD: now also R499.1, R500.1, R501.1
- net 6.5V_BUS: now also R481.2, R484.1
- net DIFF10_N: now also Z6.4
- net DIFF10_P: no longer Z6.4
- net DIFF11_N: now also Z7.4
- net DIFF11_P: no longer Z7.4
- net DIFF12_N: now also Z8.4
- net DIFF12_P: no longer Z8.4
- net DIFF13_N: now also Z17.4
- net DIFF13_P: no longer Z17.4
- net DIFF14_N: now also Z18.4
- net DIFF14_P: no longer Z18.4
- net DIFF15_N: now also Z19.4
- net DIFF15_P: no longer Z19.4
- net DIFF16_N: now also Z20.4
- net DIFF16_P: no longer Z20.4
- net DIFF1_N: now also Z1.4
- net DIFF1_P: no longer Z1.4
- net DIFF2_N: now also Z2.4
- net DIFF2_P: no longer Z2.4
- net DIFF3_N: now also Z3.4
- net DIFF3_P: no longer Z3.4
- net DIFF4_N: now also Z4.4
- net DIFF4_P: no longer Z4.4
- net DIFF5_N: now also Z21.4
- net DIFF5_P: no longer Z21.4
- net DIFF6_N: now also Z22.4
- net DIFF6_P: no longer Z22.4
- net DIFF7_N: now also Z23.4
- net DIFF7_P: no longer Z23.4
- net DIFF8_N: now also Z24.4
- net DIFF8_P: no longer Z24.4
- net DIFF9_N: now also Z5.4
- net DIFF9_P: no longer Z5.4
- net GND: now also C169.2, IC24.2, IC25.2, IC26.2, IC27.2, IC28.2, IC29.2, IC30.2, IC31.A1, IC31.A2, IC31.A3, IC31.A4, IC31.A5, IC31.A6, IC31.A7, IC31.A8, IC31.B3, IC31.B4, IC31.B5, IC31.B6, IC31.C2, IC31.C6, IC31.D3, IC31.E2, IC31.E6, IC31.E7, IC31.F1, IC31.F5, IC31.F6, IC31.F8, IC31.G2, IC31.G7, IC31.H8, IC31.J2, IC31.J7, IC31.K1, IC31.K3, IC31.K8, J2.2, J2.4, J2.6, J3.07, R474.2, R476.2, R479.2, R483.2, R485.2, R488.2, R492.2, R494.2, R497.2, R504.2, R505.2, R507.2, R509.2, U$2.2, U$3.2, U$4.2
- net N$345: now also IC32.1; no longer R471.2, U$1.1

Commit message: Working on QSPI
Parts:
- added C170: GRM31C5C1E474JE01L, SamacSys_Parts:CAPC3216X180N
- added C171, C172: 06035C270JAT2A, SamacSys_Parts:CAPC1608X90N
- added IC33: CBTL01023GM,115, SamacSys_Parts:QFN50P200X155X50-10N
- added R510: CPF0402B1K21E1, SamacSys_Parts:RESC1005X35N
- added R511: ERA-2AEB7870X, SamacSys_Parts:ERA2AED122X
- added R512: TNPW0402100RBYEP, SamacSys_Parts:RESC1005X40N
- added R513, R514, R515, R516, R517, R518, R519, R520, R521: CRG0402ZR, SamacSys_Parts:RESC1005X40N
- added T1: 782482_33VC, SamacSys_Parts:DIP1016W60P254L914H635Q6N
Connections:
- net N$345 renamed ISO_MOSI
- net N$347 renamed ISO_MISO
- net N$349 renamed ISO_SPI_SCLK
- net N$351 renamed !ISO_CS
- removed net N$352: IC32.5, IC32.6, IC32.7, IC32.8
- new net !THERMOCOUPLE_CS: R519.2
- new net 40G_GPIO: Z15.3
- new net C1: R517.1, R520.1, Z16.5
- new net C2: R518.1, R521.1, Z16.4
- new net C3: R519.1, Z16.3
- new net IBAIS: IC32.15, R510.1
- new net ICMP: IC32.14, R510.2, R511.1
- new net IM_INPUT: IC32.9, R512.2, T1.3
- new net IM_OUT1: IC33.8, Z15.4
- new net IM_OUT2: IC33.6, R518.2
- new net IM_OUTPUT: R514.2, R516.1, R516.2, T1.4
- new net IP_INPUT: IC32.10, R512.1, T1.1
- new net IP_OUT1: IC33.9, R515.1, R517.2, Z15.5
- new net IP_OUT2: IC33.7
- new net IP_OUTPUT: R513.2, R515.2, T1.6
- new net ISO_SPI_CH_SEL: IC33.4
- new net ISO_SPI_HIGH_Z_SWITCH: IC33.1
- new net ISO_SPI_SLOW: IC32.12
- new net N$345: IC33.2, R513.1
- new net N$347: IC33.3, R514.1
- new net N$356: C171.1, T1.2
- new net N$360: C172.1, T1.5
- new net THERMOCOUPLE_MISO: R521.2
- new net THERMOCOUPLE_SCLK: R520.2
- net 13.5V_BUS: now also Z15.2, Z16.2
- net 3.3V_SENSORS: now also C170.1, IC32.11, IC32.16, IC32.5, IC32.6, IC32.7, IC32.8, IC33.5
- net ADIN1_: no longer Z15.3
- net ADIN2_: no longer Z16.3
- net DIFF1_P: no longer Z15.4, Z15.5, Z16.4, Z16.5
- net GND: now also C170.2, C171.2, C172.2, IC32.13, IC32.17, IC33.10, R511.2
- net SOURCE1_10: no longer Z15.2
- net SOURCE2_10: no longer Z16.2

Commit message: Last wiring left to do then ready for board layout
Parts:
- removed R158, R159, R160, R161, R162, R163, R201, R203, R205, R207, R209, R211, SG_BUSY_2: RCS04020000Z0ED, SamacSys_Parts:RESC1005X40N@1
- added C173, C174, C175, C176, C177, C178, C179, C180, C181, C182, C183, C184, C185, C186, C187, C188: CS0402KRX7R8BB104, SamacSys_Parts:CAPC1005X65N
- added IC34, IC35, IC36, IC37, IC39, IC40, IC41, IC42, IC43, IC44, IC45, IC46, IC47, IC48, IC49, IC50: S35ML04G300WHI000, SamacSys_Parts:S35ML04G300WHI000
- added IC55: MUX36S16IRSNR, SamacSys_Parts:QFN40P400X400X80-33N
- added J4, J5, J6, J7, J8: TFM-120-02-L-D, SamacSys_Parts:SAMTEC_TFM-120-02-L-D
Connections:
- net FAULT1 renamed POWER_FAULT1
- net FAULT2 renamed POWER_FAULT2
- net FAULT3 renamed POWER_FAULT3
- removed net 14V_RAIL_VO: IC24.1, R480.2
- removed net 5V_RAIL_VO: IC26.1, R498.2
- removed net 6.5V_RAIL_VO: IC25.1, R489.2
- removed net ADIN1_10: IC17.23
- removed net ADIN1_11: IC22.23
- removed net ADIN1_12: IC23.23
- removed net ADIN2_10: IC17.18
- removed net ADIN2_11: IC22.18
- removed net ADIN2_12: IC23.18
- removed net ADIN2_9: IC16.18
- removed net POWER_TEMP1: J2.8
- removed net POWER_TEMP2: J2.10
- removed net POWER_TEMP3: J2.12
- removed net TEMP1_OUT: IC27.1, R503.2
- removed net TEMP2_OUT: IC28.1, R502.2
- removed net TEMP3_OUT: IC29.1, R506.2
- removed net TEMP4_OUT: IC30.1, R508.2
- new net !CS_INPUT: IC55.29
- new net 3.3V_DIGITAL: C110.1, C173.1, C174.1, C175.1, C176.1, C177.1, C178.1, C179.1, C180.1, C181.1, C182.1, C183.1, C184.1, C185.1, C186.1, C187.1, C188.1, IC10.2, IC10.4, IC34.8, IC35.8, IC36.8, IC37.8, IC39.8, IC40.8, IC41.8, IC42.8, IC43.8, IC44.8, IC45.8, IC46.8, IC47.8, IC48.8, IC49.8, IC50.8, IC55.16, IC55.31
- new net ADIN1_10_14V_RAIL_VO: IC17.23, IC24.1, R480.2
- new net ADIN1_11_TEMP2_OUT: IC22.23, IC28.1, R502.2
- new net ADIN1_12_TEMP4_OUT: IC23.23, IC30.1, R508.2
- new net ADIN1_8_POWER_TEMP1: IC15.23, J2.8, Z11.3
- new net ADIN1_9_5V_RAIL_VO: IC16.23, IC26.1, R498.2
- new net ADIN2_10_6.5V_RAIL_VO: IC17.18, IC25.1, R489.2
- new net ADIN2_11_TEMP1_OUT: IC22.18, IC27.1, R503.2
- new net ADIN2_12_TEMP3_OUT: IC23.18, IC29.1, R506.2
- new net ADIN2_8_POWER_TEMP2: IC15.18, J2.10, Z12.3
- new net ADIN2_9_POWER_TEMP3: IC16.18, J2.12, Z13.3
- new net MUX_0: IC55.15
- new net MUX_1: IC55.14
- new net MUX_2: IC55.11
- new net MUX_3: IC55.10
- new net N$349: J4.03
- new net N$351: J4.05
- new net N$352: J4.07
- new net N$353: J4.09
- new net N$354: J4.11
- new net N$355: J4.13
- new net N$357: J4.15
- new net N$358: J4.17
- new net N$359: J4.19
- new net N$361: J4.21
- new net N$362: J4.23
- new net N$363: J4.25
- new net N$364: J4.27
- new net N$365: J4.29
- new net N$366: J4.31
- new net N$367: J4.33
- new net N$368: J4.35
- new net N$369: J4.39
- new net N$370: J4.37
- new net N$371: J4.40
- new net N$372: J4.38
- new net N$373: J4.36
- new net N$374: J4.34
- new net N$375: J4.32
- new net N$376: J4.30
- new net N$377: J4.28
- new net N$378: J4.26
- new net N$379: J4.24
- new net N$380: J4.22
- new net N$381: J4.20
- new net N$382: J4.18
- new net N$383: J4.16
- new net N$384: J4.14
- new net N$385: J4.12
- new net N$386: J4.10
- new net N$387: J4.08
- new net N$388: J4.06
- new net N$389: J4.04
- new net N$390: J4.02
- new net N$391: J5.01
- new net N$392: J5.03
- new net N$393: J5.05
- new net N$394: J5.07
- new net N$395: J5.09
- new net N$396: J5.11
- new net N$397: J5.13
- new net N$398: J5.15
- new net N$399: J5.17
- new net N$400: J5.19
- new net N$401: J5.21
- new net N$402: J5.23
- new net N$403: J5.25
- new net N$404: J5.27
- new net N$405: J5.29
- new net N$406: J5.31
- new net N$407: J5.33
- new net N$408: J5.35
- new net N$409: J5.39
- new net N$410: J5.37
- new net N$411: J5.40
- new net N$412: J5.38
- new net N$413: J5.36
- new net N$414: J5.34
- new net N$415: J5.32
- new net N$416: J5.30
- new net N$417: J5.28
- new net N$418: J5.26
- new net N$419: J5.24
- new net N$420: J5.22
- new net N$421: J5.20
- new net N$422: J5.18
- new net N$423: J5.16
- new net N$424: J5.14
- new net N$425: J5.12
- new net N$426: J5.10
- new net N$427: J5.08
- new net N$428: J5.06
- new net N$429: J5.04
- new net N$430: J5.02
- new net N$431: J6.01
- new net N$432: J6.03
- new net N$433: J6.05
- new net N$434: J6.07
- new net N$435: J6.09
- new net N$436: J6.11
- new net N$437: J6.13
- new net N$438: J6.15
- new net N$439: J6.17
- new net N$440: J6.19
- new net N$441: J6.21
- new net N$442: J6.23
- new net N$443: J6.25
- new net N$444: J6.27
- new net N$445: J6.29
- new net N$446: J6.31
- new net N$447: J6.33
- new net N$448: J6.35
- new net N$449: J6.39
- new net N$450: J6.37
- new net N$451: J6.40
- new net N$452: J6.38
- new net N$453: J6.36
- new net N$454: J6.34
- new net N$455: J6.32
- new net N$456: J6.30
- new net N$457: J6.28
- new net N$458: J6.26
- new net N$459: J6.24
- new net N$460: J6.22
- new net N$461: J6.20
- new net N$462: J6.18
- new net N$463: J6.16
- new net N$464: J6.14
- new net N$465: J6.12
- new net N$466: J6.10
- new net N$467: J6.08
- new net N$468: J6.06
- new net N$469: J6.04
- new net N$470: J6.02
- new net N$471: J7.01
- new net N$472: J7.03
- new net N$473: J7.05
- new net N$474: J7.07
- new net N$475: J7.09
- new net N$476: J7.11
- new net N$477: J7.13
- new net N$478: J7.15
- new net N$479: J7.17
- new net N$480: J7.19
- new net N$481: J7.21
- new net N$482: J7.23
- new net N$483: J7.25
- new net N$484: J7.27
- new net N$485: J7.29
- new net N$486: J7.31
- new net N$487: J7.33
- new net N$488: J7.35
- new net N$489: J7.39
- new net N$490: J7.37
- new net N$491: J7.40
- new net N$492: J7.38
- new net N$493: J7.36
- new net N$494: J7.34
- new net N$495: J7.32
- new net N$496: J7.30
- new net N$497: J7.28
- new net N$498: J7.26
- new net N$499: J7.24
- new net N$500: J7.22
- new net N$501: J7.20
- new net N$502: J7.18
- new net N$503: J7.16
- new net N$504: J7.14
- new net N$505: J7.12
- new net N$506: J7.10
- new net N$507: J7.08
- new net N$508: J7.06
- new net N$509: J7.04
- new net N$510: J7.02
- new net N$511: J8.01
- new net N$512: J8.03
- new net N$513: J8.05
- new net N$514: J8.07
- new net N$515: J8.09
- new net N$516: J8.11
- new net N$517: J8.13
- new net N$518: J8.15
- new net N$519: J8.17
- new net N$520: J8.19
- new net N$521: J8.21
- new net N$522: J8.23
- new net N$523: J8.25
- new net N$524: J8.27
- new net N$525: J8.29
- new net N$526: J8.31
- new net N$527: J8.33
- new net N$528: J8.35
- new net N$529: J8.39
- new net N$530: J8.37
- new net N$531: J8.40
- new net N$532: J8.38
- new net N$533: J8.36
- new net N$534: J8.34
- new net N$535: J8.32
- new net N$536: J8.30
- new net N$537: J8.28
- new net N$538: J8.26
- new net N$539: J8.24
- new net N$540: J8.22
- new net N$541: J8.20
- new net N$542: J8.18
- new net N$543: J8.16
- new net N$544: J8.14
- new net N$545: J8.12
- new net N$546: J8.10
- new net N$547: J8.08
- new net N$548: J8.06
- new net N$549: J8.04
- new net N$550: J8.02
- new net NAND1: IC34.1, IC55.17
- new net NAND10: IC44.1, IC55.7
- new net NAND11: IC45.1, IC55.6
- new net NAND12: IC46.1, IC55.5
- new net NAND13: IC47.1, IC55.4
- new net NAND14: IC48.1, IC55.3
- new net NAND15: IC49.1, IC55.2
- new net NAND16: IC50.1, IC55.1
- new net NAND2: IC35.1, IC55.18
- new net NAND3: IC36.1, IC55.19
- new net NAND4: IC37.1, IC55.20
- new net NAND5: IC39.1, IC55.21
- new net NAND6: IC40.1, IC55.22
- new net NAND7: IC41.1, IC55.23
- new net NAND8: IC42.1, IC55.24
- new net NAND9: IC43.1, IC55.8
- new net NAND_SPI_!HOLD/IO3: IC34.7, IC35.7, IC36.7, IC37.7, IC39.7, IC40.7, IC41.7, IC42.7, IC43.7, IC44.7, IC45.7, IC46.7, IC47.7, IC48.7, IC49.7, IC50.7
- new net NAND_SPI_!WP/IO2: IC34.2, IC35.2, IC36.2, IC37.2, IC39.2, IC40.2, IC41.2, IC42.2, IC43.2, IC44.2, IC45.2, IC46.2, IC47.2, IC48.2, IC49.2, IC50.2
- new net NAND_SPI_CLK: IC34.6, IC35.6, IC36.6, IC37.6, IC39.6, IC40.6, IC41.6, IC42.6, IC43.6, IC44.6, IC45.6, IC46.6, IC47.6, IC48.6, IC49.6, IC50.6
- new net NAND_SPI_SI/IO0: IC34.5, IC35.5, IC36.5, IC37.5, IC39.5, IC40.5, IC41.5, IC42.5, IC43.5, IC44.5, IC45.5, IC46.5, IC47.5, IC48.5, IC49.5, IC50.5
- new net NAND_SPI_SO/IO1: IC34.3, IC35.3, IC36.3, IC37.3, IC39.3, IC40.3, IC41.3, IC42.3, IC43.3, IC44.3, IC45.3, IC46.3, IC47.3, IC48.3, IC49.3, IC50.3
- net 3.3V_SENSORS: no longer C110.1, IC10.2, IC10.4
- net ADIN1_8: no longer IC15.23, Z11.3
- net ADIN1_9: no longer IC16.23, Z13.3
- net ADIN2_8: no longer IC15.18, Z12.3
- net GND: now also C173.2, C174.2, C175.2, C176.2, C177.2, C178.2, C179.2, C180.2, C181.2, C182.2, C183.2, C184.2, C185.2, C186.2, C187.2, C188.2, IC34.4, IC35.4, IC36.4, IC37.4, IC39.4, IC40.4, IC41.4, IC42.4, IC43.4, IC44.4, IC45.4, IC46.4, IC47.4, IC48.4, IC49.4, IC50.4, IC55.25, IC55.9; no longer R158.2, R159.2, R160.2, R161.2, R162.2, R163.2, R201.2, R203.2, R205.2, R207.2, R209.2, R211.2, SG_BUSY_2.1
- net N$170: no longer R162.1
- net N$180: no longer R163.1
- net N$190: no longer R201.1
- net N$20: no longer R158.1
- net N$200: no longer SG_BUSY_2.2
- net N$220: no longer R203.1
- net N$230: no longer R205.1
- net N$240: no longer R207.1
- net N$250: no longer R209.1
- net N$260: no longer R211.1
- net N$50: no longer R159.1
- net N$60: now also J4.01; no longer R160.1, STRAINGGAUGE_2.29
- net N$70: no longer R161.1

Commit message: Checking main wire up
Parts:
- removed GENERAL_PURPOSE_1, STRAINGGAUGE_2: ADS8588HIPM, SamacSys_Parts:QFP50P1200X1200X160-64N_NO_3D
- removed GEN_BUSY_1, R147, R148, R149, R150, R151, R152, R153, R154, R155, R156, R157, R221, R227, R229, R230, R231, R232, R233, R234, R235, R236, R237, R238, R239, SG_BUSY_1: RCS04020000Z0ED, SamacSys_Parts:RESC1005X40N@1
- added IC51, IC52: ADS8588HIPM, SamacSys_Parts:QFP50P1200X1200X160-64N_NO_3D
- moved IC38 1646.9 mm to (-448.8, -1268.7)
Connections:
- net N$377 renamed PB13
- net N$442 renamed PG7
- net N$524 renamed SAD2
- net N$525 renamed SCL2
- net N$541 renamed NAND_SPI_!HOLD/IO03
- removed net !CS_INPUT: IC55.29
- removed net 0: GENERAL_PURPOSE_1.13, IC38.13, STRAINGGAUGE_2.13
- removed net 1: GENERAL_PURPOSE_1.12, IC38.12, STRAINGGAUGE_2.12
- removed net 14: STRAINGGAUGE_2.24
- removed net 15: STRAINGGAUGE_2.25
- removed net 18: IC38.25
- removed net 19: IC38.24
- removed net 2: GENERAL_PURPOSE_1.11, IC38.11, STRAINGGAUGE_2.11
- removed net 3: GENERAL_PURPOSE_1.10, GENERAL_PURPOSE_1.9, IC38.10, STRAINGGAUGE_2.10, STRAINGGAUGE_2.9
- removed net 3.3V: J1.1, J1.3, J1.5, J1.7, R33.1, R35.1, R37.1, R39.1, R43.1, R45.1, R47.1, R49.1
- removed net 40: GENERAL_PURPOSE_1.24
- removed net 41: GENERAL_PURPOSE_1.25
- removed net BUSYBUSY: IC38.14, SG_BUSY_1.1
- removed net DVDD: C11.2, C24.2, C5.2, GENERAL_PURPOSE_1.23, GENERAL_PURPOSE_1.3, GENERAL_PURPOSE_1.34, GENERAL_PURPOSE_1.5, GENERAL_PURPOSE_1.6, GENERAL_PURPOSE_1.7, IC38.23, IC38.3, IC38.34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
- removed net N$1 (its old number): IC38.31, R157.1
- removed net N$10: IC38.22, R152.1
- removed net N$11: IC38.21, R151.1
- removed net N$114: C63.1, F3.3, R37.2
- removed net N$119: C64.1, F4.3, R39.2
- removed net N$12: IC38.20, R150.1
- removed net N$13: IC38.19, R149.1
- removed net N$130: IC13.5
- removed net N$132: IC13.6
- removed net N$133: IC13.7
- removed net N$136: C66.1, F6.3, R43.2
- removed net N$139: C67.1, F7.3, R45.2
- removed net N$14: IC38.18, R148.1
- removed net N$142: C68.1, F8.3, R47.2
- removed net N$145: C69.1, F9.3, R49.2
- removed net N$15: IC38.17, R147.1
- removed net N$16: IC38.16, R221.1
- removed net N$170: STRAINGGAUGE_2.27
- removed net N$171: IC38.9
- removed net N$179: IC15.6
- removed net N$180: STRAINGGAUGE_2.22
- removed net N$190: STRAINGGAUGE_2.21
- removed net N$2: C40.1, F2.3, R35.2
- removed net N$20: STRAINGGAUGE_2.31
- removed net N$200: STRAINGGAUGE_2.14
- removed net N$2000: GENERAL_PURPOSE_1.14, GEN_BUSY_1.2
- removed net N$21: IC38.15
- removed net N$210: STRAINGGAUGE_2.15
- removed net N$2100: GENERAL_PURPOSE_1.15
- removed net N$214: IC17.5
- removed net N$220: STRAINGGAUGE_2.20
- removed net N$230: STRAINGGAUGE_2.19
- removed net N$233: IC18.6
- removed net N$234: IC18.7
- removed net N$240: STRAINGGAUGE_2.18
- removed net N$249: IC19.5
- removed net N$250: STRAINGGAUGE_2.17
- removed net N$251: IC19.6
- removed net N$252: IC19.7
- removed net N$260: STRAINGGAUGE_2.16
- removed net N$269: IC20.7
- removed net N$2700: GENERAL_PURPOSE_1.31, R229.1
- removed net N$2800: GENERAL_PURPOSE_1.30, R230.1
- removed net N$283: IC21.5
- removed net N$285: IC21.7
- removed net N$2900: GENERAL_PURPOSE_1.29, R231.1
- removed net N$299: IC22.5
- removed net N$3: IC38.30, R156.1
- removed net N$300: IC22.6
- removed net N$3000: GENERAL_PURPOSE_1.28, R232.1
- removed net N$3100: GENERAL_PURPOSE_1.27, R233.1
- removed net N$315: IC23.5
- removed net N$316: IC23.6
- removed net N$3200: GENERAL_PURPOSE_1.22, R234.1
- removed net N$3300: GENERAL_PURPOSE_1.21, R235.1
- removed net N$3400: GENERAL_PURPOSE_1.20, R236.1
- removed net N$349: J4.03
- removed net N$3500: GENERAL_PURPOSE_1.19, R237.1
- removed net N$351: J4.05
- removed net N$352: J4.07
- removed net N$353: J4.09
- removed net N$354: J4.11
- removed net N$355: J4.13
- removed net N$357: J4.15
- removed net N$358: J4.17
- removed net N$359: J4.19
- removed net N$3600: GENERAL_PURPOSE_1.18, R238.1
- removed net N$361: J4.21
- removed net N$362: J4.23
- removed net N$363: J4.25
- removed net N$364: J4.27
- removed net N$365: J4.29
- removed net N$366: J4.31
- removed net N$367: J4.33
- removed net N$368: J4.35
- removed net N$369: J4.39
- removed net N$370: J4.37
- removed net N$3700: GENERAL_PURPOSE_1.17, R239.1
- removed net N$371: J4.40
- removed net N$372: J4.38
- removed net N$373: J4.36
- removed net N$374: J4.34
- removed net N$375: J4.32
- removed net N$376: J4.30
- removed net N$378: J4.26
- removed net N$379: J4.24
- removed net N$380: J4.22
- removed net N$3800: GENERAL_PURPOSE_1.16, R227.1
- removed net N$381: J4.20
- removed net N$382: J4.18
- removed net N$383: J4.16
- removed net N$384: J4.14
- removed net N$385: J4.12
- removed net N$386: J4.10
- removed net N$387: J4.08
- removed net N$388: J4.06
- removed net N$389: J4.04
- removed net N$390: J4.02
- removed net N$391: J5.01
- removed net N$392: J5.03
- removed net N$393: J5.05
- removed net N$394: J5.07
- removed net N$395: J5.09
- removed net N$396: J5.11
- removed net N$397: J5.13
- removed net N$398: J5.15
- removed net N$399: J5.17
- removed net N$4: IC38.29, R155.1
- removed net N$400: J5.19
- removed net N$401: J5.21
- removed net N$402: J5.23
- removed net N$403: J5.25
- removed net N$404: J5.27
- removed net N$405: J5.29
- removed net N$406: J5.31
- removed net N$407: J5.33
- removed net N$408: J5.35
- removed net N$409: J5.39
- removed net N$410: J5.37
- removed net N$411: J5.40
- removed net N$412: J5.38
- removed net N$413: J5.36
- removed net N$414: J5.34
- removed net N$415: J5.32
- removed net N$416: J5.30
- removed net N$417: J5.28
- removed net N$418: J5.26
- removed net N$419: J5.24
- removed net N$420: J5.22
- removed net N$421: J5.20
- removed net N$422: J5.18
- removed net N$423: J5.16
- removed net N$424: J5.14
- removed net N$425: J5.12
- removed net N$426: J5.10
- removed net N$427: J5.08
- removed net N$428: J5.06
- removed net N$429: J5.04
- removed net N$43: IC4.5
- removed net N$430: J5.02
- removed net N$431: J6.01
- removed net N$432: J6.03
- removed net N$433: J6.05
- removed net N$434: J6.07
- removed net N$435: J6.09
- removed net N$436: J6.11
- removed net N$437: J6.13
- removed net N$438: J6.15
- removed net N$439: J6.17
- removed net N$440: J6.19
- removed net N$441: J6.21
- removed net N$443: J6.25
- removed net N$444: J6.27
- removed net N$445: J6.29
- removed net N$446: J6.31
- removed net N$447: J6.33
- removed net N$448: J6.35
- removed net N$449: J6.39
- removed net N$450: J6.37
- removed net N$451: J6.40
- removed net N$452: J6.38
- removed net N$453: J6.36
- removed net N$454: J6.34
- removed net N$455: J6.32
- removed net N$456: J6.30
- removed net N$457: J6.28
- removed net N$458: J6.26
- removed net N$459: J6.24
- removed net N$46: IC4.7
- removed net N$460: J6.22
- removed net N$461: J6.20
- removed net N$462: J6.18
- removed net N$463: J6.16
- removed net N$464: J6.14
- removed net N$465: J6.12
- removed net N$466: J6.10
- removed net N$467: J6.08
- removed net N$468: J6.06
- removed net N$469: J6.04
- removed net N$470: J6.02
- removed net N$471: J7.01
- removed net N$472: J7.03
- removed net N$473: J7.05
- removed net N$474: J7.07
- removed net N$475: J7.09
- removed net N$476: J7.11
- removed net N$477: J7.13
- removed net N$478: J7.15
- removed net N$479: J7.17
- removed net N$480: J7.19
- removed net N$481: J7.21
- removed net N$482: J7.23
- removed net N$483: J7.25
- removed net N$484: J7.27
- removed net N$485: J7.29
- removed net N$486: J7.31
- removed net N$487: J7.33
- removed net N$488: J7.35
- removed net N$490: J7.37
- removed net N$491: J7.40
- removed net N$492: J7.38
- removed net N$493: J7.36
- removed net N$494: J7.34
- removed net N$495: J7.32
- removed net N$496: J7.30
- removed net N$497: J7.28
- removed net N$498: J7.26
- removed net N$499: J7.24
- removed net N$5: C38.1, F1.3, R33.2
- removed net N$50: STRAINGGAUGE_2.30
- removed net N$500: J7.22
- removed net N$501: J7.20
- removed net N$502: J7.18
- removed net N$511: J8.01
- removed net N$512: J8.03
- removed net N$513: J8.05
- removed net N$514: J8.07
- removed net N$515: J8.09
- removed net N$516: J8.11
- removed net N$517: J8.13
- removed net N$518: J8.15
- removed net N$519: J8.17
- removed net N$520: J8.19
- removed net N$521: J8.21
- removed net N$522: J8.23
- removed net N$523: J8.25
- removed net N$529: J8.39
- removed net N$531: J8.40
- removed net N$532: J8.38
- removed net N$533: J8.36
- removed net N$534: J8.34
- removed net N$535: J8.32
- removed net N$536: J8.30
- removed net N$537: J8.28
- removed net N$538: J8.26
- removed net N$539: J8.24
- removed net N$540: J8.22
- removed net N$542: J8.18
- removed net N$543: J8.16
- removed net N$544: J8.14
- removed net N$545: J8.12
- removed net N$546: J8.10
- removed net N$547: J8.08
- removed net N$548: J8.06
- removed net N$549: J8.04
- removed net N$550: J8.02
- removed net N$60: J4.01
- removed net N$64: IC11.6
- removed net N$65: IC11.7
- removed net N$70: STRAINGGAUGE_2.28
- removed net N$8: IC38.28, R154.1
- removed net N$80: IC12.5
- removed net N$81: IC12.6
- removed net N$82: IC12.7
- removed net N$9: IC38.27, R153.1
- new net !CS_ADC: IC38.13, IC51.13, IC52.13, J7.13
- new net !CS_INPUT_NAND: IC55.29, J8.10
- new net 3.3V_MCU: UC1.3V3_VDD
- new net 5V_CONNECTOR: C109.1, IC9.4, IC9.5, J6.16, J6.18
- new net BUSY_ADC_1: IC51.14, J7.15
- new net BUSY_ADC_2: IC38.14, J7.23
- new net BUSY_ADC_3: IC52.14, J7.31
- new net CONVSTAB_ADC: IC38.10, IC38.9, IC51.10, IC51.9, IC52.10, IC52.9, J7.07
- new net DOUTA_ADC_1: IC51.24, J7.21
- new net DOUTA_ADC_2: IC38.24, J7.29
- new net DOUTA_ADC_3: IC52.24, J7.37
- new net DOUTB_ADC_1: IC51.25, J7.19
- new net DOUTB_ADC_2: IC38.25, J7.27
- new net DOUTB_ADC_3: IC52.25, J7.35
- new net D_SENSE1: C40.1, F2.3, J7.26, R35.2
- new net D_SENSE2: C38.1, F1.3, J7.28, R33.2
- new net D_SENSE3: C63.1, F3.3, J7.30, R37.2
- new net D_SENSE4: C64.1, F4.3, J7.32, R39.2
- new net D_SENSE5: C66.1, F6.3, J7.34, R43.2
- new net D_SENSE6: C67.1, F7.3, J7.36, R45.2
- new net D_SENSE7: C68.1, F8.3, J7.38, R47.2
- new net D_SENSE8: C69.1, F9.3, J7.40, R49.2
- new net ETH_CRS_DV: UC1.PA7
- new net ETH_MDC: UC1.PC1
- new net ETH_MDIO: UC1.PA2
- new net ETH_REF_CLK: UC1.PA1
- new net ETH_RXD0: UC1.PC4
- new net ETH_RXD1: UC1.PC5
- new net ETH_TXD0: UC1.PG13
- new net ETH_TXD1: UC1.PB13
- new net ETH_TX_EN: UC1.PG11
- new net FIRSTDATA_ADC_1: IC51.15, J7.17
- new net FIRSTDATA_ADC_2: IC38.15, J7.25
- new net FIRSTDATA_ADC_3: IC52.15, J7.33
- new net LED_OUT1: J7.22, R52.2
- new net LED_OUT2: J7.20, R54.2
- new net LED_OUT3: J7.18, R56.2
- new net N$554: UC1.BOOT0
- new net N$566: UC1.VBAT
- new net N$582: UC1.NC_1
- new net N$605: UC1.NC_2
- new net N$606: UC1.VIN
- new net N$607: UC1.5V
- new net N$608: UC1.3V3
- new net N$609: UC1.NRST
- new net N$610: UC1.IOREF
- new net N$611: UC1.NC_3
- new net N$618: UC1.VREFP
- new net N$666: UC1.31_AGND
- new net N$677: UC1.5V_USB_STLK
- new net OS0_ADC: IC38.3, IC51.3, IC52.3, J7.01
- new net OS1_ADC: IC38.4, IC52.4, J7.03
- new net OS2_ADC: IC38.5, IC51.4, IC51.5, IC52.5, J7.05
- new net PA0: J4.01, UC1.PA0
- new net PA10: J4.15, UC1.PA10
- new net PA11: J4.17, UC1.PA11
- new net PA12: J4.19, UC1.PA12
- new net PA13: J4.21, UC1.PA13
- new net PA14: J4.23, UC1.PA14
- new net PA15: J4.25, UC1.PA15
- new net PA3: J4.03, UC1.PA3
- new net PA4: J4.05, UC1.PA4
- new net PA5: J4.07, UC1.PA5
- new net PA6: J4.09, UC1.PA6
- new net PA8: J4.11, UC1.PA8
- new net PA9: J4.13, UC1.PA9
- new net PB0: J4.27, UC1.PB0
- new net PB1: J4.29, UC1.PB1
- new net PB10: J4.34, UC1.PB10
- new net PB11: J4.32, UC1.PB11
- new net PB12: J4.30, UC1.PB12
- new net PB14: J4.26, UC1.PB14
- new net PB15: J4.24, UC1.PB15
- new net PB2: J4.31, UC1.PB2
- new net PB3: J4.33, UC1.PB3
- new net PB4: J4.35, UC1.PB4
- new net PB5: J4.37, UC1.PB5
- new net PB6: J4.39, UC1.PB6
- new net PB7: J4.40, UC1.PB7
- new net PB8: J4.38, UC1.PB8
- new net PB9: J4.36, UC1.PB9
- new net PC0: J4.22, UC1.PC0
- new net PC10: J4.08, UC1.PC10
- new net PC11: J4.06, UC1.PC11
- new net PC12: J4.04, UC1.PC12
- new net PC13: J4.02, UC1.PC13
- new net PC14-0SC32_IN: UC1.PC14
- new net PC15-OSC32_OUT: UC1.PC15
- new net PC2: J4.20, UC1.PC2
- new net PC3: J4.18, UC1.PC3
- new net PC6: J4.16, UC1.PC6
- new net PC7: J4.14, UC1.PC7
- new net PC8: J4.12, UC1.PC8
- new net PC9: J4.10, UC1.PC9
- new net PD0: J5.01, UC1.PD0
- new net PD1: J5.03, UC1.PD1
- new net PD11: J5.17, UC1.PD11
- new net PD12: J5.19, UC1.PD12
- new net PD13: J5.21, UC1.PD13
- new net PD14: J5.23, UC1.PD14
- new net PD15: J5.25, UC1.PD15
- new net PD2: J5.05, UC1.PD2
- new net PD3: J5.07, UC1.PD3
- new net PD4: J5.09, UC1.PD4
- new net PD5: J5.11, UC1.PD5
- new net PD6: J5.13, UC1.PD6
- new net PD7: J5.15, UC1.PD7
- new net PE0: J5.27, UC1.PE0
- new net PE1: J5.29, UC1.PE1
- new net PE10: J5.34, UC1.PE10
- new net PE11: J5.32, UC1.PE11
- new net PE12: J5.30, UC1.PE12
- new net PE13: J5.28, UC1.PE13
- new net PE14: J5.26, UC1.PE14
- new net PE15: J5.24, UC1.PE15
- new net PE2: J5.31, UC1.PE2
- new net PE3: J5.33, UC1.PE3
- new net PE4: J5.35, UC1.PE4
- new net PE5: J5.37, UC1.PE5
- new net PE6: J5.39, UC1.PE6
- new net PE7: J5.40, UC1.PE7
- new net PE8: J5.38, UC1.PE8
- new net PE9: J5.36, UC1.PE9
- new net PF0: UC1.PF0
- new net PF1: J5.22, UC1.PF1
- new net PF10: J5.04, UC1.PF10
- new net PF11: J5.02, UC1.PF11
- new net PF12: J6.01, UC1.PF12
- new net PF13: J6.03, UC1.PF13
- new net PF14: J6.05, UC1.PF14
- new net PF15: J6.07, UC1.PF15
- new net PF2: J5.20, UC1.PF2
- new net PF3: J5.18, UC1.PF3
- new net PF4: J5.16, UC1.PF4
- new net PF5: J5.14, UC1.PF5
- new net PF6: J5.12, UC1.PF6
- new net PF7: J5.10, UC1.PF7
- new net PF8: J5.08, UC1.PF8
- new net PF9: J5.06, UC1.PF9
- new net PG0: J6.09, UC1.PG0
- new net PG1: J6.11, UC1.PG1
- new net PG10: J6.29, UC1.PG10
- new net PG12: J6.31, UC1.PG12
- new net PG14: J6.33, UC1.PG14
- new net PG15: J6.35, UC1.PG15
- new net PG2: J6.13, UC1.PG2
- new net PG3: J6.15, UC1.PG3
- new net PG4: J6.17, UC1.PG4
- new net PG5: J6.19, UC1.PG5
- new net PG6: J6.21, UC1.PG6
- new net PG8: J6.25, UC1.PG8
- new net PG9: J6.27, UC1.PG9
- new net PH0-OSC_IN: UC1.PH0
- new net PH1: J6.37, UC1.PH1
- new net P_LED: J7.24, R42.2
- new net RESET_ADC: IC38.11, IC51.11, IC52.11, J7.09
- new net SCLK_ADC: IC38.12, IC51.12, IC52.12, J7.11
- new net USART3_TX: UC1.PD8
- new net USART4_RX: UC1.PD9
- new net USB_FS_OVCR: UC1.PG7
- new net USB_FS_PWR_EN: UC1.PD10
- net !IMU_CS: now also J8.03
- net !IMU_RST: now also J8.01
- net !ISO_CS: now also J8.28
- net !THERMOCOUPLE_CS: now also J8.36
- net 13.5V_BUS: now also J6.10, J6.12, J6.14
- net 14V_BUS_FROM_CONNECTOR: now also J6.32
- net 3.3V_DIGITAL: now also C11.2, C170.1, C24.2, C5.2, IC11.6, IC13.5, IC13.6, IC15.6, IC17.5, IC19.5, IC21.5, IC23.5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
- net 3.3V_SENSORS: no longer C170.1, IC32.11, IC32.16, IC32.5, IC32.6, IC32.7, IC32.8
- net 3.3V_SWITCHING: now also J1.1, J1.3, J1.5, J1.7, J6.20, J6.26, R33.1, R35.1, R37.1, R39.1, R43.1, R45.1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
- net 5V_BUS_FROM_CONNECTOR: now also J6.28
- net 5V_MCU: now also UC1.5V_EXT
- net 5V_ON_BOARD: now also C1.1, C10.2, C12.2, C15.2, C18.2, C19.1, C23.2, C27.2, C4.2, C6.2, C7.1, IC38.1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; no longer C109.1, IC9.4, IC9.5
- net 6.5V_BUS_FROM_CONNECTOR: now also J6.30
- net AVDD: now also IC52.1; no longer C1.1, C10.2, C12.2, C15.2, C18.2, C19.1, C23.2, C27.2, C4.2, C6.2, C7.1, GENERAL_PURPOSE_1.1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
- net DIN5: no longer R42.2
- net DIN6: no longer R52.2
- net DIN7: no longer R54.2
- net DIN8: no longer R56.2
- net GND: now also IC11.7, IC12.5, IC12.6, IC12.7, IC13.7, IC18.6, IC18.7, IC19.6, IC19.7, IC20.7, IC21.7, IC22.5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; no longer GENERAL_PURPOSE_1.2, GENERAL_PURPOSE_1.26, GENERAL_PURPOSE_1.32, GENERAL_PURPOSE_1.33, GENERAL_PURPOSE_1.35, GENERAL_PURPOSE_1.4, GENERAL_PURPOSE_1.40, GENERAL_PURPOSE_1.41, GENERAL_PURPOSE_1.43, GENERAL_PURPOSE_1.46, GENERAL_PURPOSE_1.47, GENERAL_PURPOSE_1.8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
- net GPS_EN: now also J8.39
- net GPS_RX: now also J8.40
- net GPS_TX: now also J8.38
- net GP_1_N: now also IC52.50; no longer GENERAL_PURPOSE_1.50
- net GP_1_P: now also IC52.49; no longer GENERAL_PURPOSE_1.49
- net GP_2_N: now also IC52.52; no longer GENERAL_PURPOSE_1.52
- net GP_2_P: now also IC52.51; no longer GENERAL_PURPOSE_1.51
- net GP_3_N: now also IC52.54; no longer GENERAL_PURPOSE_1.54
- net GP_3_P: now also IC52.53; no longer GENERAL_PURPOSE_1.53
- net GP_4_N: now also IC52.56; no longer GENERAL_PURPOSE_1.56
- net GP_4_P: now also IC52.55; no longer GENERAL_PURPOSE_1.55
- net GP_5_N: now also IC52.58; no longer GENERAL_PURPOSE_1.58
- net GP_5_P: now also IC52.57; no longer GENERAL_PURPOSE_1.57
- net GP_6_N: now also IC52.60; no longer GENERAL_PURPOSE_1.60
- net GP_6_P: now also IC52.59; no longer GENERAL_PURPOSE_1.59
- net GP_7_N: now also IC52.62; no longer GENERAL_PURPOSE_1.62
- net GP_7_P: now also IC52.61; no longer GENERAL_PURPOSE_1.61
- net GP_8_N: now also IC52.64; no longer GENERAL_PURPOSE_1.64
- net GP_8_P: now also IC52.63; no longer GENERAL_PURPOSE_1.63
- net IMU_DIN: now also J8.05
- net IMU_DOUT: now also J8.07
- net IMU_DR: now also J8.13
- net IMU_SCLK: now also J8.09
- net IMU_SYNC: now also J8.11
- net ISO_MISO: now also J8.26
- net ISO_MOSI: now also J8.24
- net ISO_SPI_SCLK: now also J8.22
- net ISO_SPI_SLOW: now also J8.30
- net MASS_ON: now also J8.25
- net MUX_0: now also J8.02
- net MUX_1: now also J8.04
- net MUX_2: now also J8.06
- net MUX_3: now also J8.08
- net NAND_SPI_!WP/IO2: now also J8.18
- net NAND_SPI_CLK: now also J8.12
- net NAND_SPI_SI/IO0: now also J8.14
- net NAND_SPI_SO/IO1: now also J8.16
- net POWER_FAULT1: now also J8.15
- net POWER_FAULT2: now also J8.17
- net POWER_FAULT3: now also J8.19
- net REFCAPAB: now also IC51.44, IC51.45; no longer IC38.44, IC38.45
- net REFCAPAB0: now also IC38.44, IC38.45; no longer STRAINGGAUGE_2.44, STRAINGGAUGE_2.45
- net REFCAPAB00: now also IC52.44, IC52.45; no longer GENERAL_PURPOSE_1.44, GENERAL_PURPOSE_1.45
- net REFIN/OUT: now also IC51.42; no longer IC38.42
- net REFIN/OUT0: now also IC38.42; no longer STRAINGGAUGE_2.42
- net REFIN/OUT00: now also IC52.42; no longer GENERAL_PURPOSE_1.42
- net REGCAP1: now also IC51.36; no longer IC38.36
- net REGCAP10: now also IC38.36; no longer STRAINGGAUGE_2.36
- net REGCAP100: now also IC52.36; no longer GENERAL_PURPOSE_1.36
- net REGCAP2: now also IC51.39; no longer IC38.39
- net REGCAP20: now also IC38.39; no longer STRAINGGAUGE_2.39
- net REGCAP200: now also IC52.39; no longer GENERAL_PURPOSE_1.39
- net SCL1: now also J8.23
- net SDA1: now also J8.21
- net THERMOCOUPLE_MISO: now also J8.34
- net THERMOCOUPLE_SCLK: now also J8.32
- net VIN10_N: now also IC38.52; no longer STRAINGGAUGE_2.52
- net VIN10_P: now also IC38.51; no longer STRAINGGAUGE_2.51
- net VIN11_N: now also IC38.54; no longer STRAINGGAUGE_2.54
- net VIN11_P: now also IC38.53; no longer STRAINGGAUGE_2.53
- net VIN12_N: now also IC38.56; no longer STRAINGGAUGE_2.56
- net VIN12_P: now also IC38.55; no longer STRAINGGAUGE_2.55
- net VIN13_N: now also IC38.58; no longer STRAINGGAUGE_2.58
- net VIN13_P: now also IC38.57; no longer STRAINGGAUGE_2.57
- net VIN14_N: now also IC38.60; no longer STRAINGGAUGE_2.60
- net VIN14_P: now also IC38.59; no longer STRAINGGAUGE_2.59
- net VIN15_N: now also IC38.62; no longer STRAINGGAUGE_2.62
- net VIN15_P: now also IC38.61; no longer STRAINGGAUGE_2.61
- net VIN16_N: now also IC38.64; no longer STRAINGGAUGE_2.64
- net VIN16_P: now also IC38.63; no longer STRAINGGAUGE_2.63
- net VIN1_N: now also IC51.50; no longer IC38.50
- net VIN1_P: now also IC51.49; no longer IC38.49
- net VIN2_N: now also IC51.52; no longer IC38.52
- net VIN2_P: now also IC51.51; no longer IC38.51
- net VIN3_N: now also IC51.54; no longer IC38.54
- net VIN3_P: now also IC51.53; no longer IC38.53
- net VIN4_N: now also IC51.56; no longer IC38.56
- net VIN4_P: now also IC51.55; no longer IC38.55
- net VIN5_N: now also IC51.58; no longer IC38.58
- net VIN5_P: now also IC51.57; no longer IC38.57
- net VIN6_N: now also IC51.60; no longer IC38.60
- net VIN6_P: now also IC51.59; no longer IC38.59
- net VIN7_N: now also IC51.62; no longer IC38.62
- net VIN7_P: now also IC51.61; no longer IC38.61
- net VIN8_N: now also IC51.64; no longer IC38.64
- net VIN8_P: now also IC51.63; no longer IC38.63
- net VIN9_N: now also IC38.50; no longer STRAINGGAUGE_2.50
- net VIN9_P: now also IC38.49; no longer STRAINGGAUGE_2.49

Commit message: Began board layout!
Parts:
- removed C26: C3225X7R1N106K250AC, SamacSys_Parts:CAPC3225X230N
- added C190: CGA4J3X7R1H105K125AB, SamacSys_Parts:CAPC2012X145N
- added R147, R148, R149, R150: CRCW04021K30FKTD, SamacSys_Parts:RESC1005X40N
- C1: value CGA4J3X7R1H105K125AB -> C3225X7R1N106K250AC; device SamacSys_Parts:CAPC2012X145N -> SamacSys_Parts:CAPC3225X230N
- C13, C16, C17: value CNA6P1X7R1H106K250AE -> C3225X7R1N106K250AC; device SamacSys_Parts:CAPC3225X270N -> SamacSys_Parts:CAPC3225X230N
- C14: value CNA6P1X7R1H106K250AE -> CGA4J3X7R1H105K125AB; device SamacSys_Parts:CAPC3225X270N -> SamacSys_Parts:CAPC2012X145N
- C22: value 06033C105KAT4A -> C3225X7R1N106K250AC; device SamacSys_Parts:CAPC1608X90N -> SamacSys_Parts:CAPC3225X230N
- moved J6 1406.4 mm to (75.7, 60.2)
- moved J7 1406.4 mm to (75.7, 47.5)
- moved J5 1375.3 mm to (54.2, 47.7), turned to 90 degrees
- moved J4 1359.1 mm to (41.4, 47.8), turned to 90 degrees
- moved J8 1336.3 mm to (75.5, 35.0)
- moved C180 1291.1 mm to (-310.6, -86.4)
- moved C181 1291.1 mm to (-310.6, -22.9)
- moved C182 1291.1 mm to (-290.3, -22.9)
- moved IC39 1291.1 mm to (-318.2, -151.2)
- moved C174 1291.1 mm to (-310.6, -193.1)
- moved C175 1291.1 mm to (-310.6, -175.3)
- moved C176 1291.1 mm to (-310.6, -157.5)
- moved C177 1291.1 mm to (-310.6, -94.0)
- moved C178 1291.1 mm to (-310.6, -91.5)
- moved C179 1291.1 mm to (-310.6, -89.0)
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Connections:
- removed net AVDD: C22.2, IC52.1
- removed net N$528: J8.35
- removed net N$530: J8.37
- removed net SAD2: J8.27
- new net N$2: J8.38
- new net N$3: J8.40
- new net SDA2: IC14.19, IC15.19, IC16.19, IC17.19, IC19.19, IC22.19, IC23.19, J8.27, R149.1
- net 3.3V_DIGITAL: now also R147.2, R148.2, R149.2, R150.2
- net 5V_ON_BOARD: now also C14.2, C190.1, IC52.1; no longer C1.1
- net GND: now also C14.1, C190.2, C22.2; no longer C14.2, C22.1, C26.2
- net GPS_RX: now also J8.37; no longer J8.40
- net GPS_TX: now also J8.35; no longer J8.38
- net REFCAPAB0: now also C22.1; no longer C16.1
- net REFIN/OUT: now also C1.1; no longer C14.1
- net REFIN/OUT0: now also C16.1; no longer C17.1
- net REFIN/OUT00: now also C17.1; no longer C26.1
- net SCL1: now also R148.1; no longer IC14.20, IC15.20, IC16.20, IC17.20, IC19.20, IC22.20, IC23.20
- net SCL2: now also IC14.20, IC15.20, IC16.20, IC17.20, IC19.20, IC22.20, IC23.20, R150.1
- net SDA1: now also R147.1; no longer IC14.19, IC15.19, IC16.19, IC17.19, IC19.19, IC22.19, IC23.19
Other:
- board size 443.2 x 345.1 mm -> 279.4 x 330.2 mm
