File: MasterPCB_transfer.brd (EAGLE design)
At the start: 259.8 x 281.7 mm, 1001 parts, among them IC1 NCS21911SN2T1G, IC10 LDL1117S33R, IC11 LTC4222CUH#PBF, IC12 LTC4222CUH#PBF, IC13 LTC4222CUH#PBF, IC14 LTC4222CUH#PBF, IC15 LTC4222CUH#PBF, IC16 LTC4222CUH#PBF, IC17 LTC4222CUH#PBF, IC18 LTC4222CUH#PBF, IC19 LTC4222CUH#PBF, IC2 NCS21911SN2T1G, IC20 LTC4222CUH#PBF, IC21 LTC4222CUH#PBF, IC22 LTC4222CUH#PBF, IC23 LTC4222CUH#PBF, IC24 NCS21911SN2T1G, IC25 NCS21911SN2T1G, IC26 NCS21911SN2T1G, IC27 NCS21911SN2T1G, IC28 NCS21911SN2T1G, IC29 NCS21911SN2T1G, IC3 NCS21911SN2T1G, IC30 NCS21911SN2T1G, IC31 ADIS16500AMLZ, IC32 LTC6820IUD#PBF, IC33 CBTL01023GM,115, IC34 S35ML04G300WHI000, IC35 S35ML04G300WHI000, IC36 S35ML04G300WHI000, IC37 S35ML04G300WHI000, IC38 ADS8588HIPM, IC39 S35ML04G300WHI000, IC4 LTC4222CUH#PBF, IC40 S35ML04G300WHI000, IC41 S35ML04G300WHI000, IC42 S35ML04G300WHI000, IC43 S35ML04G300WHI000, IC44 S35ML04G300WHI000, IC45 S35ML04G300WHI000, IC46 S35ML04G300WHI000, IC47 S35ML04G300WHI000, IC48 S35ML04G300WHI000, IC49 S35ML04G300WHI000, IC5 LP38692SDX-5.0_NOPB, IC50 S35ML04G300WHI000, IC51 ADS8588HIPM, IC52 ADS8588HIPM, IC55 MUX36S16IRSNR, IC6 LP38692SDX-5.0_NOPB, IC7 LDL1117S33R, IC8 LDL1117S33R, IC9 LP38692SDX-5.0_NOPB, J1 SAMTEC-SMM-104-02-X-DJ, J2 SAMTEC-CLP-106-02-X-DJ, J4 TFM-120-02-L-D, J5 TFM-120-02-L-D, J6 TFM-120-02-L-D, J7 TFM-120-02-L-D, J8 TFM-120-02-L-D, J9 SSM-109-L-SV, M1 NTLUS4C12NTAG, M10 NTLUS4C12NTAG, M11 NTLUS4C12NTAG, M12 NTLUS4C12NTAG, M13 NTLUS4C12NTAG, M14 NTLUS4C12NTAG, M15 NTLUS4C12NTAG, M16 NTLUS4C12NTAG, M17 NTLUS4C12NTAG, M18 NTLUS4C12NTAG, M19 NTLUS4C12NTAG, M2 NTLUS4C12NTAG, M20 NTLUS4C12NTAG, M21 NTLUS4C12NTAG, M22 NTLUS4C12NTAG, M23 NTLUS4C12NTAG, M24 NTLUS4C12NTAG, M25 NTLUS4C12NTAG, M26 NTLUS4C12NTAG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

Commit message: Doing dangerous moves
Parts:
- moved R31 513.7 mm to (300.8, -14.4)
- moved R19 506.2 mm to (298.7, 43.8)
- moved R30 493.2 mm to (301.0, -10.0)
- moved C62 482.2 mm to (301.1, -17.3), turned to 90 degrees
- moved R29 472.2 mm to (301.0, -4.20)
- moved C61 457.5 mm to (301.3, -7.10), turned to 90 degrees
- moved R28 451.1 mm to (300.6, 0.59)
- moved C60 432.5 mm to (300.9, 3.52), turned to 90 degrees
- moved R27 430.2 mm to (300.6, 6.41)
- moved C59 407.0 mm to (300.0, 29.2), turned to 90 degrees
- moved R26 406.9 mm to (299.7, 26.2)
- moved R25 386.2 mm to (299.7, 32.0)
- moved C58 383.3 mm to (300.4, 15.6), turned to 90 degrees
- moved C89 382.5 mm to (299.1, -17.3), turned to 90 degrees
- moved C85 381.8 mm to (298.0, 29.1), turned to 90 degrees
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
Commit message: Dangerous maneuvers currently... Board reshaping
Parts:
- removed U$11, U$16: THROUGH_HOLE, SamacSys_Parts:1/16TH_BOLT
- moved C30 197.0 mm to (87.9, 58.3), turned to 90 degrees
- moved C29 193.3 mm to (80.3, 65.4), turned to 90 degrees
- moved C28 193.2 mm to (49.1, 61.6), turned to 90 degrees
- moved R58 189.5 mm to (76.9, 104.1)
- moved R57 186.6 mm to (76.9, 109.9)
- moved R70 179.1 mm to (87.6, 55.4)
- moved R69 176.2 mm to (87.6, 61.2)
- moved R68 173.8 mm to (80.0, 62.5)
- moved J1 173.8 mm to (179.1, 55.5)
- moved R67 170.9 mm to (80.0, 68.3)
- moved R66 170.8 mm to (48.9, 58.7)
- moved R65 167.6 mm to (48.8, 64.5)
- moved C31 160.4 mm to (92.9, 96.6), turned to 90 degrees
- moved R72 145.5 mm to (92.6, 93.7)
- moved R71 143.0 mm to (92.5, 99.5)
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
Commit message: New shrunken board
Parts:
- moved R148 495.7 mm to (154.4, -161.4), turned to 90 degrees
- moved D87 491.5 mm to (101.4, -135.7), turned to 90 degrees
- moved D80 490.9 mm to (95.0, -137.7), turned to 90 degrees
- moved R147 487.2 mm to (152.2, -155.5), turned to 90 degrees
- moved D79 486.0 mm to (91.3, -133.4), turned to 90 degrees
- moved C190 486.0 mm to (113.2, -131.3), turned to 90 degrees
- moved D86 485.8 mm to (97.9, -131.2), turned to 90 degrees
- moved C2 485.5 mm to (120.1, -131.3), turned to 90 degrees
- moved C6 483.8 mm to (101.7, -160.0), turned to 90 degrees
- moved C7 481.8 mm to (123.7, -160.0), turned to 90 degrees
- moved C4 481.8 mm to (144.4, -160.0), turned to 90 degrees
- moved C9 481.6 mm to (130.6, -160.0), turned to 90 degrees
- moved C10 481.6 mm to (137.5, -160.0), turned to 90 degrees
- moved D78 480.9 mm to (87.7, -128.9), turned to 90 degrees
- moved D85 480.1 mm to (94.3, -126.7), turned to 90 degrees
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Other:
- board size 259.8 x 281.7 mm -> 276.4 x 237 mm

Commit message: Connectors are moved to new locations, need to move mounting points
Parts:
- moved J1 5.36 mm to (182.1, 137.8)
- moved U$7 4.24 mm to (190.1, 4.45)
- moved C159 3.86 mm to (206.5, 112.5)
- moved C161 3.86 mm to (207.7, 109.9)
- moved D77 3.86 mm to (212.9, 93.2)
- moved LED64 3.86 mm to (197.7, 107.3)
- moved R403 3.86 mm to (204.3, 115.2)
- moved R404 3.86 mm to (205.3, 114.1)
- moved R406 3.86 mm to (203.3, 117.3)
- moved R409 3.86 mm to (200.5, 112.7)
- moved R410 3.86 mm to (201.7, 112.8)
- moved R415 3.86 mm to (205.7, 109.4)
- moved R416 3.86 mm to (206.7, 110.5)
- moved R419 3.86 mm to (200.3, 104.7)
- moved R421 3.86 mm to (201.7, 110.3)
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
Commit message: New board dimensions
Parts:
- moved U$10 7.23 mm to (110.6, 157.6)
Other:
- board size 276.4 x 237 mm -> 261.3 x 165.1 mm

Commit message: swapping
Parts:
- moved C24 265.8 mm to (90.2, 108.4), turned to 270 degrees
- moved C23 264.2 mm to (93.7, 108.4), turned to 270 degrees
- moved C196 263.0 mm to (97.0, 108.4), turned to 270 degrees
- moved C21 259.8 mm to (84.7, 104.6), turned to 180 degrees
- moved C20 257.0 mm to (84.7, 102.5), turned to 180 degrees
- moved C25 255.6 mm to (84.0, 100.5), turned to 180 degrees
- moved C17 252.2 mm to (84.0, 98.1), turned to 180 degrees
- moved C19 250.0 mm to (84.7, 96.0), turned to 180 degrees
- moved C14 195.4 mm to (100.1, 93.0)
- moved C10 185.8 mm to (80.8, 16.9), turned to 0 degrees
- moved C4 182.7 mm to (191.2, 16.6), flipped to the bottom, turned to 270 degrees
- moved C6 182.3 mm to (185.3, 2.03), flipped to the bottom
- moved C7 178.5 mm to (98.1, 16.7), turned to 0 degrees
- moved C9 171.3 mm to (98.0, 8.20), turned to 0 degrees
- moved C1 162.3 mm to (98.9, 12.2), turned to 0 degrees
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
Commit message: Doing power supply review now
Parts:
- moved D87 293.0 mm to (174.8, 148.0), turned to 270 degrees
- moved D86 290.6 mm to (178.3, 148.0), turned to 270 degrees
- moved D85 288.3 mm to (181.8, 148.0), turned to 270 degrees
- moved D84 286.3 mm to (185.3, 148.1), turned to 270 degrees
- moved D48 267.6 mm to (185.1, 126.4)
- moved D45 263.0 mm to (180.3, 126.5)
- moved R51 252.7 mm to (183.2, 144.2)
- moved R41 249.7 mm to (185.2, 144.2)
- moved D75 249.5 mm to (196.3, 98.5), turned to 0 degrees
- moved D78 247.8 mm to (196.3, 93.8), turned to 0 degrees
- moved D79 245.2 mm to (203.1, 84.8), turned to 270 degrees
- moved D80 245.0 mm to (197.7, 84.7), turned to 270 degrees
- moved R459 240.6 mm to (180.1, 125.5), flipped to the bottom
- moved D81 240.5 mm to (221.1, 86.1), turned to 270 degrees
- moved LED85 239.5 mm to (182.7, 127.5), flipped to the bottom, turned to 270 degrees
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
Commit message: Near done with layout
Parts:
- moved C195 292.2 mm to (136.8, 146.7), flipped to the bottom, turned to 0 degrees
- moved R504 288.0 mm to (134.2, 146.0), flipped to the bottom
- moved R503 286.2 mm to (139.7, 143.8), flipped to the bottom, turned to 270 degrees
- moved IC27 283.6 mm to (136.6, 143.5), flipped to the bottom
- moved R471 277.0 mm to (133.5, 143.0), flipped to the bottom, turned to 270 degrees
- moved U$1 270.4 mm to (136.6, 140.2), flipped to the bottom, turned to 180 degrees
- moved C194 261.7 mm to (217.9, 55.5), flipped to the bottom, turned to 180 degrees
- moved R502 260.9 mm to (220.8, 52.5), flipped to the bottom, turned to 270 degrees
- moved R505 258.6 mm to (215.3, 54.8), flipped to the bottom
- moved IC28 254.9 mm to (217.7, 52.3), flipped to the bottom
- moved R499 247.8 mm to (214.6, 52.1), flipped to the bottom
- moved U$2 242.4 mm to (217.8, 48.8), flipped to the bottom, turned to 180 degrees
- moved C169 223.8 mm to (148.8, 109.4), flipped to the bottom, turned to 270 degrees
- moved LED83 194.8 mm to (196.9, 113.8), flipped to the bottom
- moved R457 194.7 mm to (202.7, 112.3), turned to 180 degrees
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