File: thermo_final.brd (EAGLE design)
At the start: 7.9 x 13.4 mm, 109 parts, among them IC1 DG4051EEQ-T1-GE3, IC10 LDL1117S33R, IC2 DG4051EEQ-T1-GE3, IC3 D-type, IC4 LTC6820IUD#PBF, IC5 MAX6675ISA+, IC6 AND1, IC7 INVERTER, IC8 AND2, IC9 OR, J1 PCC-SMD-20, J2 PCC-SMD-20, J3 PCC-SMD-20, J4 PCC-SMD-20, J5 PCC-SMD-20, J6 PCC-SMD-20, J7 PCC-SMD-20, J8 PCC-SMD-20, T1 782482_33VC

Commit message: ready for routing
Parts:
- removed IC10: LDL1117S33R, SamacSys_Parts:SOT230P700X180-4N
- removed IC3: D-type, SamacSys_Parts:SOIC127P1032X265-20N
- removed IC4: LTC6820IUD#PBF, SamacSys_Parts:QFN50P300X300X80-17N
- removed IC6: AND1, SamacSys_Parts:SOIC127P600X175-14N
- removed IC7: INVERTER, SamacSys_Parts:SOIC127P600X175-14N
- removed IC8: AND2, SamacSys_Parts:SOIC127P600X175-14N
- removed IC9: OR, SamacSys_Parts:SOIC127P600X175-14N
- removed J1, J2, J4, J5, J6, J7, J8: PCC-SMD-20, PCC-SMD-20:OMEGA_PCC-SMD-20
- removed LED10, LED11, LED12, LED13, LED14, LED2, LED4, LED5, LED6, LED7, LED8, LED9: AA3021LSYSK_J3-TR, SamacSys_Parts:AA3021LSYSKJ3TR
- removed LED15, LED16, LED17: APTD1608LCGCK, SamacSys_Parts:APT1608CGCK
- removed PS1: XC6901D331MR-G, SamacSys_Parts:SOT95P280X130-5N
- removed PS2: TMR_6-2422WIR, SamacSys_Parts:TMR67212WIR
- removed TP10, TP11, TP2, TP3, TP4, TP5, TP8, TP9: S1751-46R, SamacSys_Parts:S175146R
- added AND1: AND1, SamacSys_Parts:SOIC127P600X175-14N
- added AND2: AND2, SamacSys_Parts:SOIC127P600X175-14N
- added CONNECTOR_0, CONNECTOR_1, CONNECTOR_2, CONNECTOR_4, CONNECTOR_5, CONNECTOR_6, CONNECTOR_7: PCC-SMD-20, PCC-SMD-20:OMEGA_PCC-SMD-20
- added D-TYPE: D-type, SamacSys_Parts:SOIC127P1032X265-20N
- added INVERTER: INVERTER, SamacSys_Parts:SOIC127P600X175-14N
- added LED_-3.3V, LED_12V, LED_3.3V, LED_Q0, LED_Q1, LED_Q2, LED_Q3, LED_Q4, LED_Q5, LED_Q6, LED_Q7, LED_SCK: AA3021LSYSK_J3-TR, SamacSys_Parts:AA3021LSYSKJ3TR
- added LED_A0, LED_A1, LED_A2: APTD1608LCGCK, SamacSys_Parts:APT1608CGCK
- added OR: OR, SamacSys_Parts:SOIC127P600X175-14N
- added PS_-3.3V: XC6901D331MR-G, SamacSys_Parts:SOT95P280X130-5N
- added PS_12V: TMR_6-2422WIR, SamacSys_Parts:TMR67212WIR
- added PS_3.3V: LDL1117S33R, SamacSys_Parts:SOT230P700X180-4N
- added SPI: LTC6820IUD#PBF, SamacSys_Parts:QFN50P300X300X80-17N
- added TEST_CLK, TEST_CS, TEST_GND1, TEST_GND2, TEST_GND3, TEST_GND4, TEST_MISO, TEST_SCK: S1751-46R, SamacSys_Parts:S175146R
- moved R26 138.7 mm to (81.2, 3.68), flipped to the bottom, turned to 90 degrees
- moved R25 132.7 mm to (81.2, 0.64), turned to 90 degrees
- moved R24 128.7 mm to (81.2, -2.92), turned to 90 degrees
- moved R20 118.3 mm to (47.6, 4.57), turned to 90 degrees
- moved R2 114.5 mm to (72.5, 21.7), turned to 270 degrees
- moved R1 114.4 mm to (72.5, 18.9), turned to 270 degrees
- moved R27 110.9 mm to (81.2, 6.99), turned to 270 degrees
- moved R18 103.5 mm to (74.8, 29.0), turned to 270 degrees
- moved R30 101.5 mm to (61.7, 21.1), turned to 270 degrees
- moved R29 98.2 mm to (64.8, 21.1), turned to 270 degrees
- moved R23 34.6 mm to (47.8, -3.17), turned to 270 degrees
- moved R13 19.3 mm to (37.7, 14.7), flipped to the top, turned to 270 degrees
- moved D8 9.03 mm to (102.1, -18.9)
- moved D16 9.03 mm to (102.1, -1.14)
- moved C3 8.92 mm to (57.9, 37.7), flipped to the bottom
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- renumbered J3 to CONNECTOR_3, LED1 to LED_MISO, LED3 to LED_CS, TP1 to TEST_CJ+, TP7 to TEST_CJ-
Connections:
- net !CS: now also AND1.2, INVERTER.2; no longer IC6.2, IC7.2
- net !Q1: now also AND1.5, INVERTER.6; no longer IC6.5, IC7.6
- net !Q3: now also AND1.10, AND2.2, INVERTER.8; no longer IC6.10, IC7.8, IC8.2
- net !Q5: now also AND1.13, INVERTER.10; no longer IC6.13, IC7.10
- net !Q7: now also AND2.5, D-TYPE.1, INVERTER.12, INVERTER.4; no longer IC3.1, IC7.12, IC7.4, IC8.5
- net -VCC: now also LED_-3.3V.1, PS_-3.3V.5; no longer LED5.1, PS1.5
- net A1: now also LED_A1.1, OR.3; no longer IC9.3, LED16.1
- net A2: now also LED_A2.1, OR.11; no longer IC9.11, LED17.1
- net CLK: now also AND1.3, D-TYPE.11, TEST_CLK.1; no longer IC3.11, IC6.3, TP3.1
- net CS: now also AND1.1, D-TYPE.3, INVERTER.1, SPI.4, TEST_CS.1; no longer IC3.3, IC4.4, IC6.1, IC7.1, TP2.1
- net GND: now also AND1.7, AND2.10, AND2.11, AND2.12, AND2.13, AND2.7, AND2.8, AND2.9, D-TYPE.10, INVERTER.7, OR.7, PS_-3.3V.1, PS_12V.1, PS_12V.3, PS_12V.7, PS_3.3V.1, SPI.11, SPI.13, SPI.17, TEST_GND1.1, TEST_GND2.1, TEST_GND3.1, TEST_GND4.1; no longer IC10.1, IC3.10, IC4.11, IC4.13, IC4.17, IC6.7, IC7.7, IC8.10, IC8.11, IC8.12, IC8.13, IC8.7, IC8.8, IC8.9, IC9.7, PS1.1, PS2.1, PS2.3, PS2.7, TP10.1, TP11.1, TP8.1, TP9.1
- net IM: now also SPI.9; no longer IC4.9
- net IP: now also SPI.10; no longer IC4.10
- net MISO: now also SPI.2, TEST_MISO.1; no longer IC4.2, TP4.1
- net N$11: now also SPI.15; no longer IC4.15
- net N$12: now also LED_Q1.1; no longer LED8.1
- net N$16: now also LED_Q2.1; no longer LED9.1
- net N$17: now also LED_Q3.1; no longer LED10.1
- net N$2: now also LED_12V.1; no longer LED6.1
- net N$22: now also SPI.1; no longer IC4.1
- net N$23: now also LED_SCK.2; no longer LED2.2
- net N$25: now also LED_3.3V.1; no longer LED4.1
- net N$26: now also LED_-3.3V.2; no longer LED5.2
- net N$27: now also LED_Q4.1; no longer LED11.1
- net N$28: now also LED_Q5.1; no longer LED12.1
- net N$29: now also LED_Q6.1; no longer LED13.1
- net N$30: now also LED_Q7.1; no longer LED14.1
- net N$34: now also LED_A0.2; no longer LED15.2
- net N$35: now also LED_A1.2; no longer LED16.2
- net N$36: now also LED_A2.2; no longer LED17.2
- net N$6: now also SPI.14; no longer IC4.14
- net N$7: now also LED_Q0.1; no longer LED7.1
- net OR1: now also OR.12, OR.6; no longer IC9.12, IC9.6
- net OR2: now also OR.13, OR.8; no longer IC9.13, IC9.8
- net Q0: now also AND1.4, D-TYPE.2, D-TYPE.4, LED_Q0.2; no longer IC3.2, IC3.4, IC6.4, LED7.2
- net Q0!Q1: now also AND1.6, OR.4; no longer IC6.6, IC9.4
- net Q1: now also AND2.1, D-TYPE.5, D-TYPE.7, INVERTER.5, LED_Q1.2; no longer IC3.5, IC3.7, IC7.5, IC8.1, LED8.2
- net Q1!Q3: now also AND2.3, OR.1; no longer IC8.3, IC9.1
- net Q2: now also AND1.9, D-TYPE.6, D-TYPE.8, LED_Q2.2; no longer IC3.6, IC3.8, IC6.9, LED9.2
- net Q2!Q3: now also AND1.8, OR.5; no longer IC6.8, IC9.5
- net Q3: now also D-TYPE.13, D-TYPE.9, INVERTER.9, LED_A0.1, LED_Q3.2; no longer IC3.13, IC3.9, IC7.9, LED10.2, LED15.1
- net Q4: now also AND1.12, D-TYPE.12, D-TYPE.14, LED_Q4.2; no longer IC3.12, IC3.14, IC6.12, LED11.2
- net Q4!Q5: now also AND1.11, OR.9; no longer IC6.11, IC9.9
- net Q5: now also AND2.4, D-TYPE.15, D-TYPE.17, INVERTER.11, LED_Q5.2; no longer IC3.15, IC3.17, IC7.11, IC8.4, LED12.2
- net Q5!Q7: now also AND2.6, OR.2; no longer IC8.6, IC9.2
- net Q6: now also D-TYPE.16, D-TYPE.18, LED_Q6.2, OR.10; no longer IC3.16, IC3.18, IC9.10, LED13.2
- net Q7: now also D-TYPE.19, INVERTER.13, INVERTER.3, LED_Q7.2; no longer IC3.19, IC7.13, IC7.3, LED14.2
- net SCK: now also LED_SCK.1, SPI.3, TEST_SCK.1; no longer IC4.3, LED2.1, TP5.1
- net T0+: now also CONNECTOR_0.1; no longer J7.1
- net T0-: now also CONNECTOR_0.2; no longer J7.2
- net T1+: now also CONNECTOR_1.1; no longer J1.1
- net T1-: now also CONNECTOR_1.2; no longer J1.2
- net T2+: now also CONNECTOR_2.1; no longer J2.1
- net T2-: now also CONNECTOR_2.2; no longer J2.2
- net T4+: now also CONNECTOR_4.1; no longer J4.1
- net T4-: now also CONNECTOR_4.2; no longer J4.2
- net T5+: now also CONNECTOR_5.1; no longer J5.1
- net T5-: now also CONNECTOR_5.2; no longer J5.2
- net T6+: now also CONNECTOR_6.1; no longer J6.1
- net T6-: now also CONNECTOR_6.2; no longer J6.2
- net T7+: now also CONNECTOR_7.1; no longer J8.1
- net T7-: now also CONNECTOR_7.2; no longer J8.2
- net V+: now also PS_12V.6, PS_3.3V.3; no longer IC10.3, PS2.6
- net V-: now also PS_-3.3V.2, PS_12V.8; no longer PS1.2, PS2.8
- net VCC: now also AND1.14, AND2.14, D-TYPE.20, INVERTER.14, LED_3.3V.2, OR.14, PS_-3.3V.3, PS_3.3V.2, PS_3.3V.4, SPI.12, SPI.16, SPI.5, SPI.6, SPI.7, SPI.8; no longer IC10.2, IC10.4, IC3.20, IC4.12, IC4.16, IC4.5, IC4.6, IC4.7, IC4.8, IC6.14, IC7.14, IC8.14, IC9.14, LED4.2, PS1.3
- net VDD: now also LED_12V.2, PS_12V.2; no longer LED6.2, PS2.2

Commit message: routing save
Parts:
- removed T1: 782482_33VC, SamacSys_Parts:DIP1016W60P254L914H635Q6N
- added TRANSFORMER: 782482_33VC, SamacSys_Parts:DIP1016W60P254L914H635Q6N
- moved TEST_GND4 49.3 mm to (38.1, 0.00)
- moved TEST_MISO 38.2 mm to (86.1, 29.5), turned to 0 degrees
- moved TEST_GND3 31.4 mm to (68.6, 22.9)
- moved R13 21.5 mm to (56.5, 25.1), turned to 90 degrees
- moved R28 19.0 mm to (51.1, 12.2), turned to 0 degrees
- moved LED_SCK 14.3 mm to (53.5, 23.2), turned to 90 degrees
- moved LED_A0 14.2 mm to (54.6, 12.2), turned to 180 degrees
- moved OR 13.5 mm to (86.6, -14.1), turned to 90 degrees
- moved R29 12.4 mm to (52.7, 18.4), turned to 0 degrees
- moved D1 9.25 mm to (69.8, 56.6)
- moved D2 9.25 mm to (84.2, 56.6)
- moved D3 9.25 mm to (74.4, 56.6)
- moved JP3 9.25 mm to (77.1, 62.5)
- moved R36 9.25 mm to (67.4, 53.1)
- moved R37 9.25 mm to (69.8, 52.6)
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Connections:
- net IM: now also TRANSFORMER.3; no longer T1.3
- net IMOUT: now also TRANSFORMER.4; no longer T1.4
- net IP: now also TRANSFORMER.1; no longer T1.1
- net IPOUT: now also TRANSFORMER.6; no longer T1.6
- net N$10: now also TRANSFORMER.2; no longer T1.2
- net N$14: now also TRANSFORMER.5; no longer T1.5
Routing:
- net Q3: track 0.00 -> 132.2 mm, vias 0 -> 8
- net CS: track 0.00 -> 113.1 mm, vias 0 -> 4
- net Q1: track 0.00 -> 96.5 mm, vias 0 -> 5
- net T3+: track 0.00 -> 85.6 mm, vias 0 -> 2
- net Q7: track 0.00 -> 84.5 mm, vias 0 -> 3
- net T2-: track 0.00 -> 83.3 mm, vias 0 -> 3
- net T1-: track 0.00 -> 83.3 mm, vias 0 -> 9
- net !Q7: track 0.00 -> 81.8 mm, vias 0 -> 4
- net A1: track 0.00 -> 81.3 mm, vias 0 -> 4
- net T5-: track 0.00 -> 80.0 mm, vias 0 -> 3
- net T7-: track 0.00 -> 73.9 mm, vias 0 -> 1
- net T3-: track 0.00 -> 73.7 mm, vias 0 -> 3
- net !Q3: track 0.00 -> 72.5 mm, vias 0 -> 9
- net Q5: track 0.00 -> 72.1 mm, vias 0 -> 4
- net T0-: track 0.00 -> 71.1 mm, vias 0 -> 7
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- added copper zone on layer 1, net GND
Other:
- board size 7.9 x 13.4 mm -> 82.5 x 88.9 mm

Commit message: final routing for the night
Parts:
- moved C8 4.62 mm to (42.8, 20.4), turned to 0 degrees
- moved TEST_CS 1.66 mm to (42.0, 23.2)
- moved R14 0.74 mm to (42.5, 13.7)
- moved R15 0.72 mm to (38.2, 13.7)
- moved R3 0.63 mm to (40.4, 18.3)
Connections:
- removed net N$6: SPI.14
- net N$5: now also SPI.14
Routing:
- net VCC: track 48.8 -> 256.0 mm, vias 7 -> 16
- net MISO: track 4.47 -> 65.0 mm, vias 0 -> 5
- net -VCC: track 0.00 -> 48.0 mm, vias 0 -> 5
- net VDD: track 13.3 -> 48.7 mm
- net N$5: track 2.42 -> 7.61 mm
- net CS: track 113.1 -> 116.4 mm
- net N$26: track 0.00 -> 2.79 mm
- net T3-: track 73.7 -> 75.3 mm
- net !Q3: track 72.5 -> 74.0 mm
- net V-: track 1.74 -> 3.28 mm
- net GND: track 5.54 -> 4.17 mm
- net A1: track 81.3 -> 82.4 mm
- net T5-: track 80.0 -> 81.0 mm
- net Q3: track 132.2 -> 133.1 mm
- net Q1!Q3: track 21.7 -> 22.4 mm
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- added copper zone on layer 16, net GND

Commit message: gawd I hope I'm right...
Parts:
- moved TEST_GND4 80.0 mm to (49.8, 79.2), turned to 90 degrees
- moved R24 69.0 mm to (20.4, 28.9), flipped to the bottom
- moved C10 67.2 mm to (26.8, 66.2), flipped to the bottom, turned to 0 degrees
- moved R25 65.8 mm to (20.4, 24.5), flipped to the bottom
- moved OR 65.1 mm to (25.1, 7.42), flipped to the bottom
- moved R26 63.6 mm to (20.4, 20.3)
- moved TRANSFORMER 63.4 mm to (23.9, 66.3)
- moved LED_Q4 63.1 mm to (22.7, 29.5), turned to 0 degrees
- moved R38 62.7 mm to (27.5, 74.4), flipped to the bottom, turned to 270 degrees
- moved R27 62.1 mm to (20.4, 16.3), flipped to the bottom, turned to 90 degrees
- moved D2 60.7 mm to (27.5, 78.3)
- moved JP2 60.7 mm to (27.5, 83.9)
- moved C9 59.6 mm to (20.9, 66.3), flipped to the bottom, turned to 0 degrees
- moved TEST_GND2 59.5 mm to (51.8, 53.4)
- moved D20 59.4 mm to (24.2, 78.1)
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Connections:
- net !Q7: no longer INVERTER.4
- net GND: now also INVERTER.3, INVERTER.4
- net Q7: no longer INVERTER.3
Routing:
- net VCC: track 256.0 -> 0.00 mm, vias 16 -> 0
- net Q3: track 133.1 -> 45.3 mm, vias 8 -> 5
- net A1: track 82.4 -> 0.00 mm, vias 4 -> 0
- net CS: track 116.4 -> 35.9 mm, vias 4 -> 1
- net MISO: track 65.0 -> 0.00 mm, vias 5 -> 0
- net A2: track 59.9 -> 0.00 mm, vias 2 -> 0
- net Q7: track 84.5 -> 27.0 mm, vias 3 -> 2
- net VDD: track 48.7 -> 0.00 mm
- net -VCC: track 48.0 -> 0.00 mm, vias 5 -> 0
- net !Q7: track 81.8 -> 34.6 mm, vias 4 -> 6
- net !Q3: track 74.0 -> 27.7 mm, vias 9 -> 4
- net Q1: track 96.5 -> 52.8 mm, vias 5 -> 6
- net T1-: track 83.2 -> 42.0 mm, vias 9 -> 2
- net T0-: track 71.1 -> 40.8 mm, vias 7 -> 2
- net CLK: track 29.6 -> 0.00 mm, vias 4 -> 0
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Other:
- board size 82.5 x 88.9 mm -> 70.4 x 88.9 mm

Commit message: gawd I hope I'm right pt 2...
Parts:
- moved R15 1.12 mm to (22.0, 47.3)
- moved R5 1.07 mm to (29.2, 47.9)
- moved R39 0.95 mm to (28.9, 74.9), flipped to the top
- moved R36 0.89 mm to (14.3, 74.7), flipped to the top
- moved R38 0.71 mm to (26.8, 74.4), flipped to the top
- moved R37 0.59 mm to (16.4, 74.0), flipped to the top
- moved R13 0.15 mm to (46.0, 48.7), turned to 180 degrees
Routing:
- net CS: track 35.9 -> 158.0 mm, vias 1 -> 9
- net MISO: track 0.00 -> 68.1 mm, vias 0 -> 7
- net SCK: track 0.00 -> 66.8 mm, vias 0 -> 4
- net A1: track 0.00 -> 65.2 mm, vias 0 -> 5
- net CJ-: track 0.00 -> 54.4 mm, vias 0 -> 4
- net Q3: track 45.3 -> 90.9 mm, vias 5 -> 10
- net A2: track 0.00 -> 43.9 mm, vias 0 -> 2
- net CLK: track 0.00 -> 43.5 mm, vias 0 -> 3
- net VCC: track 0.00 -> 35.4 mm, vias 0 -> 4
- net CJ+: track 0.00 -> 33.2 mm, vias 0 -> 5
- net VDD: track 0.00 -> 32.2 mm, vias 0 -> 1
- net IP: track 0.00 -> 28.7 mm, vias 0 -> 2
- net IM: track 0.00 -> 21.7 mm, vias 0 -> 2
- net IPOUT: track 0.00 -> 19.0 mm
- net -VCC: track 0.00 -> 14.5 mm, vias 0 -> 1
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
Commit message: Final routing
Parts:
- moved D2 6.21 mm to (33.6, 79.5), turned to 0 degrees
- moved JP2 4.75 mm to (32.3, 83.9)
- moved D20 4.44 mm to (28.3, 79.6), turned to 0 degrees
- moved JP3 2.80 mm to (24.4, 84.0)
- moved LED_12V 2.36 mm to (39.2, 79.3)
- moved R19 2.36 mm to (39.2, 79.8)
- moved D3 2.23 mm to (20.5, 79.7), turned to 180 degrees
- moved R36 1.60 mm to (15.0, 76.2)
- moved R37 1.60 mm to (17.0, 75.5)
- moved D1 1.49 mm to (15.4, 79.7), turned to 180 degrees
- moved D10 1.05 mm to (4.34, 64.1)
- moved CONNECTOR_0 1.05 mm to (6.12, 55.1)
- moved CONNECTOR_1 1.05 mm to (6.12, 33.7)
- moved CONNECTOR_2 1.05 mm to (6.12, 12.2)
- moved D18 1.05 mm to (4.34, 46.2)
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Connections:
- removed net N$8: D1.2, JP1.1
- removed net N$9: D2.2, JP2.1
- net CS: no longer D20.2
- net GND: now also D1.2, D2.2, D20.2, D3.2
- net N$37: now also JP1.1
- net N$40: now also JP2.1
- net VDD: no longer D3.2
Routing:
- net VCC: track 35.4 -> 181.1 mm, vias 4 -> 17
- net V+: track 6.78 -> 67.5 mm, vias 1 -> 4
- net CS: track 158.0 -> 199.6 mm, vias 9 -> 11
- net V-: track 6.92 -> 38.8 mm, vias 1 -> 2
- net N$40: track 3.82 -> 15.3 mm
- net N$37: track 4.14 -> 9.75 mm
- net N$9: track 4.19 -> 0.00 mm
- net N$8: track 4.19 -> 0.00 mm
- net N$11: track 5.94 -> 8.32 mm
- net IPOUT: track 19.0 -> 20.1 mm
- net T3-: track 50.7 -> 49.8 mm
- net T0-: track 40.7 -> 39.7 mm
- net T0+: track 50.4 -> 49.5 mm
- net T2+: track 37.8 -> 36.9 mm
- net T1-: track 42.1 -> 41.3 mm
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Other:
- board size 70.4 x 88.9 mm -> 69.4 x 89 mm

Commit message: Board Complete
Parts:
- removed IC1, IC2: DG4051EEQ-T1-GE3, SamacSys_Parts:SOP65P640X120-16N
- added MUX+, MUX-: DG4051EEQ-T1-GE3, SamacSys_Parts:SOP65P640X120-16N
- moved D14 2.74 mm to (64.4, 64.4)
- moved CONNECTOR_4 2.74 mm to (62.7, 12.2)
- moved CONNECTOR_5 2.74 mm to (62.7, 77.0)
- moved CONNECTOR_6 2.74 mm to (62.7, 34.0)
- moved CONNECTOR_7 2.74 mm to (62.7, 55.4)
- moved D12 2.74 mm to (64.4, 86.0)
- moved D13 2.74 mm to (64.4, 43.1)
- moved D16 2.74 mm to (64.4, 21.1)
- moved D4 2.74 mm to (64.4, 68.2)
- moved D5 2.74 mm to (64.4, 25.2)
- moved D6 2.74 mm to (64.4, 46.7)
- moved D8 2.74 mm to (64.4, 3.35)
- moved C3 1.06 mm to (46.6, 69.1)
- moved C4 1.06 mm to (50.4, 69.1)
- moved JP2 1.06 mm to (31.2, 84.1)
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Connections:
- net -VCC: now also MUX+.7, MUX-.7; no longer IC1.7, IC2.7
- net A1: now also MUX+.10, MUX-.10; no longer IC1.10, IC2.10
- net A2: now also MUX+.9, MUX-.9; no longer IC1.9, IC2.9
- net CJ+: now also MUX+.3; no longer IC1.3
- net CJ-: now also MUX-.3; no longer IC2.3
- net GND: now also MUX+.8, MUX-.8; no longer IC1.8, IC2.8
- net Q3: now also MUX+.11, MUX-.11; no longer IC1.11, IC2.11
- net T0+: now also MUX+.13; no longer IC1.13
- net T0-: now also MUX-.13; no longer IC2.13
- net T1+: now also MUX+.14; no longer IC1.14
- net T1-: now also MUX-.14; no longer IC2.14
- net T2+: now also MUX+.15; no longer IC1.15
- net T2-: now also MUX-.15; no longer IC2.15
- net T3+: now also MUX+.12; no longer IC1.12
- net T3-: now also MUX-.12; no longer IC2.12
- net T4+: now also MUX+.1; no longer IC1.1
- net T4-: now also MUX-.1; no longer IC2.1
- net T5+: now also MUX+.5; no longer IC1.5
- net T5-: now also MUX-.5; no longer IC2.5
- net T6+: now also MUX+.2; no longer IC1.2
- net T6-: now also MUX-.2; no longer IC2.2
- net T7+: now also MUX+.4; no longer IC1.4
- net T7-: now also MUX-.4; no longer IC2.4
- net VCC: now also MUX+.16, MUX+.6, MUX-.16, MUX-.6; no longer IC1.16, IC1.6, IC2.16, IC2.6
Routing:
- net VCC: track 181.1 -> 248.7 mm, vias 17 -> 21
- net -VCC: track 14.5 -> 33.2 mm, vias 1 -> 3
- net T4-: track 43.8 -> 42.1 mm
- net T7+: track 32.1 -> 30.4 mm
- net T6+: track 33.5 -> 32.0 mm
- net T4+: track 52.6 -> 51.2 mm
- net T6-: track 36.8 -> 35.4 mm
- net T5-: track 72.9 -> 71.6 mm
- net Q3: track 90.9 -> 92.2 mm
- net T3+: track 69.4 -> 70.6 mm
- net N$40: track 15.3 -> 14.6 mm
- net VDD: track 32.6 -> 32.0 mm
- net T5+: track 47.3 -> 46.7 mm
Other:
- board size 69.4 x 89 mm -> 67.8 x 89 mm
- board text added: "Ethan Edwards Baja SAE WAGMI"
