File: thermo_final.sch (EAGLE design)
At the start: 115 parts, among them IC1 DG4051EEQ-T1-GE3, IC10 LDL1117S33R, IC2 DG4051EEQ-T1-GE3, IC3 D-type, IC4 LTC6820IUD#PBF, IC5 MAX6675ISA+, IC6 AND1, IC7 INVERTER, IC8 AND2, IC9 OR, J1 PCC-SMD-20, J2 PCC-SMD-20, J3 PCC-SMD-20, J4 PCC-SMD-20, J5 PCC-SMD-20, J6 PCC-SMD-20, J7 PCC-SMD-20, J8 PCC-SMD-20, T1 782482_33VC

Commit message: update layout
Parts:
- removed 3.3K: RC0402JR-133K3L, SamacSys_Parts:RC0402JR-133K3L
- removed R10, R11, R12, R6, R7, R9: 0, SamacSys_Parts:CRG0402ZR
- added D20: PTVS12VS1UR,115, SamacSys_Parts:PTVS12VS1UR,115
- R4, R5: value 0 -> 3.3K; device SamacSys_Parts:CRG0402ZR -> SamacSys_Parts:RC0402JR-133K3L
Connections:
- removed net N$13: R9.1, T1.SECONDARY_3
- removed net N$15: R12.1, T1.SECONDARY_1
- removed net N$33: R30.1
- net CS: now also D20.A, D20.K
- net GND: now also R30.1; no longer D1.A, D2.A, D3.A
- net IM: now also T1.PRIMARY_3; no longer R6.1, R7.1
- net IMOUT: now also T1.SECONDARY_1; no longer R11.2, R12.2
- net IP: now also T1.PRIMARY_1; no longer R4.1, R5.1
- net IPOUT: now also T1.SECONDARY_3; no longer R10.2, R9.2
- net MISO: now also R4.1
- net N$10: no longer R5.2, R6.2
- net N$14: no longer R10.1, R11.1
- net N$22: now also R5.2; no longer 3.3K.2
- net N$37: now also D1.K; no longer JP1.1
- net N$40: now also D2.K; no longer JP2.1
- net N$8: now also D1.A, JP1.1; no longer R4.2, T1.PRIMARY_1
- net N$9: now also D2.A, JP2.1; no longer R7.2, T1.PRIMARY_3
- net T4+: no longer D3.K
- net T5+: no longer D1.K
- net V+: no longer IC10.VOUT_2
- net VCC: now also IC10.VOUT_2, R4.2, R5.1; no longer 3.3K.1
- net VDD: now also D3.A, D3.K; no longer D2.K
Other:
- moved on the sheet: D1, D2, D3, R36, R37, R38, R39, R4, R5

Commit message: ready for routing
Parts:
- renumbered IC10 to PS_3.3V, IC3 to D-TYPE, IC4 to SPI, IC6 to AND1, IC7 to INVERTER, IC8 to AND2, IC9 to OR, J1 to CONNECTOR_1, J2 to CONNECTOR_2, J3 to CONNECTOR_3, J4 to CONNECTOR_4, J5 to CONNECTOR_5, J6 to CONNECTOR_6, J7 to CONNECTOR_0, J8 to CONNECTOR_7, LED1 to LED_MISO, LED10 to LED_Q3, LED11 to LED_Q4, LED12 to LED_Q5, LED13 to LED_Q6, LED14 to LED_Q7, LED15 to LED_A0, LED16 to LED_A1, LED17 to LED_A2, LED2 to LED_SCK, LED3 to LED_CS, LED4 to LED_3.3V, LED5 to LED_-3.3V, LED6 to LED_12V, LED7 to LED_Q0, LED8 to LED_Q1, LED9 to LED_Q2, PS1 to PS_-3.3V, PS2 to PS_12V, TP1 to TEST_CJ+, TP10 to TEST_GND3, TP11 to TEST_GND4, TP2 to TEST_CS, TP3 to TEST_CLK, TP4 to TEST_MISO, TP5 to TEST_SCK, TP7 to TEST_CJ-, TP8 to TEST_GND1, TP9 to TEST_GND2

Commit message: routing save
Parts:
- renumbered T1 to TRANSFORMER
Changed lines of the file:
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@@
 <part name="CONNECTOR_0" library="PCC-SMD-20" deviceset="PCC-SMD-20" device=""/>
 <part name="CONNECTOR_7" library="PCC-SMD-20" deviceset="PCC-SMD-20" device=""/>
-<part name="T1" library="SamacSys_Parts" deviceset="782482_33VC" device=""/>
+<part name="TRANSFORMER" library="SamacSys_Parts" deviceset="782482_33VC" device=""/>
 <part name="D4" library="SamacSys_Parts" deviceset="PTVS12VS1UR,115" device=""/>
 <part name="D5" library="SamacSys_Parts" deviceset="PTVS12VS1UR,115" device=""/>
@@
 <attribute name="VALUE" x="-55.88" y="-68.58" size="1.778" layer="96"/>
 </instance>
-<instance part="T1" gate="G$1" x="279.4" y="93.98" smashed="yes">
+<instance part="TRANSFORMER" gate="G$1" x="279.4" y="93.98" smashed="yes">
 <attribute name="NAME" x="295.91" y="101.6" size="1.778" layer="95" align="center-left"/>
 <attribute name="VALUE" x="295.91" y="99.06" size="1.778" layer="96" align="center-left"/>
@@
 </segment>
 <segment>
-<pinref part="T1" gate="G$1" pin="PRIMARY_1"/>
+<pinref part="TRANSFORMER" gate="G$1" pin="PRIMARY_1"/>
 <wire x1="279.4" y1="93.98" x2="269.24" y2="93.98" width="0.1524" layer="91"/>
 <label x="266.7" y="93.98" size="1.778" layer="95"/>
@@
 </segment>
 <segment>
-<pinref part="T1" gate="G$1" pin="PRIMARY_3"/>
+<pinref part="TRANSFORMER" gate="G$1" pin="PRIMARY_3"/>
 <wire x1="279.4" y1="88.9" x2="269.24" y2="88.9" width="0.1524" layer="91"/>
 <label x="266.7" y="88.9" size="1.778" layer="95"/>
@@
 <net name="N$10" class="0">
 <segment>
-<pinref part="T1" gate="G$1" pin="PRIMARY_2"/>
+<pinref part="TRANSFORMER" gate="G$1" pin="PRIMARY_2"/>
 <wire x1="279.4" y1="91.44" x2="251.46" y2="91.44" width="0.1524" layer="91"/>
 <pinref part="C9" gate="G$1" pin="2"/>
@@
 <net name="N$14" class="0">
 <segment>
-<pinref part="T1" gate="G$1" pin="SECONDARY_2"/>
+<pinref part="TRANSFORMER" gate="G$1" pin="SECONDARY_2"/>
 <wire x1="322.58" y1="91.44" x2="350.52" y2="91.44" width="0.1524" layer="91"/>
 <pinref part="C10" gate="G$1" pin="1"/>
@@
 </segment>
 <segment>
-<pinref part="T1" gate="G$1" pin="SECONDARY_3"/>
+<pinref part="TRANSFORMER" gate="G$1" pin="SECONDARY_3"/>
 <wire x1="322.58" y1="93.98" x2="332.74" y2="93.98" width="0.1524" layer="91"/>
 <label x="332.74" y="93.98" size="1.778" layer="95"/>
@@
 </segment>
 <segment>
-<pinref part="T1" gate="G$1" pin="SECONDARY_1"/>
+<pinref part="TRANSFORMER" gate="G$1" pin="SECONDARY_1"/>
 <wire x1="322.58" y1="88.9" x2="332.74" y2="88.9" width="0.1524" layer="91"/>
 <label x="332.74" y="88.9" size="1.778" layer="95"/>

Commit message: final routing for the night
Connections:
- removed net N$6: SPI.ICMP
- net N$5: now also SPI.ICMP
Changed lines of the file:
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@@
 <pinref part="R15" gate="G$1" pin="1"/>
+</segment>
+<segment>
+<pinref part="SPI" gate="G$1" pin="ICMP"/>
+<wire x1="254" y1="33.02" x2="254" y2="45.72" width="0.1524" layer="91"/>
+<wire x1="274.32" y1="53.34" x2="274.32" y2="45.72" width="0.1524" layer="91"/>
+<wire x1="254" y1="45.72" x2="274.32" y2="45.72" width="0.1524" layer="91"/>
+<label x="272.288" y="53.848" size="1.778" layer="95"/>
 </segment>
 </net>
@@
 </segment>
 </net>
-<net name="N$6" class="0">
-<segment>
-<pinref part="SPI" gate="G$1" pin="ICMP"/>
-<wire x1="254" y1="33.02" x2="254" y2="45.72" width="0.1524" layer="91"/>
-<wire x1="274.32" y1="53.34" x2="274.32" y2="45.72" width="0.1524" layer="91"/>
-<wire x1="254" y1="45.72" x2="274.32" y2="45.72" width="0.1524" layer="91"/>
-</segment>
-</net>

Commit message: gawd I hope I'm right...
Connections:
- net !Q7: no longer INVERTER.2Y
- net GND: now also INVERTER.2A, INVERTER.2Y
- net Q7: no longer INVERTER.2A
Changed lines of the file:
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@@
 <setting verticaltext="up"/>
 </settings>
-<grid distance="0.1" unitdist="inch" unit="inch" style="lines" multiple="1" display="yes" altdistance="0.01" altunitdist="inch" altunit="inch"/>
+<grid distance="0.1" unitdist="inch" unit="inch" style="lines" multiple="1" display="no" altdistance="0.01" altunitdist="inch" altunit="inch"/>
 <layers>
 <layer number="1" name="Top" color="4" fill="1" visible="no" active="no"/>
@@
 <pinref part="GND55" gate="1" pin="GND"/>
 </segment>
+<segment>
+<pinref part="INVERTER" gate="G$1" pin="2A"/>
+<wire x1="38.1" y1="-91.44" x2="30.48" y2="-91.44" width="0.1524" layer="91"/>
+<label x="25.4" y="-91.44" size="1.778" layer="95"/>
+</segment>
+<segment>
+<pinref part="INVERTER" gate="G$1" pin="2Y"/>
+<wire x1="38.1" y1="-93.98" x2="30.48" y2="-93.98" width="0.1524" layer="91"/>
+<label x="25.4" y="-93.98" size="1.778" layer="95"/>
+</segment>
 </net>
 <net name="T2-" class="0">
@@
 </segment>
 <segment>
-<pinref part="INVERTER" gate="G$1" pin="2A"/>
-<wire x1="38.1" y1="-91.44" x2="30.48" y2="-91.44" width="0.1524" layer="91"/>
-<label x="25.4" y="-91.44" size="1.778" layer="95"/>
-</segment>
-<segment>
 <wire x1="414.02" y1="-121.92" x2="414.02" y2="-124.46" width="0.1524" layer="91"/>
 <label x="411.48" y="-121.92" size="1.778" layer="95"/>
@@
 </segment>
 <segment>
-<pinref part="INVERTER" gate="G$1" pin="2Y"/>
-<wire x1="38.1" y1="-93.98" x2="30.48" y2="-93.98" width="0.1524" layer="91"/>
-<label x="25.4" y="-93.98" size="1.778" layer="95"/>
-</segment>
-<segment>

Commit message: Final routing
Connections:
- removed net N$8: D1.A, JP1.1
- removed net N$9: D2.A, JP2.1
- net CS: no longer D20.A
- net GND: now also D1.A, D2.A, D20.A, D3.A
- net N$37: now also JP1.1
- net N$40: now also JP2.1
- net VDD: no longer D3.A
Other:
- note added: "Cold Junction compensation unit with analog to digital conversion"
- note added: "Dual MUX for Positive and Negative Terminal Inputs"
- note added: "K Type Thermocouple - PCB Connectors"
- note added: "Pin header with 0 ohm resistors to switch to direct SPI link if needed"
- note added: "Voltage sinking resistors with minimum resistance to ensure parasitic capacitance discharge in small time intervals."
- note added: "isoSPI (Slave)"
- note removed: "PCB Connectors"
- moved on the sheet: AND1, AND2, C1, C10, C2, C3, C4, C5, C6, C7, C8, C9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

Commit message: Board Complete
Parts:
- renumbered IC1 to MUX+, IC2 to MUX-
Changed lines of the file:
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@@
 </classes>
 <parts>
-<part name="IC1" library="SamacSys_Parts" deviceset="DG4051EEQ-T1-GE3" device=""/>
-<part name="IC2" library="SamacSys_Parts" deviceset="DG4051EEQ-T1-GE3" device=""/>
+<part name="MUX+" library="SamacSys_Parts" deviceset="DG4051EEQ-T1-GE3" device=""/>
+<part name="MUX-" library="SamacSys_Parts" deviceset="DG4051EEQ-T1-GE3" device=""/>
 <part name="GND1" library="supply1" library_urn="urn:adsk.eagle:library:371" deviceset="GND" device=""/>
 <part name="GND2" library="supply1" library_urn="urn:adsk.eagle:library:371" deviceset="GND" device=""/>
@@
 </plain>
 <instances>
-<instance part="IC1" gate="G$1" x="-114.3" y="25.4" smashed="yes">
+<instance part="MUX+" gate="G$1" x="-114.3" y="25.4" smashed="yes">
 <attribute name="NAME" x="-102.87" y="33.02" size="1.778" layer="95" align="center-left"/>
 <attribute name="VALUE" x="-110.49" y="30.48" size="1.778" layer="96" align="center-left"/>
 </instance>
-<instance part="IC2" gate="G$1" x="-114.3" y="-12.7" smashed="yes">
+<instance part="MUX-" gate="G$1" x="-114.3" y="-12.7" smashed="yes">
 <attribute name="NAME" x="-102.87" y="-5.08" size="1.778" layer="95" align="center-left"/>
 <attribute name="VALUE" x="-110.49" y="-7.62" size="1.778" layer="96" align="center-left"/>
@@
 <net name="T7+" class="0">
 <segment>
-<pinref part="IC1" gate="G$1" pin="X7"/>
+<pinref part="MUX+" gate="G$1" pin="X7"/>
 <wire x1="-114.3" y1="17.78" x2="-121.92" y2="17.78" width="0.1524" layer="91"/>
 <label x="-124.46" y="17.78" size="1.778" layer="95"/>
@@
 <net name="CJ-" class="0">
 <segment>
-<pinref part="IC2" gate="G$1" pin="X"/>
+<pinref part="MUX-" gate="G$1" pin="X"/>
 <wire x1="-114.3" y1="-17.78" x2="-121.92" y2="-17.78" width="0.1524" layer="91"/>
 <label x="-124.46" y="-17.78" size="1.778" layer="95"/>
@@
 <net name="T1+" class="0">
 <segment>
-<pinref part="IC1" gate="G$1" pin="X1"/>
+<pinref part="MUX+" gate="G$1" pin="X1"/>
 <wire x1="-86.36" y1="20.32" x2="-78.74" y2="20.32" width="0.1524" layer="91"/>
 <label x="-78.74" y="20.32" size="1.778" layer="95"/>
@@
 <net name="T2+" class="0">
 <segment>
-<pinref part="IC1" gate="G$1" pin="X2"/>
+<pinref part="MUX+" gate="G$1" pin="X2"/>
 <wire x1="-86.36" y1="22.86" x2="-78.74" y2="22.86" width="0.1524" layer="91"/>
 <label x="-78.74" y="22.86" size="1.778" layer="95"/>
@@
 <net name="T3+" class="0">
 <segment>
-<pinref part="IC1" gate="G$1" pin="X3"/>
+<pinref part="MUX+" gate="G$1" pin="X3"/>
 <wire x1="-86.36" y1="15.24" x2="-78.74" y2="15.24" width="0.1524" layer="91"/>
 <label x="-78.74" y="15.24" size="1.778" layer="95"/>
@@
 <net name="T4+" class="0">
 <segment>
-<pinref part="IC1" gate="G$1" pin="X4"/>
+<pinref part="MUX+" gate="G$1" pin="X4"/>
 <wire x1="-114.3" y1="25.4" x2="-121.92" y2="25.4" width="0.1524" layer="91"/>
 <label x="-124.46" y="25.4" size="1.778" layer="95"/>
@@
 <net name="T6+" class="0">
 <segment>
-<pinref part="IC1" gate="G$1" pin="X6"/>
+<pinref part="MUX+" gate="G$1" pin="X6"/>
 <wire x1="-114.3" y1="22.86" x2="-121.92" y2="22.86" width="0.1524" layer="91"/>
 <label x="-124.46" y="22.86" size="1.778" layer="95"/>
@@
 <net name="CJ+" class="0">
 <segment>
-<pinref part="IC1" gate="G$1" pin="X"/>
+<pinref part="MUX+" gate="G$1" pin="X"/>
 <wire x1="-114.3" y1="20.32" x2="-121.92" y2="20.32" width="0.1524" layer="91"/>
 <label x="-124.46" y="20.32" size="1.778" layer="95"/>
@@
 <net name="T5+" class="0">
 <segment>
-<pinref part="IC1" gate="G$1" pin="X5"/>
+<pinref part="MUX+" gate="G$1" pin="X5"/>
 <wire x1="-114.3" y1="15.24" x2="-121.92" y2="15.24" width="0.1524" layer="91"/>
 <label x="-124.46" y="15.24" size="1.778" layer="95"/>
@@
 <net name="GND" class="0">
 <segment>
-<pinref part="IC1" gate="G$1" pin="GND"/>
+<pinref part="MUX+" gate="G$1" pin="GND"/>
 <wire x1="-114.3" y1="7.62" x2="-124.46" y2="7.62" width="0.1524" layer="91"/>
 <pinref part="GND1" gate="1" pin="GND"/>
@@
 </segment>
 <segment>
-<pinref part="IC2" gate="G$1" pin="GND"/>
+<pinref part="MUX-" gate="G$1" pin="GND"/>
 <wire x1="-114.3" y1="-30.48" x2="-124.46" y2="-30.48" width="0.1524" layer="91"/>
 <wire x1="-124.46" y1="-30.48" x2="-124.46" y2="-35.56" width="0.1524" layer="91"/>
@@
 <net name="T2-" class="0">
 <segment>
-<pinref part="IC2" gate="G$1" pin="X2"/>
+<pinref part="MUX-" gate="G$1" pin="X2"/>
 <wire x1="-86.36" y1="-15.24" x2="-78.74" y2="-15.24" width="0.1524" layer="91"/>
 <label x="-78.74" y="-15.24" size="1.778" layer="95"/>
@@
 <net name="T1-" class="0">
 <segment>
-<pinref part="IC2" gate="G$1" pin="X1"/>
+<pinref part="MUX-" gate="G$1" pin="X1"/>
 <wire x1="-86.36" y1="-17.78" x2="-78.74" y2="-17.78" width="0.1524" layer="91"/>
 <label x="-78.74" y="-17.78" size="1.778" layer="95"/>
@@
 <net name="T3-" class="0">
 <segment>
-<pinref part="IC2" gate="G$1" pin="X3"/>
+<pinref part="MUX-" gate="G$1" pin="X3"/>
 <wire x1="-86.36" y1="-22.86" x2="-78.74" y2="-22.86" width="0.1524" layer="91"/>
 <label x="-78.74" y="-22.86" size="1.778" layer="95"/>
@@
 <net name="T4-" class="0">
 <segment>
-<pinref part="IC2" gate="G$1" pin="X4"/>
+<pinref part="MUX-" gate="G$1" pin="X4"/>
 <wire x1="-114.3" y1="-12.7" x2="-121.92" y2="-12.7" width="0.1524" layer="91"/>
 <label x="-124.46" y="-12.7" size="1.778" layer="95"/>
@@
 <net name="T6-" class="0">
 <segment>
-<pinref part="IC2" gate="G$1" pin="X6"/>
+<pinref part="MUX-" gate="G$1" pin="X6"/>
 <wire x1="-114.3" y1="-15.24" x2="-121.92" y2="-15.24" width="0.1524" layer="91"/>
 <label x="-124.46" y="-15.24" size="1.778" layer="95"/>
@@
 <net name="T7-" class="0">
 <segment>
-<pinref part="IC2" gate="G$1" pin="X7"/>
+<pinref part="MUX-" gate="G$1" pin="X7"/>
 <wire x1="-114.3" y1="-20.32" x2="-121.92" y2="-20.32" width="0.1524" layer="91"/>
 <label x="-124.46" y="-20.32" size="1.778" layer="95"/>
@@
 <net name="T5-" class="0">
 <segment>
-<pinref part="IC2" gate="G$1" pin="X5"/>
+<pinref part="MUX-" gate="G$1" pin="X5"/>
 <wire x1="-114.3" y1="-22.86" x2="-121.92" y2="-22.86" width="0.1524" layer="91"/>
 <label x="-124.46" y="-22.86" size="1.778" layer="95"/>
@@
 <net name="T0+" class="0">
 <segment>
-<pinref part="IC1" gate="G$1" pin="X0"/>
+<pinref part="MUX+" gate="G$1" pin="X0"/>
 <wire x1="-86.36" y1="17.78" x2="-78.74" y2="17.78" width="0.1524" layer="91"/>
 <label x="-78.74" y="17.78" size="1.778" layer="95"/>
@@
 <net name="T0-" class="0">
 <segment>
-<pinref part="IC2" gate="G$1" pin="X0"/>
+<pinref part="MUX-" gate="G$1" pin="X0"/>
 <wire x1="-86.36" y1="-20.32" x2="-78.74" y2="-20.32" width="0.1524" layer="91"/>
 <label x="-78.74" y="-20.32" size="1.778" layer="95"/>
@@
 <net name="VCC" class="0">
 <segment>
-<pinref part="IC1" gate="G$1" pin="V+"/>
+<pinref part="MUX+" gate="G$1" pin="V+"/>
 <wire x1="-86.36" y1="25.4" x2="-78.74" y2="25.4" width="0.1524" layer="91"/>
 <label x="-78.74" y="25.4" size="1.778" layer="95"/>
 </segment>
 <segment>
-<pinref part="IC1" gate="G$1" pin="ENABLE"/>
+<pinref part="MUX+" gate="G$1" pin="ENABLE"/>
 <wire x1="-114.3" y1="12.7" x2="-124.46" y2="12.7" width="0.1524" layer="91"/>
 <label x="-124.46" y="12.7" size="1.778" layer="95"/>
 </segment>
 <segment>
-<pinref part="IC2" gate="G$1" pin="V+"/>
+<pinref part="MUX-" gate="G$1" pin="V+"/>
 <wire x1="-86.36" y1="-12.7" x2="-78.74" y2="-12.7" width="0.1524" layer="91"/>
 <label x="-78.74" y="-12.7" size="1.778" layer="95"/>
 </segment>
 <segment>
-<pinref part="IC2" gate="G$1" pin="ENABLE"/>
+<pinref part="MUX-" gate="G$1" pin="ENABLE"/>
 <wire x1="-114.3" y1="-25.4" x2="-124.46" y2="-25.4" width="0.1524" layer="91"/>
 <label x="-124.46" y="-25.4" size="1.778" layer="95"/>
@@
 <net name="-VCC" class="0">
 <segment>
-<pinref part="IC1" gate="G$1" pin="V-"/>
+<pinref part="MUX+" gate="G$1" pin="V-"/>
 <wire x1="-114.3" y1="10.16" x2="-124.46" y2="10.16" width="0.1524" layer="91"/>
 <label x="-124.46" y="10.16" size="1.778" layer="95"/>
 </segment>
 <segment>
-<pinref part="IC2" gate="G$1" pin="V-"/>
+<pinref part="MUX-" gate="G$1" pin="V-"/>
 <wire x1="-114.3" y1="-27.94" x2="-124.46" y2="-27.94" width="0.1524" layer="91"/>
 <label x="-124.46" y="-27.94" size="1.778" layer="95"/>
@@
 </segment>
 <segment>
-<pinref part="IC1" gate="G$1" pin="A"/>
+<pinref part="MUX+" gate="G$1" pin="A"/>
 <wire x1="-86.36" y1="12.7" x2="-78.74" y2="12.7" width="0.1524" layer="91"/>
 <label x="-78.74" y="12.7" size="1.778" layer="95"/>
 </segment>
 <segment>
-<pinref part="IC2" gate="G$1" pin="A"/>
+<pinref part="MUX-" gate="G$1" pin="A"/>
 <wire x1="-86.36" y1="-25.4" x2="-78.74" y2="-25.4" width="0.1524" layer="91"/>
 <label x="-78.74" y="-25.4" size="1.778" layer="95"/>
@@
 </segment>
 <segment>
-<pinref part="IC1" gate="G$1" pin="B"/>
+<pinref part="MUX+" gate="G$1" pin="B"/>
 <wire x1="-86.36" y1="10.16" x2="-78.74" y2="10.16" width="0.1524" layer="91"/>
 <label x="-78.74" y="10.16" size="1.778" layer="95"/>
 </segment>
 <segment>
-<pinref part="IC2" gate="G$1" pin="B"/>
+<pinref part="MUX-" gate="G$1" pin="B"/>
 <wire x1="-86.36" y1="-27.94" x2="-78.74" y2="-27.94" width="0.1524" layer="91"/>
 <label x="-78.74" y="-27.94" size="1.778" layer="95"/>
@@
 </segment>
 <segment>
-<pinref part="IC2" gate="G$1" pin="C"/>
+<pinref part="MUX-" gate="G$1" pin="C"/>
 <wire x1="-86.36" y1="-30.48" x2="-78.74" y2="-30.48" width="0.1524" layer="91"/>
 <label x="-78.74" y="-30.48" size="1.778" layer="95"/>
 </segment>
 <segment>
-<pinref part="IC1" gate="G$1" pin="C"/>
+<pinref part="MUX+" gate="G$1" pin="C"/>
 <wire x1="-86.36" y1="7.62" x2="-78.74" y2="7.62" width="0.1524" layer="91"/>
 <label x="-78.74" y="7.62" size="1.778" layer="95"/>

Commit message: Actually finished i swear
Parts:
- AND1: value AND1 -> AND2
- AND2: value AND2 -> AND1
- renumbered IC5 to COLD_JUNCTION
Connections:
- net !CS: now also AND2.1B; no longer AND1.1B
- net !Q1: now also AND2.2B; no longer AND1.2B
- net !Q3: now also AND1.1B, AND2.3B; no longer AND1.3B, AND2.1B
- net !Q5: now also AND2.4B; no longer AND1.4B
- net !Q7: now also AND1.2B; no longer AND2.2B
- net CLK: now also AND2.1Y; no longer AND1.1Y
- net CS: now also AND2.1A; no longer AND1.1A
- net GND: now also AND1.3A, AND1.3B, AND1.3Y, AND1.4A, AND1.4B, AND1.4Y; no longer AND2.3A, AND2.3B, AND2.3Y, AND2.4A, AND2.4B, AND2.4Y
- net Q0: now also AND2.2A; no longer AND1.2A
- net Q0!Q1: now also AND2.2Y; no longer AND1.2Y
- net Q1: now also AND1.1A; no longer AND2.1A
- net Q1!Q3: now also AND1.1Y; no longer AND2.1Y
- net Q2: now also AND2.3A; no longer AND1.3A
- net Q2!Q3: now also AND2.3Y; no longer AND1.3Y
- net Q4: now also AND2.4A; no longer AND1.4A
- net Q4!Q5: now also AND2.4Y; no longer AND1.4Y
- net Q5: now also AND1.2A; no longer AND2.2A
- net Q5!Q7: now also AND1.2Y; no longer AND2.2Y
Other:
- moved on the sheet: AND1, AND2
