File: thermo_final.sch (EAGLE design)
At the start: 116 parts

Commit message: Added bypass caps on logic gates and did one last review
Parts:
- added C13, C14, C15, C16: 0.1uF, SamacSys_Parts:CGA3E2X7R1H104K080AE
- AND1: value AND2 -> AND1
- AND2: value AND1 -> AND2
Connections:
- net GND: now also C13.1, C14.1, C15.1, C16.1
- net VCC: now also C13.2, C14.2, C15.2, C16.2
Other:
- moved on the sheet: AND1, AND2
