File: ReducedSolidWorksModel.brd (EAGLE design)
At the start: 259.8 x 281.7 mm, 49 parts, among them J1 SAMTEC-SMM-104-02-X-DJ, J2 SAMTEC-CLP-106-02-X-DJ, J4 TFM-120-02-L-D, J5 TFM-120-02-L-D, J6 TFM-120-02-L-D, J7 TFM-120-02-L-D, J8 TFM-120-02-L-D, J9 SSM-109-L-SV

Commit message: New solid works model
Parts:
- removed U$1, U$10, U$11, U$12, U$2, U$3, U$4, U$5, U$6, U$7, U$8, U$9: THROUGH_HOLE, SamacSys_Parts:1/16TH_BOLT
- moved J9 201.7 mm to (137.8, 70.1), flipped to the bottom, turned to 0 degrees
- moved J1 98.3 mm to (182.1, 137.8)
- moved UC1 45.0 mm to (104.8, 133.1)
- moved Z12 42.1 mm to (83.3, 124.5)
- moved Z14 37.1 mm to (89.2, 60.5), turned to 180 degrees
- moved Z15 37.0 mm to (187.2, 60.5), turned to 180 degrees
- moved Z25 35.3 mm to (193.0, 124.5)
- moved Z26 30.9 mm to (209.3, 96.5)
- moved Z13 29.7 mm to (89.2, 76.7), turned to 180 degrees
- moved Z11 27.7 mm to (67.1, 96.5)
- moved Z16 23.7 mm to (187.2, 76.7), turned to 180 degrees
- moved J5 13.7 mm to (138.4, 25.4), flipped to the bottom, turned to 270 degrees
- moved J6 13.7 mm to (163.8, 25.4), flipped to the bottom, turned to 270 degrees
- moved J4 13.7 mm to (113.0, 25.4), flipped to the bottom, turned to 90 degrees
- moved J8 13.7 mm to (125.7, 25.4), flipped to the bottom, turned to 270 degrees
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Connections:
- removed net DIFF1_N: Z1.4
- new net 40G_GPIO: Z15.3
- new net ACCELEROMETER_Y: Z14.4
- new net ACCELEROMETER_Z: Z14.3
- new net C2: Z16.4
- new net C3: Z16.3
- new net DIN7: Z28.4
- new net DIN8: Z28.3
- new net IM_OUT1: Z15.4
- new net SOURCE1_10: Z15.2
- new net SOURCE2_10: Z16.2
- net 13.5V_BUS: no longer Z15.2, Z16.2, Z27.2, Z27.5, Z28.2, Z28.5
- net SOURCE1_11: now also Z25.2
- net SOURCE1_12: now also Z27.2, Z27.5; no longer Z26.5
- net SOURCE2_11: now also Z26.2, Z26.5; no longer Z25.2
- net SOURCE2_12: now also Z28.2, Z28.5; no longer Z26.2
Other:
- board size 259.8 x 281.7 mm -> 261.3 x 165.1 mm
