File: ReducedSolidWorksModel.sch (EAGLE design)
At the start: 49 parts, among them J1 SAMTEC-SMM-104-02-X-DJ, J2 SAMTEC-CLP-106-02-X-DJ, J4 TFM-120-02-L-D, J5 TFM-120-02-L-D, J6 TFM-120-02-L-D, J7 TFM-120-02-L-D, J8 TFM-120-02-L-D, J9 SSM-109-L-SV

Commit message: New solid works model
Parts:
- removed U$1, U$10, U$11, U$12, U$2, U$3, U$4, U$5, U$6, U$7, U$8, U$9: THROUGH_HOLE, SamacSys_Parts:THROUGH_HOLE
Connections:
- removed net DIFF1_N: Z1.3
- new net 40G_GPIO: Z15.2
- new net ACCELEROMETER_Y: Z14.3
- new net ACCELEROMETER_Z: Z14.2
- new net C2: Z16.3
- new net C3: Z16.2
- new net DIN7: Z28.3
- new net DIN8: Z28.2
- new net IM_OUT1: Z15.3
- new net SOURCE1_10: Z15.1
- new net SOURCE2_10: Z16.1
- net 13.5V_BUS: no longer Z15.1, Z16.1, Z27.1, Z27.4, Z28.1, Z28.4
- net SOURCE1_11: now also Z25.1
- net SOURCE1_12: now also Z27.1, Z27.4; no longer Z26.4
- net SOURCE2_11: now also Z26.1, Z26.4; no longer Z25.1
- net SOURCE2_12: now also Z28.1, Z28.4; no longer Z26.1
Other:
- note added: "Analog accelerometer"
- note added: "Single ended digital inputs Splice GND node between 2 sensors 2 sensors share same short circuit protection"
- note removed: "!CS MUX"
- note removed: "Output power supply temperature voltage"
