File: MasterPCB_transfer.sch (EAGLE design)
At the start: 1070 parts, among them IC1 NCS21911SN2T1G, IC10 LDL1117S33R, IC11 LTC4222CUH#PBF, IC12 LTC4222CUH#PBF, IC13 LTC4222CUH#PBF, IC14 LTC4222CUH#PBF, IC15 LTC4222CUH#PBF, IC16 LTC4222CUH#PBF, IC17 LTC4222CUH#PBF, IC18 LTC4222CUH#PBF, IC19 LTC4222CUH#PBF, IC2 NCS21911SN2T1G, IC20 LTC4222CUH#PBF, IC21 LTC4222CUH#PBF, IC22 LTC4222CUH#PBF, IC23 LTC4222CUH#PBF, IC24 NCS21911SN2T1G, IC25 NCS21911SN2T1G, IC26 NCS21911SN2T1G, IC27 NCS21911SN2T1G, IC28 NCS21911SN2T1G, IC29 NCS21911SN2T1G, IC3 NCS21911SN2T1G, IC30 NCS21911SN2T1G, IC31 ADIS16500AMLZ, IC32 LTC6820IUD#PBF, IC33 CBTL01023GM,115, IC34 MAX889TESA+, IC35 NCS21911SN2T1G, IC36 NCS21911SN2T1G, IC37 NCS21911SN2T1G, IC38 ADS8588HIPM, IC39 NCS21911SN2T1G, IC4 LTC4222CUH#PBF, IC40 NCS21911SN2T1G, IC41 NCS21911SN2T1G, IC42 NCS21911SN2T1G, IC43 NCS21911SN2T1G, IC44 NCS21911SN2T1G, IC45 NCS21911SN2T1G, IC46 NCS21911SN2T1G, IC47 NCS21911SN2T1G, IC48 NCS21911SN2T1G, IC49 NCS21911SN2T1G, IC5 LP38692SDX-5.0_NOPB, IC50 NCS21911SN2T1G, IC51 ADS8588HIPM, IC52 ADS8588HIPM, IC53 NCS21911SN2T1G, IC54 NCS21911SN2T1G, IC55 NCS21911SN2T1G, IC56 NCS21911SN2T1G, IC57 NCS21911SN2T1G, IC58 NCS21911SN2T1G, IC59 NCS21911SN2T1G, IC6 LP38692SDX-5.0_NOPB, IC60 NCS21911SN2T1G, IC61 NCS21911SN2T1G, IC62 NCS21911SN2T1G, IC63 NCS21911SN2T1G, IC64 NCS21911SN2T1G, IC65 NCS21911SN2T1G, IC66 NCS21911SN2T1G, IC67 NCS21911SN2T1G, IC68 NCS21911SN2T1G, IC69 NCS21911SN2T1G, IC7 LDL1117S33R, IC70 NCS21911SN2T1G, IC71 NCS21911SN2T1G, IC72 NCS21911SN2T1G, IC73 NCS21911SN2T1G, IC74 NCS21911SN2T1G, IC75 NCS21911SN2T1G, IC76 NCS21911SN2T1G, IC77 NCS21911SN2T1G, IC78 NCS21911SN2T1G, IC79 NCS21911SN2T1G, IC8 LDL1117S33R, IC9 LP38692SDX-5.0_NOPB, J1 SAMTEC-SMM-104-02-X-DJ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

Commit message: save point, adding gnd nodes
Connections:
- removed net GND1: J5.07
- removed net GND2: J5.17
- removed net GND3: J5.27
- removed net GND4: J5.37, J5.39
- removed net N$365: J5.71
- removed net N$366: J5.69
- removed net N$369: J5.63
- removed net N$370: J5.61
- removed net N$50: J5.09
- removed net N$60: J5.19
- removed net N$64: J5.29
- removed net N$65: J5.77
- removed net N$70: J5.79
- net GND: now also J5.07, J5.09, J5.17, J5.19, J5.27, J5.29, J5.37, J5.39, J5.41, J5.43, J5.45, J5.47, J5.49, J5.51, J5.53, J5.55, J5.61, J5.63, J5.69, J5.71, J5.77, J5.79, J6.32, J6.34, J6.36, J6.38, J6.40
Changed lines of the file:
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@@
 <part name="GND22" library="supply1" library_urn="urn:adsk.eagle:library:371" deviceset="GND" device=""/>
 <part name="GND578" library="supply1" library_urn="urn:adsk.eagle:library:371" deviceset="GND" device=""/>
+<part name="GND579" library="supply1" library_urn="urn:adsk.eagle:library:371" deviceset="GND" device=""/>
+<part name="GND580" library="supply1" library_urn="urn:adsk.eagle:library:371" deviceset="GND" device=""/>
 </parts>
 <sheets>
@@
 <attribute name="VALUE" x="-175.26" y="-2.54" size="1.778" layer="96"/>
 </instance>
+<instance part="GND579" gate="1" x="-264.16" y="0" smashed="yes">
+<attribute name="VALUE" x="-266.7" y="-2.54" size="1.778" layer="96"/>
+</instance>
+<instance part="GND580" gate="1" x="-116.84" y="63.5" smashed="yes" rot="R90">
+<attribute name="VALUE" x="-114.3" y="60.96" size="1.778" layer="96" rot="R90"/>
+</instance>
 </instances>
 <busses>
@@
 <junction x="-175.26" y="7.62"/>
 </segment>
+<segment>
+<wire x1="-264.16" y1="99.06" x2="-233.68" y2="99.06" width="0.1524" layer="91"/>
+<pinref part="J5" gate="G$1" pin="07"/>
+<pinref part="J5" gate="G$1" pin="09"/>
+<wire x1="-233.68" y1="96.52" x2="-264.16" y2="96.52" width="0.1524" layer="91"/>
+<wire x1="-264.16" y1="99.06" x2="-264.16" y2="96.52" width="0.1524" layer="91"/>
+<wire x1="-233.68" y1="86.36" x2="-264.16" y2="86.36" width="0.1524" layer="91"/>
+<pinref part="J5" gate="G$1" pin="17"/>
+<wire x1="-264.16" y1="96.52" x2="-264.16" y2="86.36" width="0.1524" layer="91"/>
+<junction x="-264.16" y="96.52"/>
+<pinref part="J5" gate="G$1" pin="19"/>
+<wire x1="-233.68" y1="83.82" x2="-264.16" y2="83.82" width="0.1524" layer="91"/>
+<wire x1="-264.16" y1="86.36" x2="-264.16" y2="83.82" width="0.1524" layer="91"/>
+<junction x="-264.16" y="86.36"/>
+<wire x1="-233.68" y1="73.66" x2="-264.16" y2="73.66" width="0.1524" layer="91"/>
+<pinref part="J5" gate="G$1" pin="27"/>
+<wire x1="-264.16" y1="83.82" x2="-264.16" y2="73.66" width="0.1524" layer="91"/>
+<junction x="-264.16" y="83.82"/>
+<pinref part="J5" gate="G$1" pin="29"/>
+<wire x1="-233.68" y1="71.12" x2="-264.16" y2="71.12" width="0.1524" layer="91"/>
+<wire x1="-264.16" y1="73.66" x2="-264.16" y2="71.12" width="0.1524" layer="91"/>
+<junction x="-264.16" y="73.66"/>
+<wire x1="-233.68" y1="60.96" x2="-264.16" y2="60.96" width="0.1524" layer="91"/>
+<wire x1="-233.68" y1="58.42" x2="-264.16" y2="58.42" width="0.1524" layer="91"/>
+<pinref part="J5" gate="G$1" pin="37"/>
+<pinref part="J5" gate="G$1" pin="39"/>
+<wire x1="-264.16" y1="71.12" x2="-264.16" y2="60.96" width="0.1524" layer="91"/>
+<junction x="-264.16" y="71.12"/>
+<wire x1="-264.16" y1="60.96" x2="-264.16" y2="58.42" width="0.1524" layer="91"/>
+<junction x="-264.16" y="60.96"/>
+<pinref part="GND579" gate="1" pin="GND"/>
+<wire x1="-264.16" y1="58.42" x2="-264.16" y2="55.88" width="0.1524" layer="91"/>
+<junction x="-264.16" y="58.42"/>
+<pinref part="J5" gate="G$1" pin="79"/>
+<wire x1="-264.16" y1="55.88" x2="-264.16" y2="53.34" width="0.1524" layer="91"/>
+<wire x1="-264.16" y1="53.34" x2="-264.16" y2="50.8" width="0.1524" layer="91"/>
+<wire x1="-264.16" y1="50.8" x2="-264.16" y2="48.26" width="0.1524" layer="91"/>
+<wire x1="-264.16" y1="48.26" x2="-264.16" y2="45.72" width="0.1524" layer="91"/>
+<wire x1="-264.16" y1="45.72" x2="-264.16" y2="43.18" width="0.1524" layer="91"/>
+<wire x1="-264.16" y1="43.18" x2="-264.16" y2="40.64" width="0.1524" layer="91"/>
+<wire x1="-264.16" y1="40.64" x2="-264.16" y2="38.1" width="0.1524" layer="91"/>
+<wire x1="-264.16" y1="38.1" x2="-264.16" y2="30.48" width="0.1524" layer="91"/>
+<wire x1="-264.16" y1="30.48" x2="-264.16" y2="27.94" width="0.1524" layer="91"/>
+<wire x1="-264.16" y1="27.94" x2="-264.16" y2="20.32" width="0.1524" layer="91"/>
+<wire x1="-264.16" y1="20.32" x2="-264.16" y2="17.78" width="0.1524" layer="91"/>
+<wire x1="-264.16" y1="17.78" x2="-264.16" y2="10.16" width="0.1524" layer="91"/>
+<wire x1="-264.16" y1="10.16" x2="-264.16" y2="7.62" width="0.1524" layer="91"/>
+<wire x1="-264.16" y1="7.62" x2="-264.16" y2="2.54" width="0.1524" layer="91"/>
+<wire x1="-233.68" y1="7.62" x2="-264.16" y2="7.62" width="0.1524" layer="91"/>
+<junction x="-264.16" y="7.62"/>
+<pinref part="J5" gate="G$1" pin="77"/>
+<wire x1="-233.68" y1="10.16" x2="-264.16" y2="10.16" width="0.1524" layer="91"/>
+<junction x="-264.16" y="10.16"/>
+<pinref part="J5" gate="G$1" pin="71"/>
+<wire x1="-233.68" y1="17.78" x2="-264.16" y2="17.78" width="0.1524" layer="91"/>
+<junction x="-264.16" y="17.78"/>
+<pinref part="J5" gate="G$1" pin="69"/>
+<wire x1="-233.68" y1="20.32" x2="-264.16" y2="20.32" width="0.1524" layer="91"/>
+<junction x="-264.16" y="20.32"/>
+<pinref part="J5" gate="G$1" pin="63"/>
+<wire x1="-233.68" y1="27.94" x2="-264.16" y2="27.94" width="0.1524" layer="91"/>
+<junction x="-264.16" y="27.94"/>
+<pinref part="J5" gate="G$1" pin="61"/>
+<wire x1="-233.68" y1="30.48" x2="-264.16" y2="30.48" width="0.1524" layer="91"/>
+<junction x="-264.16" y="30.48"/>
+<pinref part="J5" gate="G$1" pin="55"/>
+<wire x1="-233.68" y1="38.1" x2="-264.16" y2="38.1" width="0.1524" layer="91"/>
+<junction x="-264.16" y="38.1"/>
+<pinref part="J5" gate="G$1" pin="53"/>
+<wire x1="-233.68" y1="40.64" x2="-264.16" y2="40.64" width="0.1524" layer="91"/>
+<junction x="-264.16" y="40.64"/>
+<pinref part="J5" gate="G$1" pin="51"/>
+<wire x1="-233.68" y1="43.18" x2="-264.16" y2="43.18" width="0.1524" layer="91"/>
+<junction x="-264.16" y="43.18"/>
+<pinref part="J5" gate="G$1" pin="49"/>
+<wire x1="-233.68" y1="45.72" x2="-264.16" y2="45.72" width="0.1524" layer="91"/>
+<junction x="-264.16" y="45.72"/>
+<pinref part="J5" gate="G$1" pin="47"/>
+<wire x1="-233.68" y1="48.26" x2="-264.16" y2="48.26" width="0.1524" layer="91"/>
+<junction x="-264.16" y="48.26"/>
+<pinref part="J5" gate="G$1" pin="45"/>
+<wire x1="-233.68" y1="50.8" x2="-264.16" y2="50.8" width="0.1524" layer="91"/>
+<junction x="-264.16" y="50.8"/>
+<pinref part="J5" gate="G$1" pin="43"/>
+<wire x1="-233.68" y1="53.34" x2="-264.16" y2="53.34" width="0.1524" layer="91"/>
+<junction x="-264.16" y="53.34"/>
+<pinref part="J5" gate="G$1" pin="41"/>
+<wire x1="-233.68" y1="55.88" x2="-264.16" y2="55.88" width="0.1524" layer="91"/>
+<junction x="-264.16" y="55.88"/>
+</segment>
+<segment>
+<pinref part="J6" gate="G$1" pin="32"/>
+<wire x1="-124.46" y1="68.58" x2="-119.38" y2="68.58" width="0.1524" layer="91"/>
+<pinref part="J6" gate="G$1" pin="40"/>
+<wire x1="-119.38" y1="68.58" x2="-119.38" y2="66.04" width="0.1524" layer="91"/>
+<wire x1="-119.38" y1="66.04" x2="-119.38" y2="63.5" width="0.1524" layer="91"/>
+<wire x1="-119.38" y1="63.5" x2="-119.38" y2="60.96" width="0.1524" layer="91"/>
+<wire x1="-119.38" y1="60.96" x2="-119.38" y2="58.42" width="0.1524" layer="91"/>
+<wire x1="-119.38" y1="58.42" x2="-124.46" y2="58.42" width="0.1524" layer="91"/>
+<pinref part="J6" gate="G$1" pin="38"/>
+<wire x1="-124.46" y1="60.96" x2="-119.38" y2="60.96" width="0.1524" layer="91"/>
+<junction x="-119.38" y="60.96"/>
+<pinref part="J6" gate="G$1" pin="36"/>
+<wire x1="-124.46" y1="63.5" x2="-119.38" y2="63.5" width="0.1524" layer="91"/>
+<junction x="-119.38" y="63.5"/>
+<pinref part="J6" gate="G$1" pin="34"/>
+<wire x1="-124.46" y1="66.04" x2="-119.38" y2="66.04" width="0.1524" layer="91"/>
+<junction x="-119.38" y="66.04"/>
+<pinref part="GND580" gate="1" pin="GND"/>
+</segment>
 </net>
 <net name="DIFF1_P" class="0">
@@
 </segment>
 </net>
-<net name="GND1" class="0">
-<segment>
-<wire x1="-264.16" y1="99.06" x2="-233.68" y2="99.06" width="0.1524" layer="91"/>
-<pinref part="J5" gate="G$1" pin="07"/>
-</segment>
-</net>
-<net name="N$50" class="0">
-<segment>
-<pinref part="J5" gate="G$1" pin="09"/>
-<wire x1="-233.68" y1="96.52" x2="-264.16" y2="96.52" width="0.1524" layer="91"/>
-</segment>
-</net>
-<net name="GND2" class="0">
-<segment>
-<wire x1="-233.68" y1="86.36" x2="-264.16" y2="86.36" width="0.1524" layer="91"/>
-<pinref part="J5" gate="G$1" pin="17"/>
-</segment>
-</net>
-<net name="N$60" class="0">
-<segment>
-<pinref part="J5" gate="G$1" pin="19"/>
-<wire x1="-233.68" y1="83.82" x2="-264.16" y2="83.82" width="0.1524" layer="91"/>
-</segment>
-</net>
-<net name="GND3" class="0">
-<segment>
-<wire x1="-233.68" y1="73.66" x2="-264.16" y2="73.66" width="0.1524" layer="91"/>
-<pinref part="J5" gate="G$1" pin="27"/>
-</segment>
-</net>
-<net name="N$64" class="0">
-<segment>
-<pinref part="J5" gate="G$1" pin="29"/>
-<wire x1="-233.68" y1="71.12" x2="-264.16" y2="71.12" width="0.1524" layer="91"/>
-</segment>
-</net>
-<net name="GND4" class="0">
-<segment>
-<wire x1="-233.68" y1="60.96" x2="-264.16" y2="60.96" width="0.1524" layer="91"/>
-<wire x1="-233.68" y1="58.42" x2="-264.16" y2="58.42" width="0.1524" layer="91"/>
-<pinref part="J5" gate="G$1" pin="37"/>
-<pinref part="J5" gate="G$1" pin="39"/>
-</segment>
-</net>
-<net name="N$365" class="0">
-<segment>
-<wire x1="-236.22" y1="17.78" x2="-233.68" y2="17.78" width="0.1524" layer="91"/>
-<pinref part="J5" gate="G$1" pin="71"/>
-</segment>
-</net>
-<net name="N$366" class="0">
-<segment>
-<wire x1="-236.22" y1="20.32" x2="-233.68" y2="20.32" width="0.1524" layer="91"/>
-<pinref part="J5" gate="G$1" pin="69"/>
-</segment>
-</net>
-<net name="N$369" class="0">
-<segment>
-<wire x1="-236.22" y1="27.94" x2="-233.68" y2="27.94" width="0.1524" layer="91"/>
-<pinref part="J5" gate="G$1" pin="63"/>
-</segment>
-</net>
-<net name="N$370" class="0">
-<segment>
-<wire x1="-236.22" y1="30.48" x2="-233.68" y2="30.48" width="0.1524" layer="91"/>
-<pinref part="J5" gate="G$1" pin="61"/>
-</segment>
-</net>
-<net name="N$65" class="0">
-<segment>
-<pinref part="J5" gate="G$1" pin="77"/>
-<wire x1="-236.22" y1="10.16" x2="-233.68" y2="10.16" width="0.1524" layer="91"/>
-</segment>
-</net>
-<net name="N$70" class="0">
-<segment>
-<pinref part="J5" gate="G$1" pin="79"/>
-<wire x1="-236.22" y1="7.62" x2="-233.68" y2="7.62" width="0.1524" layer="91"/>
-</segment>
-</net>

Commit message: Save point
Connections:
- net 13.5V_BUS: now also J12.02, J12.04, J12.06, J12.08; no longer J12.32, J12.49, J12.50, J12.51, J12.52, J12.53, J12.54, J12.71, J12.72
- net 3.3V_SWITCHING: now also J12.28, J12.30, J12.32, J12.34, J12.36, J12.38; no longer J12.20, J12.26, J12.59, J12.60, J12.65, J12.66
- net 5V_BUS: no longer J12.28, J12.67, J12.68
- net 5V_CONNECTOR: now also J12.20, J12.22, J12.24, J12.26; no longer J12.55, J12.56, J12.57, J12.58
- net 6.5V_BUS: no longer J12.30, J12.69, J12.70
- net GND: now also J12.49, J12.50, J12.51, J12.52, J12.53, J12.54, J12.55, J12.56, J12.57, J12.58, J12.59, J12.60, J12.65, J12.66, J12.67, J12.68, J12.69, J12.70, J12.71, J12.72; no longer J12.02, J12.04, J12.06, J12.08, J12.22, J12.24, J12.34, J12.36, J12.38
