File: Diff_AMP.brd (EAGLE design)
At the start: 10 parts, among them IC3 MCP1501T-25E_RW, IC4 NCS21911SN2T1G, IC5 NCS21911SN2T1G

Commit message: board
Parts:
- removed R10, R9: ERA-3AED3161V, SamacSys_Parts:ERA3A_(0603)
- removed R11, R12: ERA-3AED1650V, SamacSys_Parts:ERA3A_(0603)
- added C1, C3: CGA3E2X7R1H104K080AE, SamacSys_Parts:CAPC1608X90N
- added R1, R2: RT0603BRD0750KL, SamacSys_Parts:RESC1608X55N
Connections:
- removed net N$10: C2.2, IC4.3, R8.2, R9.1
- new net GND: C1.2, C3.2, IC3.2, IC3.4, IC3.5, IC3.6
- new net N$1: C1.1, IC3.7, IC3.8
- new net N$2: C3.1, IC3.1, IC3.3
- new net N$3: C2.2, IC4.3, R1.1, R8.2
- net N$11: now also R1.2; no longer R11.1, R9.2
- net N$12: no longer R11.2, R12.1
- net N$13: now also R2.1; no longer R10.1, R12.2
- net N$14: now also R2.2; no longer IC3.8, R10.2
Other:
- board outline added: 16.5 x 11.4 mm

Commit message: Ready for Rev
Parts:
- added C4, C5: CGA3E2X7R1H104K080AE, SamacSys_Parts:CAPC1608X90N
- added C6, C7: C1206F105M5RACAUTO7210, SamacSys_Parts:C1206
- added IC1: NCV8711ASN500T1G, SamacSys_Parts:SOT95P275X110-5N
- added JP1: (no value), pinhead:1X02
- added R10, R5, R6, R9: PTF56350R00BZEK, SamacSys_Parts:RESAD1559W64L635D231
- added R3, R4: RT0603BRD07505RL, SamacSys_Parts:RESC1608X55N
- C1, C3: value CGA3E2X7R1H104K080AE -> C1206F105M5RACAUTO7210; device SamacSys_Parts:CAPC1608X90N -> SamacSys_Parts:C1206
- moved R2 140.7 mm to (15.2, 5.84), flipped to the bottom, turned to 180 degrees
- moved R1 140.1 mm to (14.7, 11.9), flipped to the bottom, turned to 180 degrees
- moved C1 126.5 mm to (7.11, 12.4), flipped to the bottom, turned to 180 degrees
- moved C3 121.5 mm to (7.11, 3.30), flipped to the bottom, turned to 180 degrees
- moved IC5 112.1 mm to (19.3, 8.38), flipped to the bottom
- moved IC4 109.9 mm to (19.6, 12.7), flipped to the bottom, turned to 270 degrees
- moved R8 99.4 mm to (25.1, 12.4), flipped to the bottom, turned to 90 degrees
- moved C2 96.2 mm to (20.1, 4.06), flipped to the bottom, turned to 180 degrees
- moved R7 90.1 mm to (25.1, 6.60), flipped to the bottom, turned to 90 degrees
- moved IC3 72.9 mm to (6.86, 8.13), flipped to the bottom, turned to 90 degrees
Connections:
- removed net N$11: IC4.4, R1.2
- removed net N$15: R7.1
- removed net N$16: R8.1
- new net 13.5V: C3.2, C7.1, IC1.1, IC1.3, IC3.1, IC3.3, JP1.2
- new net N$10: C6.1, IC1.5, R10.2, R5.2
- new net N$4: C4.2, IC4.5
- new net N$5: C5.2, IC5.5
- new net N$6: R5.1, R6.2, R7.1
- new net N$7: R10.1, R8.1, R9.2
- net GND: now also C1.1, C3.1, C4.1, C5.1, C6.2, C7.2, IC1.2, IC3.9, IC4.2, IC5.2, JP1.1, R6.1, R9.1; no longer C1.2, C3.2
- net N$1: now also C1.2, R1.1; no longer C1.1
- net N$12: now also R3.2, R4.1
- net N$13: now also R4.2
- net N$2: now also IC4.4, R1.2, R3.1; no longer C3.1, IC3.1, IC3.3
- net N$3: no longer R1.1
Routing:
- net N$10: track 0.00 -> 35.1 mm
- net 13.5V: track 0.00 -> 28.9 mm
- net N$7: track 0.00 -> 21.9 mm
- net N$3: track 0.00 -> 15.7 mm
- net N$12: track 0.00 -> 13.1 mm, vias 0 -> 2
- net N$2: track 0.00 -> 11.4 mm
- net N$1: track 0.00 -> 9.97 mm
- net N$9: track 0.00 -> 8.79 mm, vias 0 -> 2
- net N$13: track 0.00 -> 8.28 mm
- net N$14: track 0.00 -> 7.00 mm
- net N$6: track 0.00 -> 6.47 mm
- net N$5: track 0.00 -> 6.28 mm, vias 0 -> 2
- net N$4: track 0.00 -> 4.77 mm
- net GND: track 0.00 -> 2.77 mm, vias 0 -> 13
- added copper zone on layer 1, net GND
- added copper zone on layer 16, net GND
Other:
- board size 16.5 x 11.4 mm -> 30.2 x 16.8 mm
- board text added: "13.5V"
- board text added: "GND"

Commit message: rev_1
Parts:
- removed R7, R8: ERA-3VRW1911V, SamacSys_Parts:ERA3KV_(0603)
- added JP2: (no value), pinhead:1X04
- added R11, R12: ERA-3VEB1911V, SamacSys_Parts:ERA3KV_(0603)
- C2: value C1210C184J1JACAUTO -> GCJ188R71E183KA01J; device SamacSys_Parts:C1210 -> SamacSys_Parts:CAPC1608X100N
- JP1: device pinhead:1X02 -> pinhead:1X04
- moved R5 19.3 mm to (8.64, 2.54), turned to 90 degrees
- moved IC3 16.5 mm to (22.4, 13.7)
- moved C5 16.2 mm to (7.11, 14.2), turned to 180 degrees
- moved R4 13.8 mm to (10.9, 16.3), turned to 0 degrees
- moved R2 12.8 mm to (7.87, 16.3), turned to 0 degrees
- moved C4 12.7 mm to (10.2, 10.2), turned to 180 degrees
- moved R6 12.3 mm to (15.2, 18.0), turned to 270 degrees
- moved C1 11.4 mm to (18.5, 12.2), turned to 90 degrees
- moved R10 11.2 mm to (11.9, 2.54), turned to 90 degrees
- moved R9 10.3 mm to (18.5, 18.0), turned to 270 degrees
- moved IC5 9.89 mm to (10.7, 13.2), turned to 90 degrees
- moved C3 7.37 mm to (6.86, 10.7), turned to 90 degrees
- moved R3 7.33 mm to (14.0, 16.3), turned to 0 degrees
- moved C2 5.57 mm to (16.0, 7.87)
- moved IC4 5.14 mm to (14.7, 10.9)
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Connections:
- removed net 13.5V: C3.2, C7.1, IC1.1, IC1.3, IC3.1, IC3.3, JP1.2
- removed net N$10: C6.1, IC1.5, R10.2, R5.2
- removed net N$14: IC5.1, R2.2
- removed net N$6: R5.1, R6.2, R7.1
- removed net N$7: R10.1, R8.1, R9.2
- new net 5V: C3.2, C4.1, C5.1, C6.1, IC1.5, IC3.1, IC3.3, JP2.1, R10.2, R5.2
- new net VA: JP2.2, R12.1, R5.1, R6.2
- new net VB: JP2.3, R10.1, R11.1, R9.2
- new net VIN: C7.1, IC1.1, IC1.3, JP1.1
- new net VOUT: IC5.1, JP1.3, R2.2
- net GND: now also JP1.2, JP1.4, JP2.4; no longer C4.1, C5.1, JP1.1
- net N$3: now also C2.1, R11.2; no longer C2.2, R8.2
- net N$9: now also C2.2, R12.2; no longer C2.1, R7.2
Routing:
- net 5V: track 0.00 -> 48.1 mm, vias 0 -> 1
- net N$10: track 35.1 -> 0.00 mm
- net 13.5V: track 28.9 -> 0.00 mm
- net VOUT: track 0.00 -> 22.5 mm, vias 0 -> 1
- net N$7: track 21.9 -> 0.00 mm
- net VIN: track 0.00 -> 16.9 mm
- net VA: track 0.00 -> 16.7 mm, vias 0 -> 1
- net VB: track 0.00 -> 12.6 mm, vias 0 -> 2
- net N$3: track 15.7 -> 6.97 mm
- net N$12: track 13.1 -> 5.79 mm, vias 2 -> 0
- net N$14: track 7.00 -> 0.00 mm
- net N$6: track 6.47 -> 0.00 mm
- net N$13: track 8.28 -> 3.61 mm
- net N$9: track 8.79 -> 13.2 mm
- net GND: track 2.77 -> 0.00 mm, vias 13 -> 30
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Other:
- board size 30.2 x 16.8 mm -> 25.7 x 20.6 mm
- board text added: "5V"
- board text added: "RYAN THAI BAJA SAE 2021-2022 ELECTRICAL TEAM"
- board text added: "Va"
- board text added: "Vb"
- board text added: "Vin"
- board text added: "Vout"
- board text removed: "13.5V"

Commit message: revised
Parts:
- moved C3 12.7 mm to (18.5, 5.59)
- moved R12 7.66 mm to (10.2, 5.59)
- moved C2 6.04 mm to (10.4, 10.2), turned to 0 degrees
- moved C4 5.34 mm to (15.0, 7.87), turned to 0 degrees
- moved IC1 5.08 mm to (6.86, 10.7)
- moved C7 3.94 mm to (6.86, 5.33)
- moved C6 1.78 mm to (3.30, 16.0), flipped to the bottom
- moved R9 0.49 mm to (18.1, 18.1)
- moved R11 0.36 mm to (14.5, 5.08)
- moved C5 0.36 mm to (7.37, 14.5)
- moved IC4 0.25 mm to (14.7, 10.7)
- moved R5 0.25 mm to (8.89, 2.54)
- moved R6 0.25 mm to (15.0, 18.1)
Routing:
- net N$9: track 13.2 -> 4.06 mm, vias 2 -> 0
- net VIN: track 16.9 -> 8.04 mm
- net VA: track 16.7 -> 22.4 mm, vias 1 -> 2
- net 5V: track 48.1 -> 53.5 mm
- net N$3: track 6.97 -> 10.6 mm
- net VOUT: track 22.5 -> 21.2 mm
- net N$4: track 2.86 -> 1.71 mm
- net VB: track 12.6 -> 13.4 mm, vias 2 -> 0
Other:
- board text added: "RYAN THAI BAJA SAE 2021-2022 In-Amp"
- board text removed: "RYAN THAI BAJA SAE 2021-2022 ELECTRICAL TEAM"

Commit message: Revision
Parts:
- moved C4 0.40 mm to (15.1, 7.49)
Connections:
- removed net N$4: C4.2, IC4.5
- removed net N$5: C5.2, IC5.5
- net 5V: now also C4.2, C5.2, IC4.5, IC5.5; no longer C4.1, C5.1
- net GND: now also C4.1, C5.1
Routing:
- net 5V: track 53.5 -> 63.4 mm
- net VOUT: track 21.2 -> 26.6 mm, vias 1 -> 3
- net N$5: track 4.29 -> 0.00 mm
- net VIN: track 8.04 -> 10.4 mm
- net N$9: track 4.06 -> 5.86 mm
- net N$4: track 1.71 -> 0.00 mm

Commit message: revisions
Parts:
- removed R11, R12: ERA-3VEB1911V, SamacSys_Parts:ERA3KV_(0603)
- added R7, R8: ERA-3VEB1911V, SamacSys_Parts:ERA3KV_(0603)
- C1: value C1206F105M5RACAUTO7210 -> C0603C184K3RACAUTO; device SamacSys_Parts:C1206 -> SamacSys_Parts:C0603
- moved C5 33.6 mm to (40.4, 8.26), turned to 270 degrees
- moved C4 24.4 mm to (39.4, 4.95), turned to 90 degrees
- moved C2 24.1 mm to (34.2, 5.84), turned to 180 degrees
- moved R2 23.0 mm to (30.4, 11.3), flipped to the top, turned to 180 degrees
- moved R4 23.0 mm to (33.4, 11.3), flipped to the top, turned to 180 degrees
- moved R1 23.0 mm to (39.5, 11.3), flipped to the top, turned to 180 degrees
- moved R3 23.0 mm to (36.4, 11.3), flipped to the top, turned to 180 degrees
- moved IC4 22.8 mm to (37.5, 8.51), flipped to the top, turned to 180 degrees
- moved IC5 22.7 mm to (32.9, 8.51), flipped to the top, turned to 0 degrees
- moved JP2 20.4 mm to (42.8, 6.22), turned to 90 degrees
- moved R5 20.1 mm to (27.8, 9.40), flipped to the bottom, turned to 0 degrees
- moved IC3 17.1 mm to (37.0, 4.83), flipped to the top
- moved R10 16.7 mm to (27.8, 7.87), turned to 180 degrees
- moved C1 16.5 mm to (33.4, 5.08), flipped to the top, turned to 180 degrees
- moved R9 14.6 mm to (12.2, 4.72), turned to 0 degrees
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Connections:
- net GND: now also C2.2; no longer C1.1
- net N$1: no longer C1.2
- net N$3: now also C1.1, R8.2; no longer C2.1, R11.2
- net N$9: now also C1.2, C2.1, R7.2; no longer C2.2, R12.2
- net VA: now also R7.1; no longer R12.1
- net VB: now also R8.1; no longer R11.1
Routing:
- net VB: track 13.4 -> 22.9 mm
- net VA: track 22.4 -> 29.7 mm, vias 2 -> 0
- net N$3: track 10.6 -> 17.8 mm, vias 0 -> 2
- net VOUT: track 26.6 -> 32.1 mm, vias 3 -> 0
- net N$2: track 9.16 -> 3.67 mm
- net 5V: track 63.4 -> 68.5 mm, vias 1 -> 2
- net GND: track 0.00 -> 4.83 mm, vias 23 -> 5
- net VIN: track 10.4 -> 14.4 mm
- net N$9: track 5.86 -> 8.80 mm, vias 0 -> 1
- net N$13: track 3.61 -> 6.46 mm
- net N$12: track 6.04 -> 7.79 mm
- net N$1: track 9.54 -> 10.2 mm, vias 0 -> 2
Other:
- board size 25.7 x 20.6 mm -> 46.1 x 13.6 mm

Commit message: revision
Parts:
- moved C5 10.1 mm to (30.3, 8.74)
- moved C3 2.29 mm to (31.6, 4.57), turned to 270 degrees
- moved C2 0.89 mm to (35.0, 5.64)
- moved IC5 0.28 mm to (32.8, 8.26)
- moved R7 0.13 mm to (29.6, 7.72)
Routing:
- net 5V: track 68.5 -> 72.9 mm
- net GND: track 4.83 -> 8.95 mm, vias 5 -> 10
- net N$13: track 6.46 -> 7.27 mm
- net N$9: track 8.80 -> 8.20 mm
- net N$2: track 3.67 -> 4.23 mm
- net VA: track 29.7 -> 29.2 mm

Commit message: revision
Parts:
- added C8: GCJ188R71E183KA01J, SamacSys_Parts:CAPC1608X100N
- moved C2 15.7 mm to (19.4, 5.31)
- moved C1 15.2 mm to (18.2, 5.05)
- moved IC4 15.2 mm to (22.3, 8.48)
- moved R4 15.2 mm to (18.2, 11.2)
- moved C3 15.2 mm to (16.4, 4.55)
- moved C5 15.2 mm to (15.1, 8.71)
- moved IC3 15.2 mm to (21.7, 4.80)
- moved R1 15.2 mm to (24.3, 11.2)
- moved R2 15.2 mm to (15.1, 11.2)
- moved R7 15.2 mm to (14.4, 7.70)
- moved R8 15.2 mm to (14.6, 5.18)
- moved C4 15.2 mm to (24.2, 4.93)
- moved IC5 15.2 mm to (17.6, 8.23)
- moved R3 15.2 mm to (21.2, 11.2)
- moved JP2 11.7 mm to (31.1, 6.15)
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Connections:
- net 5V: now also C7.1; no longer C6.1
- net GND: now also C8.2
- net N$3: now also C8.1
- net VIN: now also C6.1; no longer C7.1
Routing:
- net VOUT: track 32.2 -> 15.8 mm
- net 5V: track 72.9 -> 64.8 mm
- net N$3: track 17.8 -> 24.2 mm, vias 2 -> 3
- net VIN: track 14.4 -> 10.9 mm, vias 0 -> 1
- net VA: track 29.2 -> 25.8 mm, vias 0 -> 2
- net GND: vias 10 -> 11
Other:
- board size 46.1 x 13.6 mm -> 34.4 x 13.5 mm
