File: Diff_AMP.sch (EAGLE design)
At the start: 10 parts, among them IC3 MCP1501T-25E_RW, IC4 NCS21911SN2T1G, IC5 NCS21911SN2T1G

Commit message: board
Parts:
- removed R10, R9: ERA-3AED3161V, SamacSys_Parts:ERA-3AED3161V
- removed R11, R12: ERA-3AED1650V, SamacSys_Parts:ERA-3AED1650V
- added C1, C3: CGA3E2X7R1H104K080AE, SamacSys_Parts:CGA3E2X7R1H104K080AE
- added R1, R2: RT0603BRD0750KL, SamacSys_Parts:RT0603BRD0750KL
Connections:
- removed net N$10: C2.2, IC4.IN+, R8.2, R9.1
- new net GND: C1.2, C3.2, IC3.GND_1, IC3.GND_2, IC3.GND_3, IC3.GND_4
- new net N$1: C1.1, IC3.FEEDBACK, IC3.OUT
- new net N$2: C3.1, IC3.!SHDN, IC3.VDD
- new net N$3: C2.2, IC4.IN+, R1.1, R8.2
- net N$11: now also R1.2; no longer R11.1, R9.2
- net N$12: no longer R11.2, R12.1
- net N$13: now also R2.1; no longer R10.1, R12.2
- net N$14: now also R2.2; no longer IC3.FEEDBACK, R10.2
Other:
- moved on the sheet: IC3

Commit message: Ready for Rev
Parts:
- added C4, C5: CGA3E2X7R1H104K080AE, SamacSys_Parts:CGA3E2X7R1H104K080AE
- added C6, C7: C1206F105M5RACAUTO7210, SamacSys_Parts:C1206F105M5RACAUTO7210
- added IC1: NCV8711ASN500T1G, SamacSys_Parts:NCV8711ASN500T1G
- added JP1: (no value), pinhead:PINHD-1X2
- added R10, R5, R6, R9: PTF56350R00BZEK, SamacSys_Parts:PTF56350R00BZEK
- added R3, R4: RT0603BRD07505RL, SamacSys_Parts:RT0603BRD07505RL
- C1, C3: value CGA3E2X7R1H104K080AE -> C1206F105M5RACAUTO7210; device SamacSys_Parts:CGA3E2X7R1H104K080AE -> SamacSys_Parts:C1206F105M5RACAUTO7210
Connections:
- removed net N$11: IC4.IN-, R1.2
- removed net N$15: R7.1
- removed net N$16: R8.1
- new net 13.5V: C3.2, C7.1, IC1.EN, IC1.IN, IC3.!SHDN, IC3.VDD, JP1.2
- new net N$10: C6.1, IC1.OUT, R10.2, R5.2
- new net N$4: C4.2, IC4.VDD
- new net N$5: C5.2, IC5.VDD
- new net N$6: R5.1, R6.2, R7.1
- new net N$7: R10.1, R8.1, R9.2
- net GND: now also C1.1, C3.1, C4.1, C5.1, C6.2, C7.2, IC1.GND, IC3.EP, IC4.VSS, IC5.VSS, JP1.1, R6.1, R9.1; no longer C1.2, C3.2
- net N$1: now also C1.2, R1.1; no longer C1.1
- net N$12: now also R3.2, R4.1
- net N$13: now also R4.2
- net N$2: now also IC4.IN-, R1.2, R3.1; no longer C3.1, IC3.!SHDN, IC3.VDD
- net N$3: no longer R1.1
Other:
- moved on the sheet: C1, C3

Commit message: rev_1
Parts:
- removed R7, R8: ERA-3VRW1911V, SamacSys_Parts:ERA-3VRW1911V
- added JP2: (no value), pinhead:PINHD-1X4
- added R11, R12: ERA-3VEB1911V, SamacSys_Parts:ERA-3VEB1911V
- C2: value C1210C184J1JACAUTO -> GCJ188R71E183KA01J; device SamacSys_Parts:C1210C184J1JACAUTO -> SamacSys_Parts:GCJ188R71E183KA01J
- JP1: device pinhead:PINHD-1X2 -> pinhead:PINHD-1X4
Connections:
- removed net 13.5V: C3.2, C7.1, IC1.EN, IC1.IN, IC3.!SHDN, IC3.VDD, JP1.2
- removed net N$10: C6.1, IC1.OUT, R10.2, R5.2
- removed net N$14: IC5.OUT, R2.2
- removed net N$6: R5.1, R6.2, R7.1
- removed net N$7: R10.1, R8.1, R9.2
- new net 5V: C3.2, C4.1, C5.1, C6.1, IC1.OUT, IC3.!SHDN, IC3.VDD, JP2.1, R10.2, R5.2
- new net VA: JP2.2, R12.1, R5.1, R6.2
- new net VB: JP2.3, R10.1, R11.1, R9.2
- new net VIN: C7.1, IC1.EN, IC1.IN, JP1.1
- new net VOUT: IC5.OUT, JP1.3, R2.2
- net GND: now also JP1.2, JP1.4, JP2.4; no longer C4.1, C5.1, JP1.1
- net N$3: now also C2.1, R11.2; no longer C2.2, R8.2
- net N$9: now also C2.2, R12.2; no longer C2.1, R7.2
Other:
- moved on the sheet: C2, C6, C7, IC1

Commit message: revised
Other:
- moved on the sheet: C5, IC5
Changed lines of the file:
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@@
 <attribute name="VALUE" x="60.96" y="-46.99" size="1.778" layer="96" rot="R90" align="center-left"/>
 </instance>
-<instance part="IC5" gate="G$1" x="101.6" y="0" smashed="yes" rot="R270">
-<attribute name="NAME" x="105.41" y="-5.08" size="1.778" layer="95" align="center-left"/>
-<attribute name="VALUE" x="105.41" y="-2.54" size="1.778" layer="96" align="center-left"/>
+<instance part="IC5" gate="G$1" x="101.6" y="-2.54" smashed="yes" rot="R270">
+<attribute name="NAME" x="105.41" y="-10.16" size="1.778" layer="95" align="center-left"/>
+<attribute name="VALUE" x="105.41" y="-7.62" size="1.778" layer="96" align="center-left"/>
 </instance>
 <instance part="R2" gate="G$1" x="104.14" y="-66.04" smashed="yes">
@@
 <attribute name="VALUE" x="36.83" y="-59.69" size="1.778" layer="96" align="center-left"/>
 </instance>
-<instance part="C5" gate="G$1" x="83.82" y="-27.94" smashed="yes">
-<attribute name="NAME" x="82.55" y="-24.13" size="1.778" layer="95" rot="R90" align="center-left"/>
-<attribute name="VALUE" x="85.09" y="-24.13" size="1.778" layer="96" rot="R90" align="center-left"/>
+<instance part="C5" gate="G$1" x="83.82" y="-30.48" smashed="yes">
+<attribute name="NAME" x="82.55" y="-26.67" size="1.778" layer="95" rot="R90" align="center-left"/>
+<attribute name="VALUE" x="85.09" y="-26.67" size="1.778" layer="96" rot="R90" align="center-left"/>
 </instance>
 <instance part="R5" gate="G$1" x="-48.26" y="0" smashed="yes" rot="R180">
@@
 <net name="N$9" class="0">
 <segment>
-<pinref part="IC5" gate="G$1" pin="IN+"/>
 <pinref part="R12" gate="G$1" pin="2"/>
 <wire x1="12.7" y1="0" x2="35.56" y2="0" width="0.1524" layer="91"/>
 <pinref part="C2" gate="G$1" pin="2"/>
+<wire x1="35.56" y1="-5.08" x2="35.56" y2="0" width="0.1524" layer="91"/>
 <wire x1="35.56" y1="0" x2="96.52" y2="0" width="0.1524" layer="91"/>
-<wire x1="35.56" y1="-5.08" x2="35.56" y2="0" width="0.1524" layer="91"/>
 <junction x="35.56" y="0"/>
+<pinref part="IC5" gate="G$1" pin="IN+"/>
+<wire x1="96.52" y1="0" x2="96.52" y2="-2.54" width="0.1524" layer="91"/>
 </segment>
 </net>
@@
 <segment>
 <pinref part="IC5" gate="G$1" pin="IN-"/>
-<wire x1="101.6" y1="-25.4" x2="101.6" y2="-66.04" width="0.1524" layer="91"/>
+<wire x1="101.6" y1="-27.94" x2="101.6" y2="-66.04" width="0.1524" layer="91"/>
 <wire x1="101.6" y1="-66.04" x2="99.06" y2="-66.04" width="0.1524" layer="91"/>
 <pinref part="R2" gate="G$1" pin="1"/>
@@
 </segment>
 <segment>
+<pinref part="GND3" gate="1" pin="GND"/>
+<pinref part="R9" gate="G$1" pin="1"/>
+<wire x1="-25.4" y1="-22.86" x2="-22.86" y2="-22.86" width="0.1524" layer="91"/>
+<wire x1="-22.86" y1="-22.86" x2="-22.86" y2="0" width="0.1524" layer="91"/>
 <pinref part="R6" gate="G$1" pin="1"/>
-<pinref part="R9" gate="G$1" pin="1"/>
-<wire x1="-25.4" y1="0" x2="-25.4" y2="-10.16" width="0.1524" layer="91"/>
-<wire x1="-25.4" y1="-10.16" x2="-25.4" y2="-22.86" width="0.1524" layer="91"/>
-<wire x1="-25.4" y1="-10.16" x2="-17.78" y2="-10.16" width="0.1524" layer="91"/>
-<junction x="-25.4" y="-10.16"/>
-<wire x1="-17.78" y1="-10.16" x2="-17.78" y2="-12.7" width="0.1524" layer="91"/>
-<pinref part="GND3" gate="1" pin="GND"/>
+<wire x1="-22.86" y1="0" x2="-25.4" y2="0" width="0.1524" layer="91"/>
+<wire x1="-22.86" y1="0" x2="-17.78" y2="0" width="0.1524" layer="91"/>
+<junction x="-22.86" y="0"/>
+<wire x1="-17.78" y1="0" x2="-17.78" y2="-12.7" width="0.1524" layer="91"/>
 </segment>
 <segment>
@@
 <segment>
 <pinref part="IC5" gate="G$1" pin="VSS"/>
-<wire x1="99.06" y1="0" x2="99.06" y2="10.16" width="0.1524" layer="91"/>
+<wire x1="99.06" y1="-2.54" x2="99.06" y2="10.16" width="0.1524" layer="91"/>
 <wire x1="99.06" y1="10.16" x2="106.68" y2="10.16" width="0.1524" layer="91"/>
 <pinref part="GND4" gate="1" pin="GND"/>
@@
 <segment>
 <pinref part="IC5" gate="G$1" pin="VDD"/>
-<wire x1="99.06" y1="-25.4" x2="99.06" y2="-27.94" width="0.1524" layer="91"/>
+<wire x1="99.06" y1="-27.94" x2="99.06" y2="-30.48" width="0.1524" layer="91"/>
 <pinref part="C5" gate="G$1" pin="2"/>
-<wire x1="99.06" y1="-27.94" x2="96.52" y2="-27.94" width="0.1524" layer="91"/>
+<wire x1="99.06" y1="-30.48" x2="96.52" y2="-30.48" width="0.1524" layer="91"/>
 </segment>
 </net>
@@
 </segment>
 <segment>
-<pinref part="IC5" gate="G$1" pin="OUT"/>
-<wire x1="101.6" y1="0" x2="124.46" y2="0" width="0.1524" layer="91"/>
 <wire x1="124.46" y1="0" x2="124.46" y2="-66.04" width="0.1524" layer="91"/>
 <wire x1="124.46" y1="-66.04" x2="121.92" y2="-66.04" width="0.1524" layer="91"/>
 <pinref part="R2" gate="G$1" pin="2"/>
 <wire x1="124.46" y1="0" x2="132.08" y2="0" width="0.1524" layer="91"/>
+<label x="134.62" y="0" size="1.778" layer="95"/>
+<pinref part="IC5" gate="G$1" pin="OUT"/>
+<wire x1="101.6" y1="-2.54" x2="101.6" y2="0" width="0.1524" layer="91"/>
+<wire x1="101.6" y1="0" x2="124.46" y2="0" width="0.1524" layer="91"/>
 <junction x="124.46" y="0"/>
-<label x="134.62" y="0" size="1.778" layer="95"/>
 </segment>
 </net>
@@
 <segment>
 <pinref part="C4" gate="G$1" pin="1"/>
-<wire x1="38.1" y1="-50.8" x2="38.1" y2="-53.34" width="0.1524" layer="91"/>
-<label x="38.1" y="-55.88" size="1.778" layer="95"/>
-</segment>
-<segment>
-<pinref part="C5" gate="G$1" pin="1"/>
-<wire x1="83.82" y1="-27.94" x2="83.82" y2="-30.48" width="0.1524" layer="91"/>
-<label x="83.82" y="-33.02" size="1.778" layer="95"/>
+<wire x1="38.1" y1="-50.8" x2="35.56" y2="-50.8" width="0.1524" layer="91"/>
+<label x="35.56" y="-48.26" size="1.778" layer="95"/>
 </segment>
 <segment>
@@
 <label x="-43.18" y="-68.58" size="1.778" layer="95"/>
 </segment>
-</net>
+<segment>
+<pinref part="C5" gate="G$1" pin="1"/>
+<wire x1="83.82" y1="-30.48" x2="81.28" y2="-30.48" width="0.1524" layer="91"/>
+<label x="81.28" y="-30.48" size="1.778" layer="95"/>
+</segment>
+</net>

Commit message: Revision
Connections:
- removed net N$4: C4.2, IC4.VDD
- removed net N$5: C5.2, IC5.VDD
- net 5V: now also C4.2, C5.2, IC4.VDD, IC5.VDD; no longer C4.1, C5.1
- net GND: now also C4.1, C5.1
Other:
- moved on the sheet: C4, IC4
Changed lines of the file:
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@@
 <part name="GND6" library="supply1" library_urn="urn:adsk.eagle:library:371" deviceset="GND" device=""/>
 <part name="C2" library="SamacSys_Parts" library_urn="urn:adsk.eagle:library:35608874" deviceset="GCJ188R71E183KA01J" device="" package3d_urn="urn:adsk.eagle:package:35615821/2"/>
+<part name="GND7" library="supply1" library_urn="urn:adsk.eagle:library:371" deviceset="GND" device=""/>
+<part name="GND8" library="supply1" library_urn="urn:adsk.eagle:library:371" deviceset="GND" device=""/>
 </parts>
 <sheets>
@@
 <attribute name="VALUE" x="-21.59" y="-58.42" size="1.778" layer="96" rot="MR180" align="center-left"/>
 </instance>
-<instance part="IC4" gate="G$1" x="55.88" y="-22.86" smashed="yes" rot="R270">
-<attribute name="NAME" x="63.5" y="-46.99" size="1.778" layer="95" rot="R90" align="center-left"/>
-<attribute name="VALUE" x="60.96" y="-46.99" size="1.778" layer="96" rot="R90" align="center-left"/>
+<instance part="IC4" gate="G$1" x="55.88" y="-25.4" smashed="yes" rot="R270">
+<attribute name="NAME" x="63.5" y="-49.53" size="1.778" layer="95" rot="R90" align="center-left"/>
+<attribute name="VALUE" x="60.96" y="-49.53" size="1.778" layer="96" rot="R90" align="center-left"/>
 </instance>
 <instance part="IC5" gate="G$1" x="101.6" y="-2.54" smashed="yes" rot="R270">
@@
 <attribute name="VALUE" x="82.55" y="-72.39" size="1.778" layer="96" align="center-left"/>
 </instance>
-<instance part="C4" gate="G$1" x="38.1" y="-50.8" smashed="yes">
-<attribute name="NAME" x="36.83" y="-57.15" size="1.778" layer="95" align="center-left"/>
-<attribute name="VALUE" x="36.83" y="-59.69" size="1.778" layer="96" align="center-left"/>
+<instance part="C4" gate="G$1" x="38.1" y="-53.34" smashed="yes">
+<attribute name="NAME" x="29.21" y="-54.61" size="1.778" layer="95" rot="R90" align="center-left"/>
+<attribute name="VALUE" x="31.75" y="-54.61" size="1.778" layer="96" rot="R90" align="center-left"/>
 </instance>
 <instance part="C5" gate="G$1" x="83.82" y="-30.48" smashed="yes">
@@
 </instance>
 <instance part="GND6" gate="1" x="63.5" y="-20.32" smashed="yes">
-<attribute name="VALUE" x="60.96" y="-22.86" size="1.778" layer="96"/>
+<attribute name="VALUE" x="60.96" y="-25.4" size="1.778" layer="96"/>
 </instance>
 <instance part="C2" gate="G$1" x="35.56" y="-17.78" smashed="yes" rot="R90">
 <attribute name="NAME" x="39.37" y="-6.35" size="1.778" layer="95" align="center-left"/>
 <attribute name="VALUE" x="39.37" y="-8.89" size="1.778" layer="96" align="center-left"/>
+</instance>
+<instance part="GND7" gate="1" x="35.56" y="-58.42" smashed="yes">
+<attribute name="VALUE" x="33.02" y="-60.96" size="1.778" layer="96"/>
+</instance>
+<instance part="GND8" gate="1" x="81.28" y="-38.1" smashed="yes">
+<attribute name="VALUE" x="78.74" y="-40.64" size="1.778" layer="96"/>
 </instance>
 </instances>
@@
 <net name="N$12" class="0">
 <segment>
-<pinref part="IC4" gate="G$1" pin="OUT"/>
-<wire x1="55.88" y1="-22.86" x2="78.74" y2="-22.86" width="0.1524" layer="91"/>
 <wire x1="78.74" y1="-22.86" x2="78.74" y2="-66.04" width="0.1524" layer="91"/>
 <wire x1="78.74" y1="-66.04" x2="76.2" y2="-66.04" width="0.1524" layer="91"/>
@@
 <wire x1="81.28" y1="-66.04" x2="78.74" y2="-66.04" width="0.1524" layer="91"/>
 <junction x="78.74" y="-66.04"/>
+<pinref part="IC4" gate="G$1" pin="OUT"/>
+<wire x1="55.88" y1="-25.4" x2="55.88" y2="-22.86" width="0.1524" layer="91"/>
+<wire x1="55.88" y1="-22.86" x2="78.74" y2="-22.86" width="0.1524" layer="91"/>
 </segment>
 </net>
@@
 <segment>
 <pinref part="IC4" gate="G$1" pin="VSS"/>
-<wire x1="53.34" y1="-22.86" x2="53.34" y2="-15.24" width="0.1524" layer="91"/>
+<wire x1="53.34" y1="-25.4" x2="53.34" y2="-15.24" width="0.1524" layer="91"/>
 <wire x1="53.34" y1="-15.24" x2="63.5" y2="-15.24" width="0.1524" layer="91"/>
 <wire x1="63.5" y1="-15.24" x2="63.5" y2="-17.78" width="0.1524" layer="91"/>
@@
 <wire x1="-116.84" y1="-20.32" x2="-116.84" y2="-17.78" width="0.1524" layer="91"/>
 </segment>
+<segment>
+<pinref part="C5" gate="G$1" pin="1"/>
+<wire x1="83.82" y1="-30.48" x2="81.28" y2="-30.48" width="0.1524" layer="91"/>
+<pinref part="GND8" gate="1" pin="GND"/>
+<wire x1="81.28" y1="-35.56" x2="81.28" y2="-30.48" width="0.1524" layer="91"/>
+</segment>
+<segment>
+<pinref part="GND7" gate="1" pin="GND"/>
+<wire x1="35.56" y1="-55.88" x2="35.56" y2="-53.34" width="0.1524" layer="91"/>
+<pinref part="C4" gate="G$1" pin="1"/>
+<wire x1="35.56" y1="-53.34" x2="38.1" y2="-53.34" width="0.1524" layer="91"/>
+</segment>
 </net>
 <net name="N$3" class="0">
 <segment>
-<pinref part="IC4" gate="G$1" pin="IN+"/>
 <pinref part="R11" gate="G$1" pin="2"/>
 <wire x1="12.7" y1="-22.86" x2="35.56" y2="-22.86" width="0.1524" layer="91"/>
 <pinref part="C2" gate="G$1" pin="1"/>
+<wire x1="35.56" y1="-17.78" x2="35.56" y2="-22.86" width="0.1524" layer="91"/>
 <wire x1="35.56" y1="-22.86" x2="50.8" y2="-22.86" width="0.1524" layer="91"/>
-<wire x1="35.56" y1="-17.78" x2="35.56" y2="-22.86" width="0.1524" layer="91"/>
 <junction x="35.56" y="-22.86"/>
+<pinref part="IC4" gate="G$1" pin="IN+"/>
+<wire x1="50.8" y1="-22.86" x2="50.8" y2="-25.4" width="0.1524" layer="91"/>
 </segment>
 </net>
@@
 <pinref part="IC4" gate="G$1" pin="IN-"/>
 <wire x1="55.88" y1="-66.04" x2="58.42" y2="-66.04" width="0.1524" layer="91"/>
-<wire x1="55.88" y1="-48.26" x2="55.88" y2="-66.04" width="0.1524" layer="91"/>
+<wire x1="55.88" y1="-50.8" x2="55.88" y2="-66.04" width="0.1524" layer="91"/>
 <junction x="55.88" y="-66.04"/>
-</segment>
-</net>
-<net name="N$4" class="0">
-<segment>
-<pinref part="IC4" gate="G$1" pin="VDD"/>
-<wire x1="53.34" y1="-48.26" x2="53.34" y2="-50.8" width="0.1524" layer="91"/>
-<pinref part="C4" gate="G$1" pin="2"/>
-<wire x1="53.34" y1="-50.8" x2="50.8" y2="-50.8" width="0.1524" layer="91"/>
-</segment>
-</net>
-<net name="N$5" class="0">
-<segment>
-<pinref part="IC5" gate="G$1" pin="VDD"/>
-<wire x1="99.06" y1="-27.94" x2="99.06" y2="-30.48" width="0.1524" layer="91"/>
-<pinref part="C5" gate="G$1" pin="2"/>
-<wire x1="99.06" y1="-30.48" x2="96.52" y2="-30.48" width="0.1524" layer="91"/>
 </segment>
 </net>
@@
 <wire x1="-203.2" y1="-30.48" x2="-195.58" y2="-30.48" width="0.1524" layer="91"/>
 <label x="-193.04" y="-30.48" size="1.778" layer="95"/>
-</segment>
-<segment>
-<pinref part="C4" gate="G$1" pin="1"/>
-<wire x1="38.1" y1="-50.8" x2="35.56" y2="-50.8" width="0.1524" layer="91"/>
-<label x="35.56" y="-48.26" size="1.778" layer="95"/>
 </segment>
 <segment>
@@
 </segment>
 <segment>
-<pinref part="C5" gate="G$1" pin="1"/>
-<wire x1="83.82" y1="-30.48" x2="81.28" y2="-30.48" width="0.1524" layer="91"/>
-<label x="81.28" y="-30.48" size="1.778" layer="95"/>
-</segment>
-</net>
+<pinref part="IC4" gate="G$1" pin="VDD"/>
+<wire x1="53.34" y1="-50.8" x2="53.34" y2="-53.34" width="0.1524" layer="91"/>
+<pinref part="C4" gate="G$1" pin="2"/>
+<wire x1="53.34" y1="-53.34" x2="50.8" y2="-53.34" width="0.1524" layer="91"/>
+<wire x1="53.34" y1="-53.34" x2="53.34" y2="-55.88" width="0.1524" layer="91"/>
+<junction x="53.34" y="-53.34"/>
+<label x="50.8" y="-58.42" size="1.778" layer="95"/>
+</segment>
+<segment>
+<pinref part="IC5" gate="G$1" pin="VDD"/>
+<wire x1="99.06" y1="-27.94" x2="99.06" y2="-30.48" width="0.1524" layer="91"/>
+<pinref part="C5" gate="G$1" pin="2"/>
+<wire x1="99.06" y1="-30.48" x2="96.52" y2="-30.48" width="0.1524" layer="91"/>
+<wire x1="99.06" y1="-30.48" x2="99.06" y2="-33.02" width="0.1524" layer="91"/>
+<junction x="99.06" y="-30.48"/>
+<label x="96.52" y="-35.56" size="1.778" layer="95"/>
+</segment>
+</net>

Commit message: revisions
Parts:
- C1: value C1206F105M5RACAUTO7210 -> C0603C184K3RACAUTO; device SamacSys_Parts:C1206F105M5RACAUTO7210 -> SamacSys_Parts:C0603C184K3RACAUTO
- renumbered R11 to R8, R12 to R7
Connections:
- net GND: now also C2.2; no longer C1.1
- net N$1: no longer C1.2
- net N$3: now also C1.1; no longer C2.1
- net N$9: now also C1.2, C2.1; no longer C2.2
Other:
- moved on the sheet: C1, C2
