File: Diff_AMP.sch (EAGLE design)
At the start: 23 parts, among them IC1 NCV8711ASN500T1G, IC3 MCP1501T-25E_RW, IC4 NCS21911SN2T1G, IC5 NCS21911SN2T1G

Commit message: revision
Parts:
- added C8: GCJ188R71E183KA01J, SamacSys_Parts:GCJ188R71E183KA01J
Connections:
- net 5V: now also C7.1; no longer C6.1
- net GND: now also C8.2
- net N$3: now also C8.1
- net VIN: now also C6.1; no longer C7.1
Other:
- moved on the sheet: C4, C6, C7
Changed lines of the file:
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@@
 <part name="R1" library="SamacSys_Parts" deviceset="RT0603BRD0750KL" device=""/>
 <part name="IC1" library="SamacSys_Parts" library_urn="urn:adsk.eagle:library:35608874" deviceset="NCV8711ASN500T1G" device="" package3d_urn="urn:adsk.eagle:package:35608985/3"/>
-<part name="C6" library="SamacSys_Parts" library_urn="urn:adsk.eagle:library:35608874" deviceset="C1206F105M5RACAUTO7210" device="" package3d_urn="urn:adsk.eagle:package:35611850/2"/>
-<part name="C7" library="SamacSys_Parts" library_urn="urn:adsk.eagle:library:35608874" deviceset="C1206F105M5RACAUTO7210" device="" package3d_urn="urn:adsk.eagle:package:35611850/2"/>
 <part name="JP1" library="pinhead" library_urn="urn:adsk.eagle:library:325" deviceset="PINHD-1X4" device="" package3d_urn="urn:adsk.eagle:package:22407/2"/>
 <part name="JP2" library="pinhead" library_urn="urn:adsk.eagle:library:325" deviceset="PINHD-1X4" device="" package3d_urn="urn:adsk.eagle:package:22407/2"/>
@@
 <part name="R7" library="SamacSys_Parts" library_urn="urn:adsk.eagle:library:35608874" deviceset="ERA-3VEB1911V" device="" package3d_urn="urn:adsk.eagle:package:35608997/2"/>
 <part name="R8" library="SamacSys_Parts" library_urn="urn:adsk.eagle:library:35608874" deviceset="ERA-3VEB1911V" device="" package3d_urn="urn:adsk.eagle:package:35608997/2"/>
+<part name="C8" library="SamacSys_Parts" library_urn="urn:adsk.eagle:library:35608874" deviceset="GCJ188R71E183KA01J" device="" package3d_urn="urn:adsk.eagle:package:35615821/2"/>
+<part name="GND10" library="supply1" library_urn="urn:adsk.eagle:library:371" deviceset="GND" device=""/>
+<part name="C6" library="SamacSys_Parts" library_urn="urn:adsk.eagle:library:35608874" deviceset="C1206F105M5RACAUTO7210" device="" package3d_urn="urn:adsk.eagle:package:35611850/2"/>
+<part name="C7" library="SamacSys_Parts" library_urn="urn:adsk.eagle:library:35608874" deviceset="C1206F105M5RACAUTO7210" device="" package3d_urn="urn:adsk.eagle:package:35611850/2"/>
 </parts>
 <sheets>
@@
 <attribute name="VALUE" x="82.55" y="-72.39" size="1.778" layer="96" align="center-left"/>
 </instance>
-<instance part="C4" gate="G$1" x="38.1" y="-53.34" smashed="yes">
-<attribute name="NAME" x="29.21" y="-54.61" size="1.778" layer="95" rot="R90" align="center-left"/>
-<attribute name="VALUE" x="31.75" y="-54.61" size="1.778" layer="96" rot="R90" align="center-left"/>
+<instance part="C4" gate="G$1" x="35.56" y="-53.34" smashed="yes">
+<attribute name="NAME" x="21.59" y="-46.99" size="1.778" layer="95" align="center-left"/>
+<attribute name="VALUE" x="21.59" y="-49.53" size="1.778" layer="96" align="center-left"/>
 </instance>
 <instance part="C5" gate="G$1" x="83.82" y="-30.48" smashed="yes">
@@
 <attribute name="VALUE" x="-151.13" y="7.62" size="1.778" layer="96" align="center-left"/>
 </instance>
-<instance part="C6" gate="G$1" x="-116.84" y="-5.08" smashed="yes" rot="R270">
-<attribute name="NAME" x="-113.03" y="-3.81" size="1.778" layer="95" align="center-left"/>
-<attribute name="VALUE" x="-113.03" y="-6.35" size="1.778" layer="96" align="center-left"/>
-</instance>
-<instance part="C7" gate="G$1" x="-165.1" y="-2.54" smashed="yes" rot="R270">
-<attribute name="NAME" x="-161.29" y="-6.35" size="1.778" layer="95" align="center-left"/>
-<attribute name="VALUE" x="-161.29" y="-8.89" size="1.778" layer="96" align="center-left"/>
-</instance>
 <instance part="JP1" gate="A" x="-200.66" y="0" smashed="yes">
 <attribute name="NAME" x="-207.01" y="8.255" size="1.778" layer="95"/>
@@
 <attribute name="VALUE" x="52.07" y="13.97" size="1.778" layer="96" align="center-left"/>
 </instance>
-<instance part="GND7" gate="1" x="35.56" y="-58.42" smashed="yes">
-<attribute name="VALUE" x="33.02" y="-60.96" size="1.778" layer="96"/>
+<instance part="GND7" gate="1" x="33.02" y="-58.42" smashed="yes">
+<attribute name="VALUE" x="30.48" y="-60.96" size="1.778" layer="96"/>
 </instance>
 <instance part="GND8" gate="1" x="81.28" y="-38.1" smashed="yes">
@@
 <attribute name="NAME" x="8.89" y="-16.51" size="1.778" layer="95" align="center-left"/>
 <attribute name="VALUE" x="8.89" y="-19.05" size="1.778" layer="96" align="center-left"/>
+</instance>
+<instance part="C8" gate="G$1" x="30.48" y="-35.56" smashed="yes" rot="R180">
+<attribute name="NAME" x="13.97" y="-26.67" size="1.778" layer="95" align="center-left"/>
+<attribute name="VALUE" x="13.97" y="-29.21" size="1.778" layer="96" align="center-left"/>
+</instance>
+<instance part="GND10" gate="1" x="12.7" y="-45.72" smashed="yes">
+<attribute name="VALUE" x="10.16" y="-50.8" size="1.778" layer="96"/>
+</instance>
+<instance part="C6" gate="G$1" x="-165.1" y="-2.54" smashed="yes" rot="R270">
+<attribute name="NAME" x="-158.75" y="-11.43" size="1.778" layer="95" rot="R270" align="center-left"/>
+<attribute name="VALUE" x="-161.29" y="-11.43" size="1.778" layer="96" rot="R270" align="center-left"/>
+</instance>
+<instance part="C7" gate="G$1" x="-116.84" y="-5.08" smashed="yes" rot="R270">
+<attribute name="NAME" x="-110.49" y="-13.97" size="1.778" layer="95" rot="R270" align="center-left"/>
+<attribute name="VALUE" x="-113.03" y="-13.97" size="1.778" layer="96" rot="R270" align="center-left"/>
 </instance>
 </instances>
@@
 </segment>
 <segment>
-<pinref part="C7" gate="G$1" pin="2"/>
-<pinref part="GND1" gate="1" pin="GND"/>
-<wire x1="-165.1" y1="-15.24" x2="-165.1" y2="-17.78" width="0.1524" layer="91"/>
-</segment>
-<segment>
 <pinref part="IC5" gate="G$1" pin="VSS"/>
 <wire x1="99.06" y1="-2.54" x2="99.06" y2="10.16" width="0.1524" layer="91"/>
@@
 </segment>
 <segment>
-<pinref part="GND2" gate="1" pin="GND"/>
-<pinref part="C6" gate="G$1" pin="2"/>
-<wire x1="-116.84" y1="-20.32" x2="-116.84" y2="-17.78" width="0.1524" layer="91"/>
-</segment>
-<segment>
 <pinref part="C5" gate="G$1" pin="1"/>
 <wire x1="83.82" y1="-30.48" x2="81.28" y2="-30.48" width="0.1524" layer="91"/>
@@
 <segment>
 <pinref part="GND7" gate="1" pin="GND"/>
-<wire x1="35.56" y1="-55.88" x2="35.56" y2="-53.34" width="0.1524" layer="91"/>
+<wire x1="33.02" y1="-55.88" x2="33.02" y2="-53.34" width="0.1524" layer="91"/>
 <pinref part="C4" gate="G$1" pin="1"/>
-<wire x1="35.56" y1="-53.34" x2="38.1" y2="-53.34" width="0.1524" layer="91"/>
+<wire x1="33.02" y1="-53.34" x2="35.56" y2="-53.34" width="0.1524" layer="91"/>
 </segment>
 <segment>
@@
 <wire x1="63.5" y1="17.78" x2="63.5" y2="22.86" width="0.1524" layer="91"/>
 </segment>
+<segment>
+<pinref part="C8" gate="G$1" pin="2"/>
+<wire x1="17.78" y1="-35.56" x2="12.7" y2="-35.56" width="0.1524" layer="91"/>
+<pinref part="GND10" gate="1" pin="GND"/>
+<wire x1="12.7" y1="-35.56" x2="12.7" y2="-43.18" width="0.1524" layer="91"/>
+</segment>
+<segment>
+<pinref part="C6" gate="G$1" pin="2"/>
+<pinref part="GND1" gate="1" pin="GND"/>
+<wire x1="-165.1" y1="-15.24" x2="-165.1" y2="-17.78" width="0.1524" layer="91"/>
+</segment>
+<segment>
+<pinref part="C7" gate="G$1" pin="2"/>
+<pinref part="GND2" gate="1" pin="GND"/>
+<wire x1="-116.84" y1="-17.78" x2="-116.84" y2="-20.32" width="0.1524" layer="91"/>
+</segment>
 </net>
 <net name="N$3" class="0">
@@
 <wire x1="12.7" y1="-22.86" x2="38.1" y2="-22.86" width="0.1524" layer="91"/>
 <pinref part="IC4" gate="G$1" pin="IN+"/>
-<wire x1="38.1" y1="-22.86" x2="50.8" y2="-22.86" width="0.1524" layer="91"/>
+<wire x1="38.1" y1="-22.86" x2="43.18" y2="-22.86" width="0.1524" layer="91"/>
+<wire x1="43.18" y1="-22.86" x2="50.8" y2="-22.86" width="0.1524" layer="91"/>
 <wire x1="50.8" y1="-22.86" x2="50.8" y2="-25.4" width="0.1524" layer="91"/>
 <pinref part="C1" gate="G$1" pin="1"/>
@@
 <junction x="38.1" y="-22.86"/>
 <pinref part="R8" gate="G$1" pin="2"/>
+<pinref part="C8" gate="G$1" pin="1"/>
+<wire x1="30.48" y1="-35.56" x2="43.18" y2="-35.56" width="0.1524" layer="91"/>
+<wire x1="43.18" y1="-35.56" x2="43.18" y2="-22.86" width="0.1524" layer="91"/>
+<junction x="43.18" y="-22.86"/>
 </segment>
 </net>
@@
 <pinref part="IC1" gate="G$1" pin="IN"/>
 <wire x1="-152.4" y1="2.54" x2="-165.1" y2="2.54" width="0.1524" layer="91"/>
-<pinref part="C7" gate="G$1" pin="1"/>
+<label x="-170.18" y="5.08" size="1.778" layer="95"/>
+<pinref part="C6" gate="G$1" pin="1"/>
+<wire x1="-165.1" y1="2.54" x2="-170.18" y2="2.54" width="0.1524" layer="91"/>
 <wire x1="-165.1" y1="-2.54" x2="-165.1" y2="2.54" width="0.1524" layer="91"/>
-<wire x1="-165.1" y1="2.54" x2="-170.18" y2="2.54" width="0.1524" layer="91"/>
 <junction x="-165.1" y="2.54"/>
-<label x="-170.18" y="5.08" size="1.778" layer="95"/>
 </segment>
 <segment>
@@
 <wire x1="-78.74" y1="-22.86" x2="-66.04" y2="-22.86" width="0.1524" layer="91"/>
 <pinref part="IC1" gate="G$1" pin="OUT"/>
-<wire x1="-116.84" y1="0" x2="-119.38" y2="0" width="0.1524" layer="91"/>
-<pinref part="C6" gate="G$1" pin="1"/>
-<wire x1="-116.84" y1="-5.08" x2="-116.84" y2="0" width="0.1524" layer="91"/>
+<wire x1="-119.38" y1="0" x2="-116.84" y2="0" width="0.1524" layer="91"/>
+<junction x="-78.74" y="0"/>
 <wire x1="-116.84" y1="0" x2="-78.74" y2="0" width="0.1524" layer="91"/>
-<junction x="-116.84" y="0"/>
-<junction x="-78.74" y="0"/>
 <wire x1="-78.74" y1="0" x2="-78.74" y2="2.54" width="0.1524" layer="91"/>
 <label x="-78.74" y="5.08" size="1.778" layer="95"/>
+<pinref part="C7" gate="G$1" pin="1"/>
+<wire x1="-116.84" y1="-5.08" x2="-116.84" y2="0" width="0.1524" layer="91"/>
+<junction x="-116.84" y="0"/>
 </segment>
 <segment>
@@
 <wire x1="53.34" y1="-50.8" x2="53.34" y2="-53.34" width="0.1524" layer="91"/>
 <pinref part="C4" gate="G$1" pin="2"/>
-<wire x1="53.34" y1="-53.34" x2="50.8" y2="-53.34" width="0.1524" layer="91"/>
+<wire x1="53.34" y1="-53.34" x2="48.26" y2="-53.34" width="0.1524" layer="91"/>
 <wire x1="53.34" y1="-53.34" x2="53.34" y2="-55.88" width="0.1524" layer="91"/>
 <junction x="53.34" y="-53.34"/>
